File: pcb/codec_and_audio.kicad_sch (KiCad schematic)
At the start: 7 parts, among them IC3 PCM3060PWR

Commit message: progress on audio pcb
Parts:
- added C15: 100nF, symbol Device:C
- added C16: 10uF, symbol Device:C_Polarized
Connections:
- net 3V3: now also IC3.28 (MODE)
- net GND: now also C15.1, C16.2
- net at IC3.21 (VCOM): now also C15.2, C16.1
Other:
- note added: "now it's in SPI mode"
- note removed: "mode, 4 ways to connect things, look into which is the right one"
- moved on the sheet: C10, C11, C12, C13, C14, C9, IC3

Commit message: progress on understanding audio schematics
Parts:
- added J2: AudioJack3, symbol Connector_Audio:AudioJack3
Connections:
- net VCOM: now reaches C15.2, C16.1, IC3.21 (VCOM)
- net 3V3 renamed VDD
Other:
- note added: "3v3 from power supply"
- note added: "5v from power supply"
- note added: "DGND, AGND1, AGND2, SGND all connected together"
- note added: "Vcom is my A ref GND basically"
- note added: "big circuit example b"
- note added: "filtering stuff i guess"
- moved on the sheet: C10, C11

Commit message: couple of things
Parts:
- removed J2: AudioJack3, symbol Connector_Audio:AudioJack3
- added J3: AudioJack3_Dual_Switch, symbol Connector_Audio:AudioJack3_Dual_Switch
Other:
- note added: "sleeve is connected to VCOM"
Changed lines of the file:
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@@
+    (effects (font (size 1.27 1.27)) (justify left bottom))
+  )
+  (text "sleeve is connected to VCOM\n" (at 205.74 18.415 0)
     (effects (font (size 1.27 1.27)) (justify left bottom))
   )
@@
     (effects (font (size 1.27 1.27)) (justify right))
   )
+  (symbol (lib_id "Connector_Audio:AudioJack3_Dual_Switch") (at 217.17 33.02 0) (mirror y) (unit 1)
+    (in_bom yes) (on_board yes) (dnp no)
+    (property "Reference" "J3" (at 219.7735 21.59 0)
+      (effects (font (size 1.27 1.27)))
+    )
+    (property "Value" "AudioJack3_Dual_Switch" (at 219.7735 24.13 0)
+      (effects (font (size 1.27 1.27)))
+    )
+    (property "Footprint" "" (at 218.44 33.02 0)
+      (effects (font (size 1.27 1.27)) hide)
+    )
+    (property "Datasheet" "~" (at 218.44 33.02 0)
+      (effects (font (size 1.27 1.27)) hide)
+    )
+    (pin "R1")
+    (pin "RN1")
+    (pin "S1")
+    (pin "SN1")
+    (pin "T1")
+    (pin "TN1")
+    (pin "R2")
+    (pin "RN2")
+    (pin "S2")
+    (pin "SN2")
+    (pin "T2")
+    (pin "TN2")
+    (instances
+      (project "bt_pcb"
+        (path "/eb787481-08cd-41a4-a128-173fa6227c32/4ada0139-8712-47ce-9d4c-ab8fef312f7b"
+          (reference "J3") (unit 1)
+        )
+      )
+    )
+  )
   (symbol (lib_id "Device:C_Polarized") (at 158.115 64.77 180) (unit 1)
     (in_bom yes) (on_board yes) (dnp no) (fields_autoplaced)
@@
     )
   )
-  (symbol (lib_id "Connector_Audio:AudioJack3") (at 242.57 26.67 0) (mirror y) (unit 1)
-    (in_bom yes) (on_board yes) (dnp no)
-    (property "Reference" "J2" (at 244.475 17.78 0)
-      (effects (font (size 1.27 1.27)))
-    )
-    (property "Value" "AudioJack3" (at 244.475 20.32 0)
-      (effects (font (size 1.27 1.27)))
-    )
-    (property "Footprint" "" (at 242.57 26.67 0)
-      (effects (font (size 1.27 1.27)) hide)
-    )
-    (property "Datasheet" "~" (at 242.57 26.67 0)
-      (effects (font (size 1.27 1.27)) hide)
-    )
-    (pin "S")
-    (pin "T")
-    (pin "R")
-    (instances
-      (project "bt_pcb"
-        (path "/eb787481-08cd-41a4-a128-173fa6227c32/4ada0139-8712-47ce-9d4c-ab8fef312f7b"
-          (reference "J2") (unit 1)
-        )
-      )
-    )
-  )
   (symbol (lib_id "SamacSys_Parts:PCM3060PWR") (at 75.565 45.72 0) (unit 1)
     (in_bom yes) (on_board yes) (dnp no) (fields_autoplaced)
@@
       (effects (font (size 1.27 1.27)) (justify left top) hide)
     )
+    (pin "1")
+    (pin "10")
     (pin "11")
+    (pin "12")
+    (pin "13")
+    (pin "14")
+    (pin "15")
+    (pin "16")
+    (pin "17")
     (pin "18")
+    (pin "19")
+    (pin "2")
+    (pin "20")
+    (pin "21")
     (pin "22")
+    (pin "23")
+    (pin "24")
     (pin "25")
-    (pin "23")
-    (pin "13")
-    (pin "24")
-    (pin "1")
+    (pin "26")
     (pin "27")
+    (pin "28")
     (pin "3")
+    (pin "4")
+    (pin "5")
     (pin "6")
-    (pin "17")
+    (pin "7")
+    (pin "8")
     (pin "9")
-    (pin "7")
-    (pin "19")
-    (pin "10")
-    (pin "26")
-    (pin "21")
-    (pin "14")
-    (pin "5")
-    (pin "15")
-    (pin "4")
-    (pin "8")
-    (pin "28")
-    (pin "2")
-    (pin "20")
-    (pin "16")
-    (pin "12")
-    (instances
-      (project "bt_pcb"
+    (instances
+      (project "bt_pcb"

Commit message: progress on audio in
Parts:
- added C17: 10uF, symbol Device:C_Polarized
- added C18: 330pF, symbol Device:C
- added R1: R, symbol Device:R
- added R2: 20k, symbol Device:R
- added U1: ${SIM.PARAMS}, symbol Simulation_SPICE:OPAMP
Connections:
- net at J3.TN1: now also C17.2
- new net: C18.1, R1.2, U1.5
- new net: C18.2, R1.1, R2.2, U1.2 (-)
- new net: C17.1, R2.1
Other:
- note added: "high pass filter"
- note added: "low pass filter"
- note added: "vcom is vcc/2"
- moved on the sheet: C10, C11, C12, C13, C14, C15, C16, C9, IC3, J3A
