File: pcb/codec_and_audio.kicad_sch (KiCad schematic)
At the start: 11 parts, among them U1 CS4272

Commit message: progress on hp
Other:
- sheet Output A ports: added none; removed AOUT_HP
- sheet Output B ports: added none; removed BOUT_HP
- sheet Output HP ports: added LEFT+, LEFT-, RIGHT+, RIGHT-, SCL, SD, SDA; removed none
- moved on the sheet: C10, C11, C12, C14, C15, C16, C18, C25, C35, C9, U1

Commit message: a lot of audio finished, now onto ui
Connections:
- net Input A/AIN+ renamed Audio input/INA+
- net Input A/AIN- renamed Audio input/INA-
- net Input B/BIN+ renamed Audio input/INB+
- net Input B/BIN- renamed Audio input/INB-
- net Output A/AOUT+ renamed Audio HP output/LEFT+
- net Output A/AOUT- renamed Audio HP output/LEFT-
- net Output B/BOUT+ renamed Audio HP output/RIGHT+
- net Output B/BOUT- renamed Audio HP output/RIGHT-
Other:
- sheet Output HP renamed Audio HP output
- removed sheet Input A
- removed sheet Input B
- removed sheet Output A
- removed sheet Output B
- added sheet Audio input (audio_input.kicad_sch)
- added sheet Audio ouput (audio_output.kicad_sch)

Commit message: a lot of work! almost ready for rev
Connections:
- net Audio HP output/LEFT+ renamed CODEC_OUTA+
- net Audio HP output/LEFT- renamed CODEC_OUTA-
- net Audio HP output/RIGHT+ renamed CODEC_OUTB+
- net Audio HP output/RIGHT- renamed CODEC_OUTB-
- net Audio input/INA+ renamed CODEC_INA+
- net Audio input/INA- renamed CODEC_INA-
- net Audio input/INB+ renamed CODEC_INB+
- net Audio input/INB- renamed CODEC_INB-
- net CS_LRCK renamed CODEC_I2S_WS
- net CS_MCLK renamed CODEC_I2S_MCK
- net CS_RST renamed CODEC_RST
- net CS_SCL renamed CODEC_I2C_SCL
- net CS_SCLK renamed CODEC_I2S_CK
- net CS_SDA renamed CODEC_I2C_SDA
- net CS_SDIN renamed CODEC_I2S_SDI
- net CS_SDOUT renamed CODEC_I2S_SDO
Other:
- sheet Audio HP output ports: added none; removed LEFT+, LEFT-, RIGHT+, RIGHT-, SCL, SD, SDA
- sheet Audio input ports: added none; removed INA+, INA-, INA_SWITCH, INB+, INB-, INB_SWITCH
- sheet Audio ouput ports: added none; removed OUTA+, OUTA-, OUTA_SWITCH, OUTB+, OUTB-, OUTB_SWITCH
- moved on the sheet: C10, C11, C12, C14, C15, C16, C18, C25, C35, C9, U1

Commit message: starting the revision from ed
Parts:
- removed C10: 100nF, symbol Device:C
- removed C9: 1uF, symbol Device:C
- added C32: 10uF, symbol Device:C
Connections:
- net +5V: now also U1.20 (VA), C32.1
- net GND: now also C32.2; no longer U1.20 (VA)
Other:
- note added: "really really close to the IC!"
- moved on the sheet: C18, C25
