File: pcb/input_a.kicad_sch (KiCad schematic)
At the start: 15 parts, among them J4 AudioJack2, J5 XLR3_Ground, U2 MCP6002-xMC

Commit message: big progress!
Parts:
- removed J4: AudioJack2, symbol Connector_Audio:AudioJack2
- removed U2: MCP6002-xMC, Package_DFN_QFN:DFN-8-1EP_3x2mm_P0.5mm_EP1.75x1.45mm, symbol Amplifier_Operational:MCP6002-xMC
- added C44: 10uF, symbol Device:C_Polarized
- added C45, C46: 470pF, symbol Device:C
- added C47: 2700pF, symbol Device:C
- added C48, C49: 10nF, symbol Device:C_Polarized
- added J10: AudioJack2_Dual_Switch, symbol Connector_Audio:AudioJack2_Dual_Switch
- added R16, R17, R18, R19: 10k, symbol Device:R
- added U4: MCP6004, symbol Amplifier_Operational:MCP6004
Connections:
- net 5V0: now also U4.4 (V+)
- net GND: now also C48.2, C49.2, J10.S1, J10.SN1, U4.11 (V-)
- net VCOM: now also C48.1, C49.1, U4.10 (+), U4.12 (+)
- net at C33.1, R7.1: now also U4.7
- net at C33.2, R6.1: now also U4.6 (-)
- net at C17.1, R2.2: now also U4.5 (+)
- net at C13.1, R1.1: now also U4.3 (+)
- net at C36.1, R9.1: now also U4.1
- net at C36.2, R8.1: now also U4.2 (-)
- new net: C44.1, R16.1
- new net: C45.2, R16.2, R17.1, U4.9 (-)
- new net: C45.1, C47.1, R17.2, R19.1, U4.8
- new net: C46.2, R18.1, R19.2, U4.13 (-)
- new net: C46.1, C47.2, R18.2, U4.14
- new net: C44.2, J10.T1, J10.TN1
Other:
- note added: "The switching circuit is still missing"
- moved on the sheet: C13, C17, C31, C33, C36, C37, J5, R1, R2, R6, R7, R8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

Commit message: progress
Changed lines of the file:
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@@
-    (effects (font (size 1.27 1.27)) (justify left))
-  )
-  (hierarchical_label "AINCS" (shape input) (at 210.185 90.17 0) (fields_autoplaced)
     (effects (font (size 1.27 1.27)) (justify left))
   )

Commit message: making up my mind on the heaphones
Parts:
- added J12: AudioJack3_Dual_Switch, symbol Connector_Audio:AudioJack3_Dual_Switch
Connections:
- net GND: now also J12.T1, J12.TN1
- net 5V0 renamed +5V
- new net: J12.R1, J12.RN1
- new net: J12.S1, J12.SN1
Other:
- moved on the sheet: U4E
Changed lines of the file:
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@@
   (junction (at 104.14 128.905) (diameter 0) (color 0 0 0 0)
   )
+  (junction (at 60.96 76.2) (diameter 0) (color 0 0 0 0)
+  )
   (junction (at 121.92 126.365) (diameter 0) (color 0 0 0 0)
   )
@@
     (stroke (width 0) (type default))
   )
+  (wire (pts (xy 60.96 73.66) (xy 60.96 76.2))
+    (stroke (width 0) (type default))
+  )
   (wire (pts (xy 154.94 135.255) (xy 154.94 146.05))
     (stroke (width 0) (type default))
@@
     (stroke (width 0) (type default))
   )
+  (wire (pts (xy 64.77 76.2) (xy 60.96 76.2))
+    (stroke (width 0) (type default))
+  )
   (wire (pts (xy 158.115 39.37) (xy 165.735 39.37))
     (stroke (width 0) (type default))
@@
     (stroke (width 0) (type default))
   )
+  (wire (pts (xy 60.96 68.58) (xy 60.96 71.12))
+    (stroke (width 0) (type default))
+  )
   (wire (pts (xy 116.84 80.645) (xy 107.315 80.645))
     (stroke (width 0) (type default))
@@
     (stroke (width 0) (type default))
   )
+  (wire (pts (xy 64.77 78.74) (xy 64.77 76.2))
+    (stroke (width 0) (type default))
+  )
   (wire (pts (xy 139.7 135.255) (xy 139.7 146.05))
     (stroke (width 0) (type default))
@@
   )
   (wire (pts (xy 165.1 67.31) (xy 157.48 67.31))
+    (stroke (width 0) (type default))
+  )
+  (wire (pts (xy 60.96 63.5) (xy 60.96 66.04))
     (stroke (width 0) (type default))
   )
@@
     (effects (font (size 1.27 1.27)) (justify left))
   )
-  (hierarchical_label "5V0" (shape input) (at 62.23 52.07 90) (fields_autoplaced)
-    (effects (font (size 1.27 1.27)) (justify left))
-  )
   (hierarchical_label "VCOM" (shape input) (at 126.365 160.02 180) (fields_autoplaced)
     (effects (font (size 1.27 1.27)) (justify right))
@@
         (path "/eb787481-08cd-41a4-a128-173fa6227c32/4ada0139-8712-47ce-9d4c-ab8fef312f7b/fb924787-351e-471a-8373-66e7df7b6a71"
           (reference "C49") (unit 1)
+        )
+      )
+    )
+  )
+  (symbol (lib_id "power:GND") (at 64.77 78.74 0) (mirror y) (unit 1)
+    (in_bom yes) (on_board yes) (dnp no) (fields_autoplaced)
+    (property "Reference" "#PWR077" (at 64.77 85.09 0)
+      (effects (font (size 1.27 1.27)) hide)
+    )
+    (property "Value" "GND" (at 64.77 83.185 0)
+      (effects (font (size 1.27 1.27)))
+    )
+    (property "Footprint" "" (at 64.77 78.74 0)
+      (effects (font (size 1.27 1.27)) hide)
+    )
+    (property "Datasheet" "" (at 64.77 78.74 0)
+      (effects (font (size 1.27 1.27)) hide)
+    )
+    (pin "1")
+    (instances
+      (project "bt_pcb"
+        (path "/eb787481-08cd-41a4-a128-173fa6227c32/4ada0139-8712-47ce-9d4c-ab8fef312f7b/fb924787-351e-471a-8373-66e7df7b6a71"
+          (reference "#PWR077") (unit 1)
         )
       )
@@
     )
   )
-  (symbol (lib_id "Amplifier_Operational:MCP6004") (at 64.77 59.69 0) (unit 5)
-    (in_bom yes) (on_board yes) (dnp no) (fields_autoplaced)
-    (property "Reference" "U4" (at 64.008 58.42 0)
-      (effects (font (size 1.27 1.27)) (justify left))
-    )
-    (property "Value" "MCP6004" (at 64.008 60.96 0)
-      (effects (font (size 1.27 1.27)) (justify left))
-    )
-    (property "Footprint" "" (at 63.5 57.15 0)
-      (effects (font (size 1.27 1.27)) hide)
-    )
-    (property "Datasheet" "http://ww1.microchip.com/downloads/en/DeviceDoc/21733j.pdf" (at 66.04 54.61 0)
+  (symbol (lib_id "Amplifier_Operational:MCP6004") (at 83.82 32.385 0) (unit 5)
+    (in_bom yes) (on_board yes) (dnp no) (fields_autoplaced)
+    (property "Reference" "U4" (at 83.058 31.115 0)
+      (effects (font (size 1.27 1.27)) (justify left))
+    )
+    (property "Value" "MCP6004" (at 83.058 33.655 0)
+      (effects (font (size 1.27 1.27)) (justify left))
+    )
+    (property "Footprint" "" (at 82.55 29.845 0)
+      (effects (font (size 1.27 1.27)) hide)
+    )
+    (property "Datasheet" "http://ww1.microchip.com/downloads/en/DeviceDoc/21733j.pdf" (at 85.09 27.305 0)
       (effects (font (size 1.27 1.27)) hide)
     )
@@
     )
   )
-  (symbol (lib_id "power:GND") (at 62.23 67.31 0) (mirror y) (unit 1)
-    (in_bom yes) (on_board yes) (dnp no) (fields_autoplaced)
-    (property "Reference" "#PWR037" (at 62.23 73.66 0)
-      (effects (font (size 1.27 1.27)) hide)
-    )
-    (property "Value" "GND" (at 62.23 71.755 0)
-      (effects (font (size 1.27 1.27)))
-    )
-    (property "Footprint" "" (at 62.23 67.31 0)
-      (effects (font (size 1.27 1.27)) hide)
-    )
-    (property "Datasheet" "" (at 62.23 67.31 0)
+  (symbol (lib_id "power:GND") (at 81.28 40.005 0) (mirror y) (unit 1)
+    (in_bom yes) (on_board yes) (dnp no) (fields_autoplaced)
+    (property "Reference" "#PWR037" (at 81.28 46.355 0)
+      (effects (font (size 1.27 1.27)) hide)
+    )
+    (property "Value" "GND" (at 81.28 44.45 0)
+      (effects (font (size 1.27 1.27)))
+    )
+    (property "Footprint" "" (at 81.28 40.005 0)
+      (effects (font (size 1.27 1.27)) hide)
+    )
+    (property "Datasheet" "" (at 81.28 40.005 0)
       (effects (font (size 1.27 1.27)) hide)
     )
@@
         (path "/eb787481-08cd-41a4-a128-173fa6227c32/4ada0139-8712-47ce-9d4c-ab8fef312f7b/fb924787-351e-471a-8373-66e7df7b6a71"
           (reference "R6") (unit 1)
+        )
+      )
+    )
+  )
+  (symbol (lib_id "power:+5V") (at 81.28 24.765 0) (unit 1)
+    (in_bom yes) (on_board yes) (dnp no) (fields_autoplaced)
+    (property "Reference" "#PWR049" (at 81.28 28.575 0)
+      (effects (font (size 1.27 1.27)) hide)
+    )
+    (property "Value" "+5V" (at 81.28 20.32 0)
+      (effects (font (size 1.27 1.27)))
+    )
+    (property "Footprint" "" (at 81.28 24.765 0)
+      (effects (font (size 1.27 1.27)) hide)
+    )
+    (property "Datasheet" "" (at 81.28 24.765 0)
+      (effects (font (size 1.27 1.27)) hide)
+    )
+    (pin "1")
+    (instances
+      (project "bt_pcb"
+        (path "/eb787481-08cd-41a4-a128-173fa6227c32/4ada0139-8712-47ce-9d4c-ab8fef312f7b/fb924787-351e-471a-8373-66e7df7b6a71"
+          (reference "#PWR049") (unit 1)
         )
       )
@@
         )
       )
+    )
+  )
+  (symbol (lib_id "Connector_Audio:AudioJack3_Dual_Switch") (at 55.88 68.58 0) (unit 1)
+    (in_bom yes) (on_board yes) (dnp no) (fields_autoplaced)
+    (property "Reference" "J12" (at 53.2765 57.785 0)
+      (effects (font (size 1.27 1.27)))
+    )
+    (property "Value" "AudioJack3_Dual_Switch" (at 53.2765 60.325 0)
+      (effects (font (size 1.27 1.27)))
+    )
+    (property "Footprint" "" (at 54.61 68.58 0)
+      (effects (font (size 1.27 1.27)) hide)
+    )
+    (property "Datasheet" "~" (at 54.61 68.58 0)
+      (effects (font (size 1.27 1.27)) hide)
+    )
+    (pin "S2")
+    (pin "TN1")
+    (pin "R1")
+    (pin "SN1")
+    (pin "SN2")
+    (pin "T2")
+    (pin "RN2")
+    (pin "T1")
+    (pin "TN2")
+    (pin "R2")
+    (pin "RN1")
+    (pin "S1")
+    (instances
+      (project "bt_pcb"
+        (path "/eb787481-08cd-41a4-a128-173fa6227c32/4ada0139-8712-47ce-9d4c-ab8fef312f7b/fb924787-351e-471a-8373-66e7df7b6a71"
+          (reference "J12") (unit 1)
+        )
+      )
