File: pcb/input_b.kicad_sch (KiCad schematic)
At the start: 15 parts, among them J3 AudioJack2, J7 XLR3_Ground, U3 MCP6002-xMC

Commit message: big progress!
Parts:
- removed C40: 10nF, symbol Device:C_Polarized
- removed C41, C42: 470pF, symbol Device:C
- removed C43: 2700pF, symbol Device:C
- removed J3: AudioJack2, symbol Connector_Audio:AudioJack2
- removed U3: MCP6002-xMC, Package_DFN_QFN:DFN-8-1EP_3x2mm_P0.5mm_EP1.75x1.45mm, symbol Amplifier_Operational:MCP6002-xMC
- added C40, C51, C53, C54: 470pF, symbol Device:C
- added C41, C42: 10uF, symbol Device:C_Polarized
- added C43, C50: 10nF, symbol Device:C_Polarized
- added C52, C55: 2700pF, symbol Device:C
- added J3: AudioJack2_Dual_Switch, symbol Connector_Audio:AudioJack2_Dual_Switch
- added R20, R22: 634, symbol Device:R
- added R21, R23: 91, symbol Device:R
- added U2: MCP6004, symbol Amplifier_Operational:MCP6004
- C39: value 10uF -> 10nF
- R12, R14: value 634 -> 10k
- R13, R15: value 91 -> 10k
Connections:
- net 5V0: now also U2.4 (V+)
- net BIN+: now also C55.1, R22.2, R23.2; no longer R14.2, R15.2
- net BIN-: now also C55.2, R20.2, R21.2; no longer R12.2, R13.2
- net GND: now also C39.2, C43.2, C50.2, J3.S1, J3.SN1, U2.11 (V-)
- net VCOM: now also C39.1, R12.2, R13.1, C43.1, C50.1, U2.10 (+), U2.12 (+); no longer R10.2, R11.1
- net at R11.2: now also R14.1, C40.1, C52.1, U2.8; no longer C39.1
- net at R15.1: now also R14.2, C51.2, U2.13 (-)
- net at J7.2: now also C41.2; no longer C38.2
- net at R12.1: now also C41.1, U2.3 (+)
- net at J7.3: now also C42.2; no longer C39.2
- new net: C54.1, R23.1, U2.1
- new net: C54.2, R22.1, U2.2 (-)
- new net: C51.1, C52.2, R15.2, U2.14
- new net: C42.1, R13.2, U2.5 (+)
- new net: C40.2, R10.2, R11.1, U2.9 (-)
- new net: C53.1, R21.1, U2.7
- new net: C53.2, R20.1, U2.6 (-)
- new net: C38.2, J3.T1, J3.TN1
Other:
- note added: "The switching circuit is still missing"

Commit message: progress
Changed lines of the file:
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@@
-    (effects (font (size 1.27 1.27)) (justify left))
-  )
-  (hierarchical_label "BINCS" (shape input) (at 206.375 113.665 0) (fields_autoplaced)
     (effects (font (size 1.27 1.27)) (justify left))
   )

Commit message: making up my mind on the heaphones
Connections:
- net 5V0 renamed +5V
Changed lines of the file:
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@@
-    (effects (font (size 1.27 1.27)) (justify left))
-  )
-  (hierarchical_label "5V0" (shape input) (at 53.975 53.975 90) (fields_autoplaced)
     (effects (font (size 1.27 1.27)) (justify left))
   )
@@
         )
       )
+    )
+  )
+  (symbol (lib_id "power:+5V") (at 53.975 53.975 0) (unit 1)
+    (in_bom yes) (on_board yes) (dnp no) (fields_autoplaced)
+    (property "Reference" "#PWR051" (at 53.975 57.785 0)
+      (effects (font (size 1.27 1.27)) hide)
+    )
+    (property "Value" "+5V" (at 53.975 49.53 0)
+      (effects (font (size 1.27 1.27)))
+    )
+    (property "Footprint" "" (at 53.975 53.975 0)
+      (effects (font (size 1.27 1.27)) hide)
+    )
+    (property "Datasheet" "" (at 53.975 53.975 0)
+      (effects (font (size 1.27 1.27)) hide)
+    )
+    (pin "1")
+    (instances
+      (project "bt_pcb"
+        (path "/eb787481-08cd-41a4-a128-173fa6227c32/4ada0139-8712-47ce-9d4c-ab8fef312f7b/393cdf85-7f27-4cef-b6a8-755ca71a41cd"
+          (reference "#PWR051") (unit 1)
+        )
+      )
