File: pcb/output_a.kicad_sch (KiCad schematic)
At the start: 17 parts, among them J4 AudioJack2_Dual_Switch, J9 XLR3_Ground, U3 MCP6004

Commit message: making up my mind on the heaphones
Connections:
- net 5V0 renamed +5V
- net T renamed AOUT_HP
Changed lines of the file:
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@@
   (junction (at 156.21 81.28) (diameter 0) (color 0 0 0 0)
+  )
+  (junction (at 156.845 66.675) (diameter 0) (color 0 0 0 0)
   )
   (junction (at 227.33 68.58) (diameter 0) (color 0 0 0 0)
@@
     (stroke (width 0) (type default))
   )
+  (wire (pts (xy 164.465 59.69) (xy 156.845 59.69))
+    (stroke (width 0) (type default))
+  )
   (wire (pts (xy 93.98 49.53) (xy 93.98 57.785))
     (stroke (width 0) (type default))
@@
     (stroke (width 0) (type default))
   )
-  (wire (pts (xy 148.59 66.675) (xy 156.21 66.675))
+  (wire (pts (xy 148.59 66.675) (xy 156.845 66.675))
     (stroke (width 0) (type default))
   )
@@
     (stroke (width 0) (type default))
   )
+  (wire (pts (xy 156.845 66.675) (xy 164.465 66.675))
+    (stroke (width 0) (type default))
+  )
   (wire (pts (xy 205.105 95.885) (xy 205.105 98.425))
     (stroke (width 0) (type default))
@@
   )
   (wire (pts (xy 131.445 57.785) (xy 131.445 64.135))
+    (stroke (width 0) (type default))
+  )
+  (wire (pts (xy 156.845 59.69) (xy 156.845 66.675))
     (stroke (width 0) (type default))
   )
@@
     (effects (font (size 1.27 1.27)) (justify right bottom))
   )
-  (label "T" (at 156.21 66.675 0) (fields_autoplaced)
+  (label "T" (at 164.465 66.675 0) (fields_autoplaced)
     (effects (font (size 1.27 1.27)) (justify left bottom))
   )
-  (hierarchical_label "5V0" (shape input) (at 30.48 67.31 90) (fields_autoplaced)
+  (hierarchical_label "AOUT_HP" (shape output) (at 164.465 59.69 0) (fields_autoplaced)
     (effects (font (size 1.27 1.27)) (justify left))
   )
@@
         )
       )
+    )
+  )
+  (symbol (lib_id "power:+5V") (at 30.48 67.31 0) (unit 1)
+    (in_bom yes) (on_board yes) (dnp no) (fields_autoplaced)
+    (property "Reference" "#PWR080" (at 30.48 71.12 0)
+      (effects (font (size 1.27 1.27)) hide)
+    )
+    (property "Value" "+5V" (at 30.48 62.865 0)
+      (effects (font (size 1.27 1.27)))
+    )
+    (property "Footprint" "" (at 30.48 67.31 0)
+      (effects (font (size 1.27 1.27)) hide)
+    )
+    (property "Datasheet" "" (at 30.48 67.31 0)
+      (effects (font (size 1.27 1.27)) hide)
+    )
+    (pin "1")
+    (instances
+      (project "bt_pcb"
+        (path "/eb787481-08cd-41a4-a128-173fa6227c32/4ada0139-8712-47ce-9d4c-ab8fef312f7b/60bf59a0-253f-4ea1-81da-7746e9b04190"
+          (reference "#PWR080") (unit 1)
+        )
+      )

Commit message: progress on hp
Connections:
- net AOUT_HP renamed T
Changed lines of the file:
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@@
   (junction (at 156.21 81.28) (diameter 0) (color 0 0 0 0)
-  )
-  (junction (at 156.845 66.675) (diameter 0) (color 0 0 0 0)
   )
   (junction (at 227.33 68.58) (diameter 0) (color 0 0 0 0)
@@
     (stroke (width 0) (type default))
   )
-  (wire (pts (xy 164.465 59.69) (xy 156.845 59.69))
-    (stroke (width 0) (type default))
-  )
   (wire (pts (xy 93.98 49.53) (xy 93.98 57.785))
     (stroke (width 0) (type default))
@@
     (stroke (width 0) (type default))
   )
-  (wire (pts (xy 148.59 66.675) (xy 156.845 66.675))
-    (stroke (width 0) (type default))
-  )
   (wire (pts (xy 227.33 53.34) (xy 227.33 55.245))
     (stroke (width 0) (type default))
@@
     (stroke (width 0) (type default))
   )
-  (wire (pts (xy 156.845 66.675) (xy 164.465 66.675))
+  (wire (pts (xy 148.59 66.675) (xy 164.465 66.675))
     (stroke (width 0) (type default))
   )
@@
   )
   (wire (pts (xy 131.445 57.785) (xy 131.445 64.135))
-    (stroke (width 0) (type default))
-  )
-  (wire (pts (xy 156.845 59.69) (xy 156.845 66.675))
     (stroke (width 0) (type default))
   )
@@
     (effects (font (size 1.27 1.27)) (justify left bottom))
   )
-  (hierarchical_label "AOUT_HP" (shape output) (at 164.465 59.69 0) (fields_autoplaced)
-    (effects (font (size 1.27 1.27)) (justify left))
-  )
   (hierarchical_label "VCOM" (shape input) (at 159.385 81.28 0) (fields_autoplaced)
