File: pcb/output_b.kicad_sch (KiCad schematic)
At the start: 17 parts, among them J11 XLR3_Ground, J8 AudioJack2_Dual_Switch, U5 MCP6004

Commit message: making up my mind on the heaphones
Connections:
- net 5V0 renamed +5V
- net T renamed BOUT_HP
Changed lines of the file:
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@@
   (junction (at 101.6 85.725) (diameter 0) (color 0 0 0 0)
   )
+  (junction (at 156.21 76.835) (diameter 0) (color 0 0 0 0)
+  )
   (junction (at 234.95 65.405) (diameter 0) (color 0 0 0 0)
   )
@@
   (junction (at 234.95 52.07) (diameter 0) (color 0 0 0 0)
   )
-  (junction (at 156.21 76.835) (diameter 0) (color 0 0 0 0)
-  )
   (junction (at 252.095 59.69) (diameter 0) (color 0 0 0 0)
   )
@@
   )
   (junction (at 101.6 67.945) (diameter 0) (color 0 0 0 0)
+  )
+  (junction (at 164.465 76.835) (diameter 0) (color 0 0 0 0)
   )
   (junction (at 118.745 85.725) (diameter 0) (color 0 0 0 0)
@@
     (stroke (width 0) (type default))
   )
-  (wire (pts (xy 156.21 76.835) (xy 163.83 76.835))
-    (stroke (width 0) (type default))
-  )
   (wire (pts (xy 212.725 116.205) (xy 204.47 116.205))
     (stroke (width 0) (type default))
@@
     (stroke (width 0) (type default))
   )
+  (wire (pts (xy 164.465 69.85) (xy 164.465 76.835))
+    (stroke (width 0) (type default))
+  )
   (wire (pts (xy 156.21 62.23) (xy 156.21 76.835))
     (stroke (width 0) (type default))
@@
     (stroke (width 0) (type default))
   )
+  (wire (pts (xy 164.465 76.835) (xy 172.085 76.835))
+    (stroke (width 0) (type default))
+  )
   (wire (pts (xy 234.95 65.405) (xy 234.95 67.31))
     (stroke (width 0) (type default))
@@
     (stroke (width 0) (type default))
   )
+  (wire (pts (xy 156.21 76.835) (xy 164.465 76.835))
+    (stroke (width 0) (type default))
+  )
   (wire (pts (xy 217.17 78.74) (xy 224.155 78.74))
     (stroke (width 0) (type default))
@@
   )
   (wire (pts (xy 244.475 78.74) (xy 244.475 59.69))
+    (stroke (width 0) (type default))
+  )
+  (wire (pts (xy 172.085 69.85) (xy 164.465 69.85))
     (stroke (width 0) (type default))
   )
@@
     (effects (font (size 1.27 1.27)) (justify left bottom))
   )
+  (label "T" (at 172.085 76.835 0) (fields_autoplaced)
+    (effects (font (size 1.27 1.27)) (justify left bottom))
+  )
   (label "T" (at 189.865 116.205 180) (fields_autoplaced)
     (effects (font (size 1.27 1.27)) (justify right bottom))
   )
-  (label "T" (at 163.83 76.835 0) (fields_autoplaced)
-    (effects (font (size 1.27 1.27)) (justify left bottom))
-  )
-  (hierarchical_label "5V0" (shape input) (at 38.1 77.47 90) (fields_autoplaced)
-    (effects (font (size 1.27 1.27)) (justify left))
-  )
   (hierarchical_label "BOUT+" (shape input) (at 90.17 54.61 180) (fields_autoplaced)
     (effects (font (size 1.27 1.27)) (justify right))
   )
   (hierarchical_label "VCOM" (shape input) (at 167.005 91.44 0) (fields_autoplaced)
+    (effects (font (size 1.27 1.27)) (justify left))
+  )
+  (hierarchical_label "BOUT_HP" (shape output) (at 172.085 69.85 0) (fields_autoplaced)
     (effects (font (size 1.27 1.27)) (justify left))
   )
@@
         )
       )
+    )
+  )
+  (symbol (lib_id "power:+5V") (at 38.1 77.47 0) (unit 1)
+    (in_bom yes) (on_board yes) (dnp no) (fields_autoplaced)
+    (property "Reference" "#PWR079" (at 38.1 81.28 0)
+      (effects (font (size 1.27 1.27)) hide)
+    )
+    (property "Value" "+5V" (at 38.1 73.025 0)
+      (effects (font (size 1.27 1.27)))
+    )
+    (property "Footprint" "" (at 38.1 77.47 0)
+      (effects (font (size 1.27 1.27)) hide)
+    )
+    (property "Datasheet" "" (at 38.1 77.47 0)
+      (effects (font (size 1.27 1.27)) hide)
+    )
+    (pin "1")
+    (instances
+      (project "bt_pcb"
+        (path "/eb787481-08cd-41a4-a128-173fa6227c32/4ada0139-8712-47ce-9d4c-ab8fef312f7b/fa59e647-d5eb-4f6f-a20b-bde1796e2368"
+          (reference "#PWR079") (unit 1)
+        )
+      )

Commit message: progress on hp
Connections:
- net BOUT_HP renamed T
Changed lines of the file:
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@@
   (junction (at 101.6 67.945) (diameter 0) (color 0 0 0 0)
-  )
-  (junction (at 164.465 76.835) (diameter 0) (color 0 0 0 0)
   )
   (junction (at 118.745 85.725) (diameter 0) (color 0 0 0 0)
@@
     (stroke (width 0) (type default))
   )
-  (wire (pts (xy 164.465 69.85) (xy 164.465 76.835))
-    (stroke (width 0) (type default))
-  )
   (wire (pts (xy 156.21 62.23) (xy 156.21 76.835))
     (stroke (width 0) (type default))
@@
     (stroke (width 0) (type default))
   )
-  (wire (pts (xy 164.465 76.835) (xy 172.085 76.835))
+  (wire (pts (xy 156.21 76.835) (xy 172.085 76.835))
     (stroke (width 0) (type default))
   )
@@
     (stroke (width 0) (type default))
   )
-  (wire (pts (xy 156.21 76.835) (xy 164.465 76.835))
-    (stroke (width 0) (type default))
-  )
   (wire (pts (xy 217.17 78.74) (xy 224.155 78.74))
     (stroke (width 0) (type default))
@@
   )
   (wire (pts (xy 244.475 78.74) (xy 244.475 59.69))
-    (stroke (width 0) (type default))
-  )
-  (wire (pts (xy 172.085 69.85) (xy 164.465 69.85))
     (stroke (width 0) (type default))
   )
@@
     (effects (font (size 1.27 1.27)) (justify left))
   )
-  (hierarchical_label "BOUT_HP" (shape output) (at 172.085 69.85 0) (fields_autoplaced)
-    (effects (font (size 1.27 1.27)) (justify left))
-  )
