File: pcb/power_supply.kicad_sch (KiCad schematic)
At the start: 16 parts, among them IC1 TLV76150DCYR, IC2 LM3940IMP-3.3_NOPB, J1 Jack-DC

Commit message: starting the revision from ed
Parts:
- removed IC1: TLV76150DCYR, SOT230P700X180-4N, symbol SamacSys_Parts:TLV76150DCYR
- removed IC2: LM3940IMP-3.3_NOPB, SOT230P700X180-4N, symbol SamacSys_Parts:LM3940IMP-3.3_NOPB
- added C103: 10uF, symbol Device:C
- added C34, C68: 1uF, symbol Device:C
- added IC12: ADPL16000BATA+, ADPL16000BATA, symbol library:ADPL16000BATA+
- added IC13: LM3940IMP-3.3_NOPB, SOT230P700X180-4N, symbol library:LM3940IMP-3.3_NOPB
- added IC14: TLV76150DCYR, SOT230P700X180-4N, symbol library:TLV76150DCYR
- added L1: 68uH, symbol Device:L
- added R72: R, symbol Device:R
Connections:
- net +3V3: now also IC13.3 (OUT)
- net +5V: now also IC13.1 (IN), IC14.2 (OUT_1), IC14.4 (OUT_2)
- net GND: now also C103.2, C34.2, C68.1, IC12.7 (GND), IC13.2 (GND_1), IC13.4 (GND_2), IC14.1 (GND)
- net at C2.1, D1.1 (K), J1.1: now also IC14.3 (IN)
- new net: IC12.8 (LX), L1.1
- new net: C68.2, IC12.4 (FB/VOUT), L1.2
- new net: C103.1, IC12.3 (VCC), R72.1
- new net: C34.1, IC12.1 (VIN), IC12.2 (EN/UVLO)
- new net: IC12.6 (~{RESET}), R72.2
- no-connect marks 0 -> 1
Other:
- moved on the sheet: C1

Commit message: progress
Parts:
- added D4: D_Schottky, symbol Device:D_Schottky
- IC12: footprint ADPL16000BATA -> library:ADPL16000BATA
- IC13, IC14: footprint SOT230P700X180-4N -> library:SOT230P700X180-4N
Connections:
- net +5V: now also D4.1 (K)
- new net VBUS: D4.2 (A)
Changed lines of the file:
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@@
     (stroke (width 0) (type default))
   )
-  (wire (pts (xy 69.85 93.345) (xy 80.01 93.345))
+  (wire (pts (xy 60.96 93.345) (xy 65.405 93.345))
     (stroke (width 0) (type default))
   )
@@
     (stroke (width 0) (type default))
   )
+  (wire (pts (xy 73.025 93.345) (xy 80.01 93.345))
+    (stroke (width 0) (type default))
+  )
   (wire (pts (xy 102.235 55.88) (xy 102.235 66.675))
     (stroke (width 0) (type default))
@@
     (stroke (width 0) (type default))
   )
-  (global_label "VBUS" (shape input) (at 69.85 93.345 180) (fields_autoplaced)
+  (global_label "VBUS" (shape input) (at 60.96 93.345 180) (fields_autoplaced)
     (effects (font (size 1.27 1.27)) (justify right))
-    (property "Intersheetrefs" "${INTERSHEET_REFS}" (at 61.9662 93.345 0)
+    (property "Intersheetrefs" "${INTERSHEET_REFS}" (at 53.0762 93.345 0)
       (effects (font (size 1.27 1.27)) (justify right) hide)
     )
@@
       (effects (font (size 1.27 1.27)) hide)
     )
-    (pin "2")
-    (pin "1")
+    (pin "1")
+    (pin "2")
     (instances
       (project "bt_pcb"
@@
       (effects (font (size 1.27 1.27)))
     )
-    (property "Footprint" "SOT230P700X180-4N" (at 231.775 186.36 0)
+    (property "Footprint" "library:SOT230P700X180-4N" (at 231.775 186.36 0)
       (effects (font (size 1.27 1.27)) (justify left top) hide)
     )
@@
     )
     (pin "1")
+    (pin "2")
+    (pin "3")
     (pin "4")
-    (pin "2")
-    (pin "3")
     (instances
       (project "bt_pcb"
@@
     )
   )
+  (symbol (lib_id "Device:D_Schottky") (at 69.215 93.345 180) (unit 1)
+    (in_bom yes) (on_board yes) (dnp no)
+    (property "Reference" "D4" (at 68.2625 90.17 90)
+      (effects (font (size 1.27 1.27)) (justify right))
+    )
+    (property "Value" "D_Schottky" (at 70.8025 90.17 90)
+      (effects (font (size 1.27 1.27)) (justify right))
+    )
+    (property "Footprint" "" (at 69.215 93.345 0)
+      (effects (font (size 1.27 1.27)) hide)
+    )
+    (property "Datasheet" "~" (at 69.215 93.345 0)
+      (effects (font (size 1.27 1.27)) hide)
+    )
+    (pin "1")
+    (pin "2")
+    (instances
+      (project "bt_pcb"
+        (path "/eb787481-08cd-41a4-a128-173fa6227c32/4ec3bf5a-5f62-4a58-b8f9-e874725801fb"
+          (reference "D4") (unit 1)
+        )
+      )
+    )
+  )
   (symbol (lib_id "power:GND") (at 128.905 135.89 0) (unit 1)
     (in_bom yes) (on_board yes) (dnp no) (fields_autoplaced)
@@
       (effects (font (size 1.27 1.27)))
     )
-    (property "Footprint" "ADPL16000BATA" (at 100.965 230.81 0)
+    (property "Footprint" "library:ADPL16000BATA" (at 100.965 230.81 0)
       (effects (font (size 1.27 1.27)) (justify left top) hide)
     )
@@
       (effects (font (size 1.27 1.27)) (justify left top) hide)
     )
-    (pin "8")
+    (pin "1")
+    (pin "2")
     (pin "3")
-    (pin "2")
-    (pin "1")
+    (pin "4")
+    (pin "5")
     (pin "6")
     (pin "7")
-    (pin "5")
-    (pin "4")
+    (pin "8")
     (instances
       (project "bt_pcb"
@@
       (effects (font (size 1.27 1.27)) hide)
     )
-    (pin "2")
-    (pin "1")
+    (pin "1")
+    (pin "2")
     (instances
       (project "bt_pcb"
@@
       (effects (font (size 1.27 1.27)))
     )
-    (property "Footprint" "SOT230P700X180-4N" (at 128.905 -39.04 0)
+    (property "Footprint" "library:SOT230P700X180-4N" (at 128.905 -39.04 0)
       (effects (font (size 1.27 1.27)) (justify left top) hide)
     )
@@
       (effects (font (size 1.27 1.27)) (justify left top) hide)
     )
+    (pin "1")
+    (pin "2")
+    (pin "3")
     (pin "4")
-    (pin "2")
-    (pin "1")
-    (pin "3")
-    (instances
-      (project "bt_pcb"
+    (instances
+      (project "bt_pcb"
