File: pcb/audio_input.kicad_sch (KiCad schematic)
At the start: 52 parts, among them IC6 ADG736BRM, IC7 ADG736BRM, J7 AudioJack3_Switch, U6 MCP6004, U7 MCP6004

Commit message: minor
Parts:
- renumbered J7 to J5, J7 to J8
Changed lines of the file:
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@@
   (symbol (lib_id "Connector_Audio:AudioJack3_Switch") (at 30.48 99.695 0) (mirror x) (unit 1)
     (in_bom yes) (on_board yes) (dnp no)
-    (property "Reference" "J7" (at 28.575 111.125 0)
+    (property "Reference" "J8" (at 28.575 111.125 0)
       (effects (font (size 1.27 1.27)))
     )
@@
     (instances
       (project "bt_pcb"
-        (path "/eb787481-08cd-41a4-a128-173fa6227c32/4ada0139-8712-47ce-9d4c-ab8fef312f7b/92a88d42-e0ca-481e-a77e-2117fd7dfc0f"
-          (reference "J7") (unit 1)
-        )
         (path "/eb787481-08cd-41a4-a128-173fa6227c32/4ada0139-8712-47ce-9d4c-ab8fef312f7b/aa7abd67-f1bd-4ae8-bc05-bae360f4c6c7"
           (reference "J8") (unit 1)
@@
   (symbol (lib_id "Connector_Audio:AudioJack3_Switch") (at 31.115 26.67 0) (mirror x) (unit 1)
     (in_bom yes) (on_board yes) (dnp no)
-    (property "Reference" "J7" (at 29.21 38.1 0)
+    (property "Reference" "J5" (at 29.21 38.1 0)
       (effects (font (size 1.27 1.27)))
     )
@@
     (instances
       (project "bt_pcb"
-        (path "/eb787481-08cd-41a4-a128-173fa6227c32/4ada0139-8712-47ce-9d4c-ab8fef312f7b/92a88d42-e0ca-481e-a77e-2117fd7dfc0f"
-          (reference "J7") (unit 1)
-        )
         (path "/eb787481-08cd-41a4-a128-173fa6227c32/4ada0139-8712-47ce-9d4c-ab8fef312f7b/aa7abd67-f1bd-4ae8-bc05-bae360f4c6c7"
           (reference "J5") (unit 1)

Commit message: a lot of work! almost ready for rev
Connections:
- net INA+ renamed CODEC_INA+
- net INA- renamed CODEC_INA-
- net INA_SWITCH renamed INA_SELECT
- net INB+ renamed CODEC_INB+
- net INB- renamed CODEC_INB-
- net INB_SWITCH renamed INB_SELECT
Other:
- moved on the sheet: C102, C89

Commit message: starting the revision from ed
Parts:
- removed IC6, IC7: ADG736BRM, SOP50P490X110-10N, symbol SamacSys:ADG736BRM
- added IC6, IC7: ADG736BRM, SOP50P490X110-10N, symbol library:ADG736BRM
- C80: value 10uF -> 470uF
Connections:
- net +5V: now also IC6.8 (VDD), IC7.8 (VDD)
- net CODEC_INA+: now also IC6.10 (D1)
- net CODEC_INA-: now also IC6.6 (D2)
- net CODEC_INB+: now also IC7.10 (D1)
- net CODEC_INB-: now also IC7.6 (D2)
- net GND: now also IC6.3 (GND), IC7.3 (GND)
- net INA+_DIFF: now also IC6.2 (S1A)
- net INA+_SE: now also IC6.9 (S1B)
- net INA-_DIFF: now also IC6.4 (S2A)
- net INA-_SE: now also IC6.7 (S2B)
- net INA_SELECT: now also IC6.1 (IN1), IC6.5 (IN2)
- net INB+_DIFF: now also IC7.2 (S1A)
- net INB+_SE: now also IC7.9 (S1B)
- net INB-_DIFF: now also IC7.4 (S2A)
- net INB-_SE: now also IC7.7 (S2B)
- net INB_SELECT: now also IC7.1 (IN1), IC7.5 (IN2)
Changed lines of the file:
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@@
     )
   )
-  (symbol (lib_id "SamacSys:ADG736BRM") (at 41.275 168.91 0) (unit 1)
+  (symbol (lib_id "library:ADG736BRM") (at 41.275 168.91 0) (unit 1)
     (in_bom yes) (on_board yes) (dnp no) (fields_autoplaced)
     (property "Reference" "IC6" (at 53.975 161.29 0)
@@
       (effects (font (size 1.27 1.27)) (justify left top) hide)
     )
-    (pin "1")
-    (pin "10")
     (pin "2")
     (pin "3")
     (pin "4")
+    (pin "1")
+    (pin "10")
+    (pin "6")
+    (pin "9")
+    (pin "8")
     (pin "5")
-    (pin "6")
     (pin "7")
-    (pin "8")
-    (pin "9")
     (instances
       (project "bt_pcb"
@@
         (path "/eb787481-08cd-41a4-a128-173fa6227c32/4ada0139-8712-47ce-9d4c-ab8fef312f7b/aa7abd67-f1bd-4ae8-bc05-bae360f4c6c7"
           (reference "R51") (unit 1)
-        )
-      )
-    )
-  )
-  (symbol (lib_id "SamacSys:ADG736BRM") (at 120.015 168.91 0) (unit 1)
-    (in_bom yes) (on_board yes) (dnp no) (fields_autoplaced)
-    (property "Reference" "IC7" (at 132.715 161.29 0)
-      (effects (font (size 1.27 1.27)))
-    )
-    (property "Value" "ADG736BRM" (at 132.715 163.83 0)
-      (effects (font (size 1.27 1.27)))
-    )
-    (property "Footprint" "SOP50P490X110-10N" (at 141.605 263.83 0)
-      (effects (font (size 1.27 1.27)) (justify left top) hide)
-    )
-    (property "Datasheet" "https://www.arrow.com/en/products/adg736brm/analog-devices?region=nac" (at 141.605 363.83 0)
-      (effects (font (size 1.27 1.27)) (justify left top) hide)
-    )
-    (property "Height" "1.1" (at 141.605 563.83 0)
-      (effects (font (size 1.27 1.27)) (justify left top) hide)
-    )
-    (property "Manufacturer_Name" "Analog Devices" (at 141.605 663.83 0)
-      (effects (font (size 1.27 1.27)) (justify left top) hide)
-    )
-    (property "Manufacturer_Part_Number" "ADG736BRM" (at 141.605 763.83 0)
-      (effects (font (size 1.27 1.27)) (justify left top) hide)
-    )
-    (property "Mouser Part Number" "" (at 141.605 863.83 0)
-      (effects (font (size 1.27 1.27)) (justify left top) hide)
-    )
-    (property "Mouser Price/Stock" "" (at 141.605 963.83 0)
-      (effects (font (size 1.27 1.27)) (justify left top) hide)
-    )
-    (property "Arrow Part Number" "ADG736BRM" (at 141.605 1063.83 0)
-      (effects (font (size 1.27 1.27)) (justify left top) hide)
-    )
-    (property "Arrow Price/Stock" "https://www.arrow.com/en/products/adg736brm/analog-devices?region=nac" (at 141.605 1163.83 0)
-      (effects (font (size 1.27 1.27)) (justify left top) hide)
-    )
-    (pin "1")
-    (pin "10")
-    (pin "2")
-    (pin "3")
-    (pin "4")
-    (pin "5")
-    (pin "6")
-    (pin "7")
-    (pin "8")
-    (pin "9")
-    (instances
-      (project "bt_pcb"
-        (path "/eb787481-08cd-41a4-a128-173fa6227c32/4ada0139-8712-47ce-9d4c-ab8fef312f7b/aa7abd67-f1bd-4ae8-bc05-bae360f4c6c7"
-          (reference "IC7") (unit 1)
         )
       )
@@
       (effects (font (size 1.27 1.27)))
     )
-    (property "Value" "10uF" (at 68.199 33.02 90)
+    (property "Value" "470uF" (at 68.199 33.02 90)
       (effects (font (size 1.27 1.27)))
     )
@@
         )
       )
+    )
+  )
+  (symbol (lib_id "library:ADG736BRM") (at 120.015 168.91 0) (unit 1)
+    (in_bom yes) (on_board yes) (dnp no) (fields_autoplaced)
+    (property "Reference" "IC7" (at 132.715 161.29 0)
+      (effects (font (size 1.27 1.27)))
+    )
+    (property "Value" "ADG736BRM" (at 132.715 163.83 0)
+      (effects (font (size 1.27 1.27)))
+    )
+    (property "Footprint" "SOP50P490X110-10N" (at 141.605 263.83 0)
+      (effects (font (size 1.27 1.27)) (justify left top) hide)
+    )
+    (property "Datasheet" "https://www.arrow.com/en/products/adg736brm/analog-devices?region=nac" (at 141.605 363.83 0)
+      (effects (font (size 1.27 1.27)) (justify left top) hide)
+    )
+    (property "Height" "1.1" (at 141.605 563.83 0)
+      (effects (font (size 1.27 1.27)) (justify left top) hide)
+    )
+    (property "Manufacturer_Name" "Analog Devices" (at 141.605 663.83 0)
+      (effects (font (size 1.27 1.27)) (justify left top) hide)
+    )
+    (property "Manufacturer_Part_Number" "ADG736BRM" (at 141.605 763.83 0)
+      (effects (font (size 1.27 1.27)) (justify left top) hide)
+    )
+    (property "Mouser Part Number" "" (at 141.605 863.83 0)
+      (effects (font (size 1.27 1.27)) (justify left top) hide)
+    )
+    (property "Mouser Price/Stock" "" (at 141.605 963.83 0)
+      (effects (font (size 1.27 1.27)) (justify left top) hide)
+    )
+    (property "Arrow Part Number" "ADG736BRM" (at 141.605 1063.83 0)
+      (effects (font (size 1.27 1.27)) (justify left top) hide)
+    )
+    (property "Arrow Price/Stock" "https://www.arrow.com/en/products/adg736brm/analog-devices?region=nac" (at 141.605 1163.83 0)
+      (effects (font (size 1.27 1.27)) (justify left top) hide)
+    )
+    (pin "2")
+    (pin "3")
+    (pin "4")
+    (pin "1")
+    (pin "10")
+    (pin "6")
+    (pin "9")
+    (pin "8")
+    (pin "5")
+    (pin "7")
+    (instances
+      (project "bt_pcb"
+        (path "/eb787481-08cd-41a4-a128-173fa6227c32/4ada0139-8712-47ce-9d4c-ab8fef312f7b/aa7abd67-f1bd-4ae8-bc05-bae360f4c6c7"
+          (reference "IC7") (unit 1)
+        )
+      )

Commit message: progress
Parts:
- IC6, IC7: footprint SOP50P490X110-10N -> library:SOP50P490X110-10N
Changed lines of the file:
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@@
       (effects (font (size 1.27 1.27)))
     )
-    (property "Footprint" "SOP50P490X110-10N" (at 62.865 263.83 0)
+    (property "Footprint" "library:SOP50P490X110-10N" (at 62.865 263.83 0)
       (effects (font (size 1.27 1.27)) (justify left top) hide)
     )
@@
       (effects (font (size 1.27 1.27)) (justify left top) hide)
     )
+    (pin "1")
+    (pin "10")
     (pin "2")
     (pin "3")
     (pin "4")
-    (pin "1")
-    (pin "10")
+    (pin "5")
     (pin "6")
+    (pin "7")
+    (pin "8")
     (pin "9")
-    (pin "8")
-    (pin "5")
-    (pin "7")
     (instances
       (project "bt_pcb"
@@
       (effects (font (size 1.27 1.27)))
     )
-    (property "Footprint" "SOP50P490X110-10N" (at 141.605 263.83 0)
+    (property "Footprint" "library:SOP50P490X110-10N" (at 141.605 263.83 0)
       (effects (font (size 1.27 1.27)) (justify left top) hide)
     )
@@
       (effects (font (size 1.27 1.27)) (justify left top) hide)
     )
+    (pin "1")
+    (pin "10")
     (pin "2")
     (pin "3")
     (pin "4")
-    (pin "1")
-    (pin "10")
+    (pin "5")
     (pin "6")
+    (pin "7")
+    (pin "8")
     (pin "9")
-    (pin "8")
-    (pin "5")
-    (pin "7")
-    (instances
-      (project "bt_pcb"
+    (instances
+      (project "bt_pcb"
