File: pcb/audio_output.kicad_sch (KiCad schematic)
At the start: 34 parts, among them IC6 ADG736BRM, J3 AudioJack3_Switch, J7 AudioJack3_Switch, U2 MCP6004, U4 MCP6004

Commit message: minor
Parts:
- renumbered C89 to C36, C89 to C39, IC6 to IC8, IC6 to IC9
Changed lines of the file:
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@@
   (symbol (lib_id "power:GND") (at 255.27 123.825 0) (mirror y) (unit 1)
     (in_bom yes) (on_board yes) (dnp no) (fields_autoplaced)
-    (property "Reference" "#PWR0103" (at 255.27 130.175 0)
+    (property "Reference" "#PWR0114" (at 255.27 130.175 0)
       (effects (font (size 1.27 1.27)) hide)
     )
@@
     (instances
       (project "bt_pcb"
-        (path "/eb787481-08cd-41a4-a128-173fa6227c32/4ada0139-8712-47ce-9d4c-ab8fef312f7b/aa7abd67-f1bd-4ae8-bc05-bae360f4c6c7"
-          (reference "#PWR0103") (unit 1)
-        )
         (path "/eb787481-08cd-41a4-a128-173fa6227c32/4ada0139-8712-47ce-9d4c-ab8fef312f7b/92a88d42-e0ca-481e-a77e-2117fd7dfc0f"
           (reference "#PWR0114") (unit 1)
@@
   (symbol (lib_id "power:GND") (at 200.66 46.355 0) (unit 1)
     (in_bom yes) (on_board yes) (dnp no) (fields_autoplaced)
-    (property "Reference" "#PWR0102" (at 200.66 52.705 0)
+    (property "Reference" "#PWR042" (at 200.66 52.705 0)
       (effects (font (size 1.27 1.27)) hide)
     )
@@
     (instances
       (project "bt_pcb"
-        (path "/eb787481-08cd-41a4-a128-173fa6227c32/4ada0139-8712-47ce-9d4c-ab8fef312f7b/aa7abd67-f1bd-4ae8-bc05-bae360f4c6c7"
-          (reference "#PWR0102") (unit 1)
-        )
         (path "/eb787481-08cd-41a4-a128-173fa6227c32/4ada0139-8712-47ce-9d4c-ab8fef312f7b/92a88d42-e0ca-481e-a77e-2117fd7dfc0f"
           (reference "#PWR042") (unit 1)
@@
   (symbol (lib_id "power:+5V") (at 200.66 105.41 0) (unit 1)
     (in_bom yes) (on_board yes) (dnp no)
-    (property "Reference" "#PWR098" (at 200.66 109.22 0)
+    (property "Reference" "#PWR077" (at 200.66 109.22 0)
       (effects (font (size 1.27 1.27)) hide)
     )
@@
     (instances
       (project "bt_pcb"
-        (path "/eb787481-08cd-41a4-a128-173fa6227c32/4ada0139-8712-47ce-9d4c-ab8fef312f7b/aa7abd67-f1bd-4ae8-bc05-bae360f4c6c7"
-          (reference "#PWR098") (unit 1)
-        )
         (path "/eb787481-08cd-41a4-a128-173fa6227c32/4ada0139-8712-47ce-9d4c-ab8fef312f7b/92a88d42-e0ca-481e-a77e-2117fd7dfc0f"
           (reference "#PWR077") (unit 1)
@@
   (symbol (lib_id "power:+5V") (at 200.66 33.655 0) (unit 1)
     (in_bom yes) (on_board yes) (dnp no)
-    (property "Reference" "#PWR098" (at 200.66 37.465 0)
+    (property "Reference" "#PWR041" (at 200.66 37.465 0)
       (effects (font (size 1.27 1.27)) hide)
     )
@@
     (instances
       (project "bt_pcb"
-        (path "/eb787481-08cd-41a4-a128-173fa6227c32/4ada0139-8712-47ce-9d4c-ab8fef312f7b/aa7abd67-f1bd-4ae8-bc05-bae360f4c6c7"
-          (reference "#PWR098") (unit 1)
-        )
         (path "/eb787481-08cd-41a4-a128-173fa6227c32/4ada0139-8712-47ce-9d4c-ab8fef312f7b/92a88d42-e0ca-481e-a77e-2117fd7dfc0f"
           (reference "#PWR041") (unit 1)
@@
   (symbol (lib_id "power:GND") (at 133.35 45.085 0) (unit 1)
     (in_bom yes) (on_board yes) (dnp no) (fields_autoplaced)
-    (property "Reference" "#PWR093" (at 133.35 51.435 0)
+    (property "Reference" "#PWR040" (at 133.35 51.435 0)
       (effects (font (size 1.27 1.27)) hide)
     )
@@
     (instances
       (project "bt_pcb"
-        (path "/eb787481-08cd-41a4-a128-173fa6227c32/4ada0139-8712-47ce-9d4c-ab8fef312f7b/aa7abd67-f1bd-4ae8-bc05-bae360f4c6c7"
-          (reference "#PWR093") (unit 1)
-        )
         (path "/eb787481-08cd-41a4-a128-173fa6227c32/4ada0139-8712-47ce-9d4c-ab8fef312f7b/92a88d42-e0ca-481e-a77e-2117fd7dfc0f"
           (reference "#PWR040") (unit 1)
@@
   (symbol (lib_id "Device:C") (at 200.66 114.3 0) (unit 1)
     (in_bom yes) (on_board yes) (dnp no) (fields_autoplaced)
-    (property "Reference" "C89" (at 203.835 113.03 0)
+    (property "Reference" "C39" (at 203.835 113.03 0)
       (effects (font (size 1.27 1.27)) (justify left))
     )
@@
     (instances
       (project "bt_pcb"
-        (path "/eb787481-08cd-41a4-a128-173fa6227c32/4ada0139-8712-47ce-9d4c-ab8fef312f7b/aa7abd67-f1bd-4ae8-bc05-bae360f4c6c7"
-          (reference "C89") (unit 1)
-        )
         (path "/eb787481-08cd-41a4-a128-173fa6227c32/4ada0139-8712-47ce-9d4c-ab8fef312f7b/92a88d42-e0ca-481e-a77e-2117fd7dfc0f"
           (reference "C39") (unit 1)
@@
   (symbol (lib_id "SamacSys:ADG736BRM") (at 147.955 106.68 0) (unit 1)
     (in_bom yes) (on_board yes) (dnp no) (fields_autoplaced)
-    (property "Reference" "IC6" (at 160.655 99.06 0)
+    (property "Reference" "IC9" (at 160.655 99.06 0)
       (effects (font (size 1.27 1.27)))
     )
@@
     (instances
       (project "bt_pcb"
-        (path "/eb787481-08cd-41a4-a128-173fa6227c32/4ada0139-8712-47ce-9d4c-ab8fef312f7b/aa7abd67-f1bd-4ae8-bc05-bae360f4c6c7"
-          (reference "IC6") (unit 1)
-        )
         (path "/eb787481-08cd-41a4-a128-173fa6227c32/4ada0139-8712-47ce-9d4c-ab8fef312f7b/92a88d42-e0ca-481e-a77e-2117fd7dfc0f"
           (reference "IC9") (unit 1)
@@
   (symbol (lib_id "Device:C") (at 200.66 42.545 0) (unit 1)
     (in_bom yes) (on_board yes) (dnp no) (fields_autoplaced)
-    (property "Reference" "C89" (at 203.835 41.275 0)
+    (property "Reference" "C36" (at 203.835 41.275 0)
       (effects (font (size 1.27 1.27)) (justify left))
     )
@@
     (instances
       (project "bt_pcb"
-        (path "/eb787481-08cd-41a4-a128-173fa6227c32/4ada0139-8712-47ce-9d4c-ab8fef312f7b/aa7abd67-f1bd-4ae8-bc05-bae360f4c6c7"
-          (reference "C89") (unit 1)
-        )
         (path "/eb787481-08cd-41a4-a128-173fa6227c32/4ada0139-8712-47ce-9d4c-ab8fef312f7b/92a88d42-e0ca-481e-a77e-2117fd7dfc0f"
           (reference "C36") (unit 1)
@@
   (symbol (lib_id "power:GND") (at 133.35 116.84 0) (unit 1)
     (in_bom yes) (on_board yes) (dnp no) (fields_autoplaced)
-    (property "Reference" "#PWR093" (at 133.35 123.19 0)
+    (property "Reference" "#PWR049" (at 133.35 123.19 0)
       (effects (font (size 1.27 1.27)) hide)
     )
@@
     (instances
       (project "bt_pcb"
-        (path "/eb787481-08cd-41a4-a128-173fa6227c32/4ada0139-8712-47ce-9d4c-ab8fef312f7b/aa7abd67-f1bd-4ae8-bc05-bae360f4c6c7"
-          (reference "#PWR093") (unit 1)
-        )
         (path "/eb787481-08cd-41a4-a128-173fa6227c32/4ada0139-8712-47ce-9d4c-ab8fef312f7b/92a88d42-e0ca-481e-a77e-2117fd7dfc0f"
           (reference "#PWR049") (unit 1)
@@
   (symbol (lib_id "power:GND") (at 200.66 118.11 0) (unit 1)
     (in_bom yes) (on_board yes) (dnp no) (fields_autoplaced)
-    (property "Reference" "#PWR0102" (at 200.66 124.46 0)
+    (property "Reference" "#PWR0112" (at 200.66 124.46 0)
       (effects (font (size 1.27 1.27)) hide)
     )
@@
     (instances
       (project "bt_pcb"
-        (path "/eb787481-08cd-41a4-a128-173fa6227c32/4ada0139-8712-47ce-9d4c-ab8fef312f7b/aa7abd67-f1bd-4ae8-bc05-bae360f4c6c7"
-          (reference "#PWR0102") (unit 1)
-        )
         (path "/eb787481-08cd-41a4-a128-173fa6227c32/4ada0139-8712-47ce-9d4c-ab8fef312f7b/92a88d42-e0ca-481e-a77e-2117fd7dfc0f"
           (reference "#PWR0112") (unit 1)
@@
   (symbol (lib_id "SamacSys:ADG736BRM") (at 147.955 34.925 0) (unit 1)
     (in_bom yes) (on_board yes) (dnp no) (fields_autoplaced)
-    (property "Reference" "IC6" (at 160.655 27.305 0)
+    (property "Reference" "IC8" (at 160.655 27.305 0)
       (effects (font (size 1.27 1.27)))
     )
@@
     (instances
       (project "bt_pcb"
-        (path "/eb787481-08cd-41a4-a128-173fa6227c32/4ada0139-8712-47ce-9d4c-ab8fef312f7b/aa7abd67-f1bd-4ae8-bc05-bae360f4c6c7"
-          (reference "IC6") (unit 1)
-        )
         (path "/eb787481-08cd-41a4-a128-173fa6227c32/4ada0139-8712-47ce-9d4c-ab8fef312f7b/92a88d42-e0ca-481e-a77e-2117fd7dfc0f"
           (reference "IC8") (unit 1)
@@
   (symbol (lib_id "power:GND") (at 255.27 52.07 0) (mirror y) (unit 1)
     (in_bom yes) (on_board yes) (dnp no) (fields_autoplaced)
-    (property "Reference" "#PWR0103" (at 255.27 58.42 0)
+    (property "Reference" "#PWR039" (at 255.27 58.42 0)
       (effects (font (size 1.27 1.27)) hide)
     )
@@
     (instances
       (project "bt_pcb"
-        (path "/eb787481-08cd-41a4-a128-173fa6227c32/4ada0139-8712-47ce-9d4c-ab8fef312f7b/aa7abd67-f1bd-4ae8-bc05-bae360f4c6c7"
-          (reference "#PWR0103") (unit 1)
-        )
         (path "/eb787481-08cd-41a4-a128-173fa6227c32/4ada0139-8712-47ce-9d4c-ab8fef312f7b/92a88d42-e0ca-481e-a77e-2117fd7dfc0f"
           (reference "#PWR039") (unit 1)

Commit message: a lot of work! almost ready for rev
Connections:
- net OUTA+ renamed CODEC_OUTA+
- net OUTA- renamed CODEC_OUTA-
- net OUTA_SWITCH renamed OUTA_SELECT
- net OUTB+ renamed CODEC_OUTB+
- net OUTB- renamed CODEC_OUTB-
- net OUTB_SWITCH renamed OUTB_SELECT
Other:
- moved on the sheet: C31, C33, C40, C41, J3, J7, R12, R13, R20, R21

Commit message: starting the revision from ed
Parts:
- removed IC8, IC9: ADG736BRM, SOP50P490X110-10N, symbol SamacSys:ADG736BRM
- added IC1, IC2: ADG736BRM, SOP50P490X110-10N, symbol library:ADG736BRM
Connections:
- net +5V: now also IC1.8 (VDD), IC2.8 (VDD)
- net GND: now also IC1.3 (GND), IC2.3 (GND)
- net OUTA+_DIFF: now also IC1.2 (S1A)
- net OUTA-_DIFF: now also IC1.4 (S2A)
- net OUTA_SE: now also IC1.9 (S1B)
- net OUTA_SELECT: now also IC1.1 (IN1), IC1.5 (IN2)
- net OUTB+_DIFF: now also IC2.2 (S1A)
- net OUTB-_DIFF: now also IC2.4 (S2A)
- net OUTB_SE: now also IC2.9 (S1B)
- net OUTB_SELECT: now also IC2.1 (IN1), IC2.5 (IN2)
- net RA: now also IC1.6 (D2)
- net RB: now also IC2.6 (D2)
- net TA: now also IC1.10 (D1)
- net TB: now also IC2.10 (D1)
- net VCOM: now also IC1.7 (S2B), IC2.7 (S2B)
Changed lines of the file:
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@@
+    )
+  )
+  (symbol (lib_id "library:ADG736BRM") (at 147.955 34.925 0) (unit 1)
+    (in_bom yes) (on_board yes) (dnp no) (fields_autoplaced)
+    (property "Reference" "IC1" (at 160.655 27.94 0)
+      (effects (font (size 1.27 1.27)))
+    )
+    (property "Value" "ADG736BRM" (at 160.655 30.48 0)
+      (effects (font (size 1.27 1.27)))
+    )
+    (property "Footprint" "SOP50P490X110-10N" (at 169.545 129.845 0)
+      (effects (font (size 1.27 1.27)) (justify left top) hide)
+    )
+    (property "Datasheet" "https://www.arrow.com/en/products/adg736brm/analog-devices?region=nac" (at 169.545 229.845 0)
+      (effects (font (size 1.27 1.27)) (justify left top) hide)
+    )
+    (property "Height" "1.1" (at 169.545 429.845 0)
+      (effects (font (size 1.27 1.27)) (justify left top) hide)
+    )
+    (property "Manufacturer_Name" "Analog Devices" (at 169.545 529.845 0)
+      (effects (font (size 1.27 1.27)) (justify left top) hide)
+    )
+    (property "Manufacturer_Part_Number" "ADG736BRM" (at 169.545 629.845 0)
+      (effects (font (size 1.27 1.27)) (justify left top) hide)
+    )
+    (property "Mouser Part Number" "" (at 169.545 729.845 0)
+      (effects (font (size 1.27 1.27)) (justify left top) hide)
+    )
+    (property "Mouser Price/Stock" "" (at 169.545 829.845 0)
+      (effects (font (size 1.27 1.27)) (justify left top) hide)
+    )
+    (property "Arrow Part Number" "ADG736BRM" (at 169.545 929.845 0)
+      (effects (font (size 1.27 1.27)) (justify left top) hide)
+    )
+    (property "Arrow Price/Stock" "https://www.arrow.com/en/products/adg736brm/analog-devices?region=nac" (at 169.545 1029.845 0)
+      (effects (font (size 1.27 1.27)) (justify left top) hide)
+    )
+    (pin "8")
+    (pin "2")
+    (pin "7")
+    (pin "10")
+    (pin "3")
+    (pin "6")
+    (pin "1")
+    (pin "5")
+    (pin "9")
+    (pin "4")
+    (instances
+      (project "bt_pcb"
+        (path "/eb787481-08cd-41a4-a128-173fa6227c32/4ada0139-8712-47ce-9d4c-ab8fef312f7b/92a88d42-e0ca-481e-a77e-2117fd7dfc0f"
+          (reference "IC1") (unit 1)
+        )
+      )
     )
   )
@@
     )
   )
+  (symbol (lib_id "library:ADG736BRM") (at 147.955 106.68 0) (unit 1)
+    (in_bom yes) (on_board yes) (dnp no) (fields_autoplaced)
+    (property "Reference" "IC2" (at 160.655 99.06 0)
+      (effects (font (size 1.27 1.27)))
+    )
+    (property "Value" "ADG736BRM" (at 160.655 101.6 0)
+      (effects (font (size 1.27 1.27)))
+    )
+    (property "Footprint" "SOP50P490X110-10N" (at 169.545 201.6 0)
+      (effects (font (size 1.27 1.27)) (justify left top) hide)
+    )
+    (property "Datasheet" "https://www.arrow.com/en/products/adg736brm/analog-devices?region=nac" (at 169.545 301.6 0)
+      (effects (font (size 1.27 1.27)) (justify left top) hide)
+    )
+    (property "Height" "1.1" (at 169.545 501.6 0)
+      (effects (font (size 1.27 1.27)) (justify left top) hide)
+    )
+    (property "Manufacturer_Name" "Analog Devices" (at 169.545 601.6 0)
+      (effects (font (size 1.27 1.27)) (justify left top) hide)
+    )
+    (property "Manufacturer_Part_Number" "ADG736BRM" (at 169.545 701.6 0)
+      (effects (font (size 1.27 1.27)) (justify left top) hide)
+    )
+    (property "Mouser Part Number" "" (at 169.545 801.6 0)
+      (effects (font (size 1.27 1.27)) (justify left top) hide)
+    )
+    (property "Mouser Price/Stock" "" (at 169.545 901.6 0)
+      (effects (font (size 1.27 1.27)) (justify left top) hide)
+    )
+    (property "Arrow Part Number" "ADG736BRM" (at 169.545 1001.6 0)
+      (effects (font (size 1.27 1.27)) (justify left top) hide)
+    )
+    (property "Arrow Price/Stock" "https://www.arrow.com/en/products/adg736brm/analog-devices?region=nac" (at 169.545 1101.6 0)
+      (effects (font (size 1.27 1.27)) (justify left top) hide)
+    )
+    (pin "2")
+    (pin "3")
+    (pin "4")
+    (pin "1")
+    (pin "10")
+    (pin "6")
+    (pin "9")
+    (pin "8")
+    (pin "5")
+    (pin "7")
+    (instances
+      (project "bt_pcb"
+        (path "/eb787481-08cd-41a4-a128-173fa6227c32/4ada0139-8712-47ce-9d4c-ab8fef312f7b/92a88d42-e0ca-481e-a77e-2117fd7dfc0f"
+          (reference "IC2") (unit 1)
+        )
+      )
+    )
+  )
   (symbol (lib_id "power:GND") (at 98.425 143.51 0) (unit 1)
     (in_bom yes) (on_board yes) (dnp no) (fields_autoplaced)
@@
     )
   )
-  (symbol (lib_id "SamacSys:ADG736BRM") (at 147.955 106.68 0) (unit 1)
-    (in_bom yes) (on_board yes) (dnp no) (fields_autoplaced)
-    (property "Reference" "IC9" (at 160.655 99.06 0)
-      (effects (font (size 1.27 1.27)))
-    )
-    (property "Value" "ADG736BRM" (at 160.655 101.6 0)
-      (effects (font (size 1.27 1.27)))
-    )
-    (property "Footprint" "SOP50P490X110-10N" (at 169.545 201.6 0)
-      (effects (font (size 1.27 1.27)) (justify left top) hide)
-    )
-    (property "Datasheet" "https://www.arrow.com/en/products/adg736brm/analog-devices?region=nac" (at 169.545 301.6 0)
-      (effects (font (size 1.27 1.27)) (justify left top) hide)
-    )
-    (property "Height" "1.1" (at 169.545 501.6 0)
-      (effects (font (size 1.27 1.27)) (justify left top) hide)
-    )
-    (property "Manufacturer_Name" "Analog Devices" (at 169.545 601.6 0)
-      (effects (font (size 1.27 1.27)) (justify left top) hide)
-    )
-    (property "Manufacturer_Part_Number" "ADG736BRM" (at 169.545 701.6 0)
-      (effects (font (size 1.27 1.27)) (justify left top) hide)
-    )
-    (property "Mouser Part Number" "" (at 169.545 801.6 0)
-      (effects (font (size 1.27 1.27)) (justify left top) hide)
-    )
-    (property "Mouser Price/Stock" "" (at 169.545 901.6 0)
-      (effects (font (size 1.27 1.27)) (justify left top) hide)
-    )
-    (property "Arrow Part Number" "ADG736BRM" (at 169.545 1001.6 0)
-      (effects (font (size 1.27 1.27)) (justify left top) hide)
-    )
-    (property "Arrow Price/Stock" "https://www.arrow.com/en/products/adg736brm/analog-devices?region=nac" (at 169.545 1101.6 0)
-      (effects (font (size 1.27 1.27)) (justify left top) hide)
-    )
-    (pin "1")
-    (pin "10")
-    (pin "2")
-    (pin "3")
-    (pin "4")
-    (pin "5")
-    (pin "6")
-    (pin "7")
-    (pin "8")
-    (pin "9")
-    (instances
-      (project "bt_pcb"
-        (path "/eb787481-08cd-41a4-a128-173fa6227c32/4ada0139-8712-47ce-9d4c-ab8fef312f7b/92a88d42-e0ca-481e-a77e-2117fd7dfc0f"
-          (reference "IC9") (unit 1)
-        )
-      )
-    )
-  )
   (symbol (lib_id "Device:C") (at 200.66 42.545 0) (unit 1)
     (in_bom yes) (on_board yes) (dnp no) (fields_autoplaced)
@@
         )
       )
-    )
-  )
-  (symbol (lib_id "SamacSys:ADG736BRM") (at 147.955 34.925 0) (unit 1)
-    (in_bom yes) (on_board yes) (dnp no) (fields_autoplaced)
-    (property "Reference" "IC8" (at 160.655 27.305 0)
-      (effects (font (size 1.27 1.27)))
-    )
-    (property "Value" "ADG736BRM" (at 160.655 29.845 0)
-      (effects (font (size 1.27 1.27)))
-    )
-    (property "Footprint" "SOP50P490X110-10N" (at 169.545 129.845 0)
-      (effects (font (size 1.27 1.27)) (justify left top) hide)
-    )
-    (property "Datasheet" "https://www.arrow.com/en/products/adg736brm/analog-devices?region=nac" (at 169.545 229.845 0)
-      (effects (font (size 1.27 1.27)) (justify left top) hide)
-    )
-    (property "Height" "1.1" (at 169.545 429.845 0)
-      (effects (font (size 1.27 1.27)) (justify left top) hide)
-    )
-    (property "Manufacturer_Name" "Analog Devices" (at 169.545 529.845 0)
-      (effects (font (size 1.27 1.27)) (justify left top) hide)
-    )
-    (property "Manufacturer_Part_Number" "ADG736BRM" (at 169.545 629.845 0)
-      (effects (font (size 1.27 1.27)) (justify left top) hide)
-    )
-    (property "Mouser Part Number" "" (at 169.545 729.845 0)
-      (effects (font (size 1.27 1.27)) (justify left top) hide)
-    )
-    (property "Mouser Price/Stock" "" (at 169.545 829.845 0)
-      (effects (font (size 1.27 1.27)) (justify left top) hide)
-    )
-    (property "Arrow Part Number" "ADG736BRM" (at 169.545 929.845 0)
-      (effects (font (size 1.27 1.27)) (justify left top) hide)
-    )
-    (property "Arrow Price/Stock" "https://www.arrow.com/en/products/adg736brm/analog-devices?region=nac" (at 169.545 1029.845 0)
-      (effects (font (size 1.27 1.27)) (justify left top) hide)
-    )
-    (pin "1")
-    (pin "10")
-    (pin "2")
-    (pin "3")
-    (pin "4")
-    (pin "5")
-    (pin "6")
-    (pin "7")
-    (pin "8")
-    (pin "9")
-    (instances
-      (project "bt_pcb"
-        (path "/eb787481-08cd-41a4-a128-173fa6227c32/4ada0139-8712-47ce-9d4c-ab8fef312f7b/92a88d42-e0ca-481e-a77e-2117fd7dfc0f"
-          (reference "IC8") (unit 1)
-        )
-      )

Commit message: progress
Parts:
- IC1, IC2: footprint SOP50P490X110-10N -> library:SOP50P490X110-10N
Changed lines of the file:
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@@
       (effects (font (size 1.27 1.27)))
     )
-    (property "Footprint" "SOP50P490X110-10N" (at 169.545 129.845 0)
+    (property "Footprint" "library:SOP50P490X110-10N" (at 169.545 129.845 0)
       (effects (font (size 1.27 1.27)) (justify left top) hide)
     )
@@
       (effects (font (size 1.27 1.27)) (justify left top) hide)
     )
+    (pin "1")
+    (pin "10")
+    (pin "2")
+    (pin "3")
+    (pin "4")
+    (pin "5")
+    (pin "6")
+    (pin "7")
     (pin "8")
-    (pin "2")
-    (pin "7")
-    (pin "10")
-    (pin "3")
-    (pin "6")
-    (pin "1")
-    (pin "5")
     (pin "9")
-    (pin "4")
     (instances
       (project "bt_pcb"
@@
       (effects (font (size 1.27 1.27)))
     )
-    (property "Footprint" "SOP50P490X110-10N" (at 169.545 201.6 0)
+    (property "Footprint" "library:SOP50P490X110-10N" (at 169.545 201.6 0)
       (effects (font (size 1.27 1.27)) (justify left top) hide)
     )
@@
       (effects (font (size 1.27 1.27)) (justify left top) hide)
     )
+    (pin "1")
+    (pin "10")
     (pin "2")
     (pin "3")
     (pin "4")
-    (pin "1")
-    (pin "10")
+    (pin "5")
     (pin "6")
+    (pin "7")
+    (pin "8")
     (pin "9")
-    (pin "8")
-    (pin "5")
-    (pin "7")
-    (instances
-      (project "bt_pcb"
+    (instances
+      (project "bt_pcb"
