File: pcb/mcus.kicad_sch (KiCad schematic)
At the start: 38 parts, among them IC11 STM32H523CEU6, IC4 STM32H750VBT6, IC5 W25Q512JVEIM, J14 Conn_02x09_Top_Bottom, J15 Conn_JTAG_SWD_10, J2 Conn_JTAG_SWD_10, Y1 Crystal, Y2 Crystal

Commit message: progress
Parts:
- IC11: footprint QFN50P700X700X60-49N-D -> library:QFN50P700X700X60-49N-D
- IC4: footprint QFP50P1600X1600X160-100N -> library:QFP50P1600X1600X160-100N
- IC5: footprint SON127P800X600X80-9N-D -> library:SON127P800X600X80-9N-D
Connections:
- net POT_0 is gone; now on net A: IC4.17 (PC2_C)
- net POT_1 is gone; now on net A: IC4.18 (PC3_C)
- net POT_2 is gone; now on net A: IC4.15 (PC0)
- net POT_3 is gone; now on net A: IC4.16 (PC1)
- net INA_SELECT: no longer IC4.22 (PA0)
- net INB_SELECT: no longer IC4.23 (PA1)
- net MCU2_DEB_SWCLK: now also IC11.37 (PA14)
- net MCU2_DEB_SWDIO: now also IC11.34 (PA13)
- net OUTA_SELECT: no longer IC4.24 (PA2)
- net OUTB_SELECT: no longer IC4.25 (PA3)
- net A: now reaches IC4.33 (PC5)
- net A: now also IC4.22 (PA0), IC4.23 (PA1), IC4.24 (PA2), IC4.25 (PA3), IC4.34 (PB0), IC4.35 (PB1)
- net BTN_0: no longer names the net of IC4.87 (PD6)
- net BTN_1: no longer names the net of IC4.86 (PD5)
- net BTN_2: no longer names the net of IC4.85 (PD4)
- net BTN_3: no longer names the net of IC4.84 (PD3)
- net BTN_4: no longer names the net of IC4.83 (PD2)
- net BTN_5: no longer names the net of IC4.82 (PD1)
- net BTN_6: no longer names the net of IC4.81 (PD0)
- net BTN_7: no longer names the net of IC4.80 (PC12)
- net ENC_A_0: no longer names the net of IC4.4 (PE5)
- net ENC_B_0: no longer names the net of IC4.5 (PE6)
- net ENC_SW_0: no longer names the net of IC4.7 (PC13)
- net INA_SW: no longer names the net of IC4.98 (PE1)
- net INB_SW: no longer names the net of IC4.97 (PE0)
- net OUTA_SW: no longer names the net of IC4.96 (PB9)
- net OUTB_SW: no longer names the net of IC4.95 (PB8)
- net POT_SW_0: no longer names the net of IC4.1 (PE2)
- net POT_SW_1: no longer names the net of IC4.2 (PE3)
- net POT_SW_2: no longer names the net of IC4.3 (PE4)
Other:
- note added: "H523CEU6 USART 1 Tx PB14, PA9, PB6, PA15() Rx PB15, PA10, PB7 USART 2 Tx PA2, PB0 Rx PA3 USART 3 Tx PB10 Rx PB1"
- note added: "H750VBT6 USART 1 Tx PB14, PA9, PB6 Rx PB15, PA10, PB7 USART 2 Tx PA2, PD5 Rx PA3, PD6 USART 3 Tx PB10, PD8, PC10 Rx PB11, PD9, PC11 USART 6 Tx PC6 Rx PC7"
- note removed: "USART 1 - rx PB15 - tx PB14 USART 2 - tx PA2 - rx PA3 USART 3 - rx PD9 - tx PD8 USART 6 - rx PC7 - tx PC6"
- moved on the sheet: C109
