File: pcb/user_interface.kicad_sch (KiCad schematic)
At the start: 31 parts, among them J9 AudioJack3_Switch, SW1 SW_Push, SW2 SW_Push, SW3 SW_Push, SW4 SW_Push, SW5 SW_Push, SW6 SW_Push, SW7 SW_Push, SW8 SW_Push, SW9 SW_Push

Commit message: minor
Parts:
- renumbered R23 to R22, R23 to R24, R23 to R25, R23 to R26, R23 to R27, R23 to R28, R23 to R29, R23 to R30, R23 to R31
Other:
- note added: "most common CW - S CCW - R Wip - T second most common CW - S Wip - R CCW - T ewwwwwwwwww CW - S Wip - T CCW - T"
- note removed: "CW - S CCW - R Wip - T CW - S Wip - R CCW - T CW - S Wip - T CCW - T"

Commit message: a lot of work! almost ready for rev
Parts:
- added C51, C52, C53, C54, C55, C56, C57, C58, C59, C60: 0.1uF, symbol Device:C
- added D6, D7, D8, D9: LED, symbol Device:LED
- added J10, J11: AudioJack3_Switch, symbol Connector_Audio:AudioJack3_Switch
- added R32, R33, R34, R35, R36, R37, R39, R40, R68, R69, R70: 10k, symbol Device:R
- added R38, R41, R42, R43: 680, symbol Device:R
- added R71: R, symbol Device:R
- added RV1: R_Potentiometer, symbol Device:R_Potentiometer
- added SW10: RotaryEncoder_Switch, symbol Device:RotaryEncoder_Switch
- added SW11, SW12, SW13: SW_Push, symbol Switch:SW_Push
- R4: value 1k -> 680
Connections:
- net +3V3: now also J9.T, J9.TN, C51.1, C52.1, C53.1, C54.1, C57.1, C58.1, C59.1, C60.1, J10.T, J10.TN, J11.T, J11.TN, R33.1, R35.1, R39.1, R40.1, RV1.1, SW10.S1, SW11.2, SW12.2, SW13.2
- net GND: now also C55.2, C56.2, D6.1 (K), D7.1 (K), D8.1 (K), D9.1 (K), J10.S, J11.S, R32.1, R34.1, R36.1, R37.2, R68.2, R69.2, R70.2, R71.2, SW10.C
- net POT_0: now reaches J9.R, J9.RN
- net POT_0: now also C52.2, R32.2
- net BTN_8 renamed INA_SW
- net SW_EXP_0 renamed POT_SW_0
- new net: D7.2 (A), R41.2
- new net: R71.1, RV1.3
- new net: D8.2 (A), R42.2
- new net: D9.2 (A), R43.2
- new net: D6.2 (A), R38.2
- new net ENC_A_0: C55.1, R39.2, SW10.A
- new net ENC_B_0: C56.1, R40.2, SW10.B
- new net ENC_SW_0: C54.2, R37.1, SW10.S2
- new net INB_SW: C58.2, R69.1, SW12.1
- new net LED_0: R38.1
- new net LED_1: R41.1
- new net LED_2: R42.1
- new net LED_3: R43.1
- new net OUTA_SW: C57.2, R68.1, SW11.1
- new net OUTB_SW: C59.2, R70.1, SW13.1
- new net POT_1: C51.2, J10.R, J10.RN, R34.2
- new net POT_2: C53.2, J11.R, J11.RN, R36.2
- new net POT_3: C60.2, RV1.2
- new net POT_SW_1: J10.SN, R33.2
- new net POT_SW_2: J11.SN, R35.2
Other:
- note added: "5 buttons for the cursor up - down - left - right - enter 3 buttons for quick functions start - lock - mute 4 switches for inA, inB, outA, outB selection 1 rotary encoder for value control 5 leds power, ready, quick functions 1 pot for headhones volume"
- note added: "680 for red, blue, orange 510 for green the pins are rated for 8mA, so we could technically go lower"
- note added: "small circles led big circle encoder squares buttons"
- moved on the sheet: C46, C47, C48, C49, R27, R28, R29, R30, SW5, SW6, SW7, SW8

Commit message: schematic finished, now under revision
Parts:
- added C61, C62, C63: 100nF, symbol Device:C
- added J4: Conn_01x10, symbol Connector_Generic:Conn_01x10
- added J6: Conn_01x14, symbol Connector_Generic:Conn_01x14
Connections:
- net +3V3: now also C61.2, C62.2, C63.2, J4.9 (Pin_9), J6.1 (Pin_1), J6.8 (Pin_8)
- net GND: now also C61.1, C62.1, C63.1, J4.10 (Pin_10), J6.2 (Pin_2)
- new net DISPLAY_GPIO_0: J4.6 (Pin_6), J6.4 (Pin_4)
- new net DISPLAY_GPIO_1: J4.5 (Pin_5), J6.3 (Pin_3)
- new net DISPLAY_GPIO_2: J4.4 (Pin_4), J6.5 (Pin_5)
- new net DISPLAY_GPIO_3: J4.3 (Pin_3)
- new net DISPLAY_SPI_MISO: J6.9 (Pin_9)
- new net DISPLAY_SPI_MOSI: J4.7 (Pin_7), J6.6 (Pin_6)
- new net DISPLAY_SPI_SCK: J4.8 (Pin_8), J6.7 (Pin_7)
- new net TOUCH_CS: J6.11 (Pin_11)
- new net TOUCH_IRQ: J6.14 (Pin_14)
- new net TOUCH_SPI_MISO: J6.13 (Pin_13)
- new net TOUCH_SPI_MOSI: J6.12 (Pin_12)
- new net TOUCH_SPI_SCK: J6.10 (Pin_10)
- no-connect marks 0 -> 4
Other:
- note added: "Display ER-OLED"
- note added: "Display ILI9341"
- note added: "GND VDD SCLK SDIN RST D/C CS1 CS2 FR1 FR2"
- note added: "VDD GND CS RST DC/RS SDI SCK LED SDO T_CLK T_CS T_DIN T_DO T_IRQ"
- note added: "from the example arduino code == Hardware connection == OLED => Arduino *1. GND -> GND *2. VCC -> 3.3 *3. SCL -> SCK *4. SDI -> MOSI *5. RES -> 8 *6. DC -> 9 *7. CS1 -> 10 *8. CS2 -> 7 *9. FR1 -> NC *10.FR2 -> NC"
- moved on the sheet: C42, C43, C44, C45, C46, C47, C48, C49, C50, C51, C52, C53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

Commit message: progress
Parts:
- removed C57, C58, C59: 0.1uF, symbol Device:C
- removed C62, C63: 100nF, symbol Device:C
- removed J6: Conn_01x14, symbol Connector_Generic:Conn_01x14
- removed R70: 10k, symbol Device:R
- removed SW11, SW12, SW13: SW_Push, symbol Switch:SW_Push
- added C116: 0.1uF, symbol Device:C
- added D10, D5: LED, symbol Device:LED
- added J16: AudioJack3_Switch, symbol Connector_Audio:AudioJack3_Switch
- added R78, R79: 10k, symbol Device:R
- R68, R69: value 10k -> 680
Connections:
- net INA_SW is gone; now on net BTN_0: C50.2, R31.1, SW9.1
- net POT_3 is gone; now on net POT_0: C60.2, RV1.2
- net +3V3: now also J4.2 (Pin_2), C116.1, J16.T, J16.TN, R78.1; no longer J4.9 (Pin_9)
- net BTN_0: no longer C42.2, R25.1, SW1.1
- net BTN_1: now also C42.2, R25.1, SW1.1; no longer C43.2, R23.1, SW2.1
- net BTN_2: now also C43.2, R23.1, SW2.1; no longer C44.2, R24.1, SW3.1
- net BTN_3: now also C44.2, R24.1, SW3.1; no longer C45.2, R26.1, SW4.1
- net BTN_4: now also C45.2, R26.1, SW4.1; no longer C46.2, R27.1, SW5.1
- net BTN_5: now also C46.2, R27.1, SW5.1; no longer C47.2, R28.1, SW6.1
- net BTN_6: now also C47.2, R28.1, SW6.1; no longer C48.2, R29.1, SW7.1
- net BTN_7: now also C48.2, R29.1, SW7.1; no longer C49.2, R30.1, SW8.1
- net DISPLAY_GPIO_1: now also J4.7 (Pin_7); no longer J4.5 (Pin_5)
- net DISPLAY_GPIO_2: now also J4.8 (Pin_8); no longer J4.4 (Pin_4)
- net DISPLAY_GPIO_3: now also J4.9 (Pin_9); no longer J4.3 (Pin_3)
- net DISPLAY_SPI_MISO: now also J4.4 (Pin_4)
- net DISPLAY_SPI_MOSI: now also J4.5 (Pin_5); no longer J4.7 (Pin_7)
- net DISPLAY_SPI_SCK: now also J4.3 (Pin_3); no longer J4.8 (Pin_8)
- net GND: now also J4.1 (Pin_1), D10.1 (K), D5.1 (K), J16.S, R79.1; no longer J4.10 (Pin_10), R68.2, R69.2
- net POT_0: no longer C52.2, J9.R, J9.RN, R32.2
- net ENC_A_0 renamed ENC_A
- net ENC_B_0 renamed ENC_B
- net ENC_SW_0 renamed ENC_SW
- net INB_SW renamed LED_5
- net OUTA_SW renamed LED_4
- net POT_1 renamed EXP_1
- net POT_2 renamed EXP_2
- net POT_SW_0 renamed EXP_SW_0
- net POT_SW_1 renamed EXP_SW_1
- net POT_SW_2 renamed EXP_SW_2
- new net: D10.2 (A), R69.2
- new net: D5.2 (A), R68.2
- new net BTN_8: C49.2, R30.1, SW8.1
- new net DISPLAY_GPIO_4: J4.10 (Pin_10)
- new net EXP_0: C52.2, J9.R, J9.RN, R32.2
- new net EXP_3: C116.2, J16.R, J16.RN, R79.2
- new net EXP_SW_3: J16.SN, R78.2
- no-connect marks 4 -> 0
Other:
- note added: "5 buttons for the cursor up - down - left - right - enter 4 buttons for quick functions start - lock - mute - beat 1 rotary encoder for value control 7 leds power, ready 1, ready 2, quick functions 1 pot for headhones volume"
- note removed: "5 buttons for the cursor up - down - left - right - enter 3 buttons for quick functions start - lock - mute 4 switches for inA, inB, outA, outB selection 1 rotary encoder for value control 5 leds power, ready, quick functions 1 pot for headhones volume"
- note removed: "GND VDD SCLK SDIN RST D/C CS1 CS2 FR1 FR2"
- moved on the sheet: C42, C43, C44, C45, C51, C52, C53, C54, C55, C56, C60, C61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
