File: pcb/bt_pcb.kicad_sch (KiCad schematic)
At the start: 23 parts, among them IC4 STM32H750VBT6, IC5 W25Q512JVEIM, J2 Conn_JTAG_SWD_10, J6 Micro_SD_Card, Y1 Crystal

Commit message: progress
Parts:
- removed J6: Micro_SD_Card, symbol Connector:Micro_SD_Card
Connections:
- net +3V3: no longer IC5.3 (~{WP_(IO2)}), IC5.7 (~{HOLD_OR_}/RESET_(IO3))
- net FLASH_QPI_MCK: now reaches IC4.36 (PB2)
- net FLASH_QPI_MCK: now also IC5.6 (CLK)
- net FLASH_QPI_IO0: now reaches IC4.37 (PE7)
- net FLASH_QPI_IO0: now also IC5.5 (DI_(IO0))
- net FLASH_QPI_IO1: now reaches IC4.38 (PE8)
- net FLASH_QPI_IO1: now also IC5.2 (DO_(IO1))
- net FLASH_QPI_IO2: now reaches IC4.39 (PE9)
- net FLASH_QPI_IO2: now also IC5.3 (~{WP_(IO2)})
- net FLASH_QPI_IO3: now reaches IC4.40 (PE10)
- net FLASH_QPI_IO3: now also IC5.7 (~{HOLD_OR_}/RESET_(IO3))
- net USB_VBUS: now reaches IC4.68 (PA9)
- net USB_D-: now reaches IC4.70 (PA11)
- net USB_D+: now reaches IC4.71 (PA12)
- net FLASH_QPI_NCS: now reaches IC4.79 (PC11)
- net FLASH_QPI_NCS: now also IC5.1 (~{CS})
- net F_SPI_CLK: no longer names the net of IC4.52 (PB13)
- net F_SPI_CLK: no longer IC5.6 (CLK)
- net F_SPI_CS: no longer names the net of IC4.51 (PB12)
- net F_SPI_CS: no longer IC5.1 (~{CS})
- net F_SPI_MISO: no longer names the net of IC4.53 (PB14)
- net F_SPI_MISO: no longer IC5.2 (DO_(IO1))
- net F_SPI_MOSI: no longer names the net of IC4.54 (PB15)
- net F_SPI_MOSI: no longer IC5.5 (DI_(IO0))
Other:
- added sheet USB Interface (usb_interface.kicad_sch)
- sheet Codec and audio IO ports: added none; removed AINCS, BINCS
- sheet Power Supply ports: added VBUS; removed none
- note added: "TODO LIST: - usb device and vbus - finish the analog - hp out - jack trs as input - UI - display and leds - adc for externals - rotary encoders"
- note removed: "TODO LIST: - make the sd card - UI - display and leds - adc for externals - rotary encoders"
- note removed: "not sure about nrst"
- moved on the sheet: C19, C20, C21, C22, C23, C24, C26, C27, C28, C29, C30, C32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

Commit message: making up my mind on the heaphones
Other:
- sheet Codec and audio IO ports: added none; removed 3V3, 5V0
- sheet Power Supply ports: added none; removed 3V3, 5V0
Changed lines of the file:
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@@
-    (stroke (width 0) (type default))
-  )
-  (wire (pts (xy 94.615 37.465) (xy 106.68 37.465))
     (stroke (width 0) (type default))
   )
@@
     (stroke (width 0) (type default))
   )
-  (wire (pts (xy 94.615 34.925) (xy 100.965 34.925))
-    (stroke (width 0) (type default))
-  )
-  (wire (pts (xy 73.025 151.765) (xy 77.47 151.765))
-    (stroke (width 0) (type default))
-  )
   (wire (pts (xy 196.215 111.76) (xy 239.395 111.76))
     (stroke (width 0) (type default))
@@
   )
   (wire (pts (xy 102.87 168.91) (xy 109.855 168.91))
-    (stroke (width 0) (type default))
-  )
-  (wire (pts (xy 66.675 154.305) (xy 77.47 154.305))
     (stroke (width 0) (type default))
   )
@@
     )
   )
-  (symbol (lib_id "power:+5V") (at 73.025 151.765 0) (unit 1)
-    (in_bom yes) (on_board yes) (dnp no) (fields_autoplaced)
-    (property "Reference" "#PWR048" (at 73.025 155.575 0)
-      (effects (font (size 1.27 1.27)) hide)
-    )
-    (property "Value" "+5V" (at 73.025 147.32 0)
-      (effects (font (size 1.27 1.27)))
-    )
-    (property "Footprint" "" (at 73.025 151.765 0)
-      (effects (font (size 1.27 1.27)) hide)
-    )
-    (property "Datasheet" "" (at 73.025 151.765 0)
-      (effects (font (size 1.27 1.27)) hide)
-    )
-    (pin "1")
-    (instances
-      (project "bt_pcb"
-        (path "/eb787481-08cd-41a4-a128-173fa6227c32"
-          (reference "#PWR048") (unit 1)
-        )
-      )
-    )
-  )
   (symbol (lib_id "power:GND") (at 197.485 159.385 0) (unit 1)
     (in_bom yes) (on_board yes) (dnp no) (fields_autoplaced)
@@
         (path "/eb787481-08cd-41a4-a128-173fa6227c32"
           (reference "C22") (unit 1)
-        )
-      )
-    )
-  )
-  (symbol (lib_id "power:+5V") (at 106.68 37.465 0) (unit 1)
-    (in_bom yes) (on_board yes) (dnp no) (fields_autoplaced)
-    (property "Reference" "#PWR050" (at 106.68 41.275 0)
-      (effects (font (size 1.27 1.27)) hide)
-    )
-    (property "Value" "+5V" (at 106.68 33.02 0)
-      (effects (font (size 1.27 1.27)))
-    )
-    (property "Footprint" "" (at 106.68 37.465 0)
-      (effects (font (size 1.27 1.27)) hide)
-    )
-    (property "Datasheet" "" (at 106.68 37.465 0)
-      (effects (font (size 1.27 1.27)) hide)
-    )
-    (pin "1")
-    (instances
-      (project "bt_pcb"
-        (path "/eb787481-08cd-41a4-a128-173fa6227c32"
-          (reference "#PWR050") (unit 1)
         )
       )
@@
     )
   )
-  (symbol (lib_id "power:+3V3") (at 100.965 34.925 0) (unit 1)
-    (in_bom yes) (on_board yes) (dnp no) (fields_autoplaced)
-    (property "Reference" "#PWR051" (at 100.965 38.735 0)
-      (effects (font (size 1.27 1.27)) hide)
-    )
-    (property "Value" "+3V3" (at 100.965 29.845 0)
-      (effects (font (size 1.27 1.27)))
-    )
-    (property "Footprint" "" (at 100.965 34.925 0)
-      (effects (font (size 1.27 1.27)) hide)
-    )
-    (property "Datasheet" "" (at 100.965 34.925 0)
-      (effects (font (size 1.27 1.27)) hide)
-    )
-    (pin "1")
-    (instances
-      (project "bt_pcb"
-        (path "/eb787481-08cd-41a4-a128-173fa6227c32"
-          (reference "#PWR051") (unit 1)
-        )
-      )
-    )
-  )
   (symbol (lib_id "power:GND") (at 210.185 122.555 0) (unit 1)
     (in_bom yes) (on_board yes) (dnp no) (fields_autoplaced)
@@
     )
   )
-  (symbol (lib_id "power:+3V3") (at 66.675 154.305 0) (unit 1)
-    (in_bom yes) (on_board yes) (dnp no) (fields_autoplaced)
-    (property "Reference" "#PWR049" (at 66.675 158.115 0)
-      (effects (font (size 1.27 1.27)) hide)
-    )
-    (property "Value" "+3V3" (at 66.675 149.225 0)
-      (effects (font (size 1.27 1.27)))
-    )
-    (property "Footprint" "" (at 66.675 154.305 0)
-      (effects (font (size 1.27 1.27)) hide)
-    )
-    (property "Datasheet" "" (at 66.675 154.305 0)
-      (effects (font (size 1.27 1.27)) hide)
-    )
-    (pin "1")
-    (instances
-      (project "bt_pcb"
-        (path "/eb787481-08cd-41a4-a128-173fa6227c32"
-          (reference "#PWR049") (unit 1)
-        )
-      )
-    )
-  )
   (symbol (lib_id "power:+3V3") (at 152.4 31.75 0) (unit 1)
     (in_bom yes) (on_board yes) (dnp no) (fields_autoplaced)
@@
       (effects (font (size 1.27 1.27)) (justify right))
     )
-    (pin "5V0" input (at 77.47 151.765 180)
-      (effects (font (size 1.27 1.27)) (justify left))
-    )
-    (pin "3V3" input (at 77.47 154.305 180)
-      (effects (font (size 1.27 1.27)) (justify left))
-    )
     (pin "CS_SDA" bidirectional (at 102.87 174.625 0)
       (effects (font (size 1.27 1.27)) (justify right))
@@
       (effects (font (size 1.27 1.27)) (justify left top))
     )
-    (pin "3V3" output (at 94.615 34.925 0)
-      (effects (font (size 1.27 1.27)) (justify right))
-    )
-    (pin "5V0" output (at 94.615 37.465 0)
-      (effects (font (size 1.27 1.27)) (justify right))
-    )
     (pin "VBUS" input (at 94.615 40.005 0)

Commit message: progress on hp
Other:
- sheet Codec and audio IO ports: added HP_SCL, HP_SD, HP_SDA; removed none
Changed lines of the file:
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@@
+    (stroke (width 0) (type default))
+  )
+  (wire (pts (xy 102.87 172.085) (xy 110.49 172.085))
+    (stroke (width 0) (type default))
+  )
+  (wire (pts (xy 257.175 44.45) (xy 257.175 41.91))
+    (stroke (width 0) (type default))
+  )
+  (wire (pts (xy 170.18 101.6) (xy 171.45 101.6))
+    (stroke (width 0) (type default))
+  )
+  (wire (pts (xy 214.63 122.555) (xy 214.63 124.46))
+    (stroke (width 0) (type default))
+  )
+  (wire (pts (xy 344.17 73.66) (xy 344.17 78.74))
+    (stroke (width 0) (type default))
+  )
+  (wire (pts (xy 307.975 173.355) (xy 319.405 173.355))
+    (stroke (width 0) (type default))
+  )
+  (wire (pts (xy 368.935 57.785) (xy 371.475 57.785))
+    (stroke (width 0) (type default))
+  )
+  (wire (pts (xy 352.425 40.005) (xy 356.235 40.005))
     (stroke (width 0) (type default))
   )
@@
     (stroke (width 0) (type default))
   )
-  (wire (pts (xy 257.175 44.45) (xy 257.175 41.91))
-    (stroke (width 0) (type default))
-  )
-  (wire (pts (xy 170.18 101.6) (xy 171.45 101.6))
-    (stroke (width 0) (type default))
-  )
-  (wire (pts (xy 214.63 122.555) (xy 214.63 124.46))
-    (stroke (width 0) (type default))
-  )
-  (wire (pts (xy 344.17 73.66) (xy 344.17 78.74))
-    (stroke (width 0) (type default))
-  )
-  (wire (pts (xy 307.975 173.355) (xy 319.405 173.355))
-    (stroke (width 0) (type default))
-  )
-  (wire (pts (xy 368.935 57.785) (xy 371.475 57.785))
-    (stroke (width 0) (type default))
-  )
-  (wire (pts (xy 352.425 40.005) (xy 356.235 40.005))
-    (stroke (width 0) (type default))
-  )
-  (wire (pts (xy 102.87 177.165) (xy 110.49 177.165))
-    (stroke (width 0) (type default))
-  )
   (wire (pts (xy 179.705 31.75) (xy 179.705 34.925))
     (stroke (width 0) (type default))
@@
     (stroke (width 0) (type default))
   )
-  (wire (pts (xy 102.87 168.91) (xy 109.855 168.91))
+  (wire (pts (xy 102.87 167.005) (xy 109.855 167.005))
     (stroke (width 0) (type default))
   )
@@
     )
   )
-  (global_label "CODEC_I2C_SCL" (shape input) (at 110.49 177.165 0) (fields_autoplaced)
-    (effects (font (size 1.27 1.27)) (justify left))
-    (property "Intersheetrefs" "${INTERSHEET_REFS}" (at 128.2918 177.165 0)
+  (global_label "CODEC_I2C_SCL" (shape input) (at 110.49 174.625 0) (fields_autoplaced)
+    (effects (font (size 1.27 1.27)) (justify left))
+    (property "Intersheetrefs" "${INTERSHEET_REFS}" (at 128.2918 174.625 0)
       (effects (font (size 1.27 1.27)) (justify left) hide)
     )
@@
     )
   )
-  (global_label "CODEC_RST" (shape input) (at 109.855 168.91 0) (fields_autoplaced)
-    (effects (font (size 1.27 1.27)) (justify left))
-    (property "Intersheetrefs" "${INTERSHEET_REFS}" (at 123.5444 168.91 0)
+  (global_label "CODEC_RST" (shape input) (at 109.855 167.005 0) (fields_autoplaced)
+    (effects (font (size 1.27 1.27)) (justify left))
+    (property "Intersheetrefs" "${INTERSHEET_REFS}" (at 123.5444 167.005 0)
       (effects (font (size 1.27 1.27)) (justify left) hide)
     )
@@
     )
   )
-  (global_label "CODEC_I2C_SDA" (shape bidirectional) (at 110.49 174.625 0) (fields_autoplaced)
-    (effects (font (size 1.27 1.27)) (justify left))
-    (property "Intersheetrefs" "${INTERSHEET_REFS}" (at 129.4636 174.625 0)
+  (global_label "CODEC_I2C_SDA" (shape bidirectional) (at 110.49 172.085 0) (fields_autoplaced)
+    (effects (font (size 1.27 1.27)) (justify left))
+    (property "Intersheetrefs" "${INTERSHEET_REFS}" (at 129.4636 172.085 0)
       (effects (font (size 1.27 1.27)) (justify left) hide)
     )
@@
       (effects (font (size 1.27 1.27)) (justify left top))
     )
-    (pin "CS_RST" input (at 102.87 168.91 0)
+    (pin "CS_RST" input (at 102.87 167.005 0)
       (effects (font (size 1.27 1.27)) (justify right))
     )
@@
       (effects (font (size 1.27 1.27)) (justify right))
     )
-    (pin "CS_SDA" bidirectional (at 102.87 174.625 0)
+    (pin "CS_SDA" bidirectional (at 102.87 172.085 0)
       (effects (font (size 1.27 1.27)) (justify right))
     )
-    (pin "CS_SCL" input (at 102.87 177.165 0)
+    (pin "CS_SCL" input (at 102.87 174.625 0)
       (effects (font (size 1.27 1.27)) (justify right))
     )
+    (pin "HP_SDA" bidirectional (at 102.87 184.785 0)
+      (effects (font (size 1.27 1.27)) (justify right))
+    )
+    (pin "HP_SD" input (at 102.87 182.245 0)
+      (effects (font (size 1.27 1.27)) (justify right))
+    )
+    (pin "HP_SCL" input (at 102.87 187.325 0)
+      (effects (font (size 1.27 1.27)) (justify right))
+    )

Commit message: a lot of audio finished, now onto ui
Parts:
- removed D2: LED, symbol Device:LED
- removed R4: 1k, symbol Device:R
- added J4: Conn_01x10, symbol Connector_Generic:Conn_01x10
Connections:
- net +3V3: now also J4.9 (Pin_9)
- net GND: now also J4.10 (Pin_10)
Other:
- added sheet User Interface (user_interface.kicad_sch)
- sheet Codec and audio IO ports: added INA_SW, INB_SW, OUTA_SW, OUTB_SW; removed none
- note added: "GND VDD SCLK SDIN RST D/C CS1 CS2 FR1 FR2"
- note added: "TODO LIST: - is ESD protection needed? - display and leds - adc for externals - rotary encoders"
- note removed: "TODO LIST: - usb device and vbus - finish the analog - hp out - jack trs as input - UI - display and leds - adc for externals - rotary encoders"
- note removed: "for pcm3060 - LRCK word select - BCK bit clock - DIN line from ADC - DOUT line to DAC - SCK == 256 * FS (system operation)"
- moved on the sheet: C21, C22, C23, C24, C26, C27, C28, C29, C30, C32, C34, IC4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

Commit message: a lot of work! almost ready for rev
Parts:
- added D10, D11, D12: ESD5Zxx, Diode_SMD:D_SOD-523, symbol Diode:ESD5Zxx
- added J12: USB_C_Receptacle, symbol Connector:USB_C_Receptacle
- added R72: 4k7, symbol Device:R
- added R73, R74: 5k1, symbol Device:R
- added R75: 10k, symbol Device:R
Connections:
- net GND: now also D10.2 (A), D11.2 (A), D12.2 (A), J12.A1 (GND), J12.A12 (GND), J12.B1 (GND), J12.B12 (GND), J12.S1 (SHIELD), R73.2, R74.2, R75.2
- net USB_D+: now also D12.1 (K), J12.A6 (D+), J12.B6 (D+)
- net USB_D-: now also D11.1 (K), J12.A7 (D-), J12.B7 (D-)
- net POT_2: now reaches IC4.15 (PC0)
- net POT_3: now reaches IC4.16 (PC1)
- net POT_0: now reaches IC4.17 (PC2_C)
- net POT_1: now reaches IC4.18 (PC3_C)
- net HP_SD: now reaches IC4.91 (PB5)
- net HP_I2C_SCL: now reaches IC4.92 (PB6)
- net HP_I2C_SDA: now reaches IC4.93 (PB7)
- net USB_VBUS renamed VBUS_SENSE
- net VBUS_SENSE: now also R72.2, R75.1
- new net: J12.B5 (CC2), R73.1
- new net: J12.A5 (CC1), R74.1
- new net VBUS: D10.1 (K), J12.A4 (VBUS), J12.A9 (VBUS), J12.B4 (VBUS), J12.B9 (VBUS), R72.1
- no-connect marks 2 -> 12
Other:
- removed sheet USB Interface
- sheet Codec and audio IO ports: added none; removed CS_LRCK, CS_MCLK, CS_RST, CS_SCL, CS_SCLK, CS_SDA, CS_SDIN, CS_SDOUT, HP_SCL, HP_SD, HP_SDA, INA_SW, INB_SW, OUTA_SW, OUTB_SW
- sheet Power Supply ports: added none; removed VBUS
- note added: "Displayyy GND VDD SCLK SDIN RST D/C CS1 CS2 FR1 FR2"
- note added: "Need to ask what diodes are good. TI says: - esd321 for data lines - esd441 for power lines"
- note added: "TODO LIST: - connect the display - place the gpio acdc"
- note removed: "GND VDD SCLK SDIN RST D/C CS1 CS2 FR1 FR2"
- note removed: "TODO LIST: - is ESD protection needed? - display and leds - adc for externals - rotary encoders"
- moved on the sheet: J4, R3
