File: pcb/bt_pcb/mcus.kicad_sch (KiCad schematic)
At the start: 32 parts, among them IC3 STM32H750VBT6, IC4 STM32H523CEU6, IC5 W25Q512JVEIM, J13 FTSH-107-01-L-DV-K-A, J14 FTSH-107-01-L-DV-K-A, J15 Conn_01x04, J16 Conn_01x04

Commit message: pcb now under revision
Parts:
- removed J13, J14: FTSH-107-01-L-DV-K-A, library:FTSH-107-XX-YYY-DV-K-A, symbol library:FTSH-107-01-L-DV-K-A
- added J13, J14: Conn_01x05, Connector_PinHeader_2.54mm:PinHeader_1x05_P2.54mm_Vertical, symbol Connector_Generic:Conn_01x05
- renumbered C43 to C47, C44 to C48, C45 to C49, C46 to C50, C47 to C51, C48 to C52, C49 to C53, C50 to C54, C51 to C55, C52 to C56, C53 to C57, C54 to C58, C55 to C59, C56 to C60, C57 to C61, C58 to C62, C59 to C63, C60 to C64, C61 to C65, R39 to R40, R40 to R41, R41 to R42, R42 to R43
Connections:
- net +3V3: now also J13.5 (Pin_5), J14.5 (Pin_5)
- net EXP_SW_0: now also IC3.54 (PB15); no longer IC3.1 (PE2)
- net EXP_SW_1: now also IC3.53 (PB14); no longer IC3.2 (PE3)
- net EXP_SW_2: now also IC3.52 (PB13); no longer IC3.3 (PE4)
- net EXP_SW_3: now also IC3.51 (PB12); no longer IC3.4 (PE5)
- net GND: now also J13.1 (Pin_1), J14.1 (Pin_1); no longer IC4.43 (PB7)
- net INA_SW: now also IC3.1 (PE2); no longer IC3.54 (PB15)
- net INB_SW: now also IC3.2 (PE3); no longer IC3.53 (PB14)
- net MCU1_DEB_SWCLK: now also J14.3 (Pin_3)
- net MCU1_DEB_SWDIO: now also J14.4 (Pin_4)
- net MCU1_NRST: now also J14.2 (Pin_2)
- net MCU2_DEB_SWCLK: now also J13.3 (Pin_3)
- net MCU2_DEB_SWDIO: now also J13.4 (Pin_4)
- net MCU2_NRST: now also J13.2 (Pin_2)
- net OUTA_SW: now also IC3.3 (PE4); no longer IC3.52 (PB13)
- net OUTB_SW: now also IC3.4 (PE5); no longer IC3.51 (PB12)
- new net BTN_9_J: IC4.43 (PB7)
- no-connect marks 14 -> 0
