File: pcb/bt_pcb/mcus.kicad_sch (KiCad schematic)
At the start: 37 parts, among them IC3 STM32H750VBT6, IC4 STM32H523CEU6, IC5 W25Q512JVEIM, J12 Conn_01x05, J13 Conn_01x05, J14 Conn_01x05

Commit message: aaaaaaa
Parts:
- removed IC4: STM32H523CEU6, library:QFN50P700X700X60-49N-D, symbol library:STM32H523CEU6
- removed TP1, TP2, TP3, TP4: TestPoint, TestPoint:TestPoint_Pad_D1.0mm, symbol Connector:TestPoint
- added IC5: STM32H523CET6, library:QFP50P900X900X160-48N, symbol library:STM32H523CET6
- renumbered C46 to C45, C44 to C46, C49 to C47, C50 to C48, C39 to C49, C55 to C50, C56 to C51, C54 to C52, C42 to C54, C41 to C55, C45 to C56, C47 to C57, C48 to C58, C40 to C59, C38 to C60, C52 to C61, C51 to C62, C43 to C63, IC5 to IC3, IC3 to IC4, J13 to J10, J12 to J11, J14 to J12, R40 to R34, R37 to R35, R39 to R36, R41 to R37, R42 to R38, R38 to R39
Connections:
- net +3V3: now also IC5.1 (VBAT), IC5.24 (VDD_1), IC5.36 (VDD_2), IC5.48 (VDD_3), IC5.9 (VDDA)
- net AUX_1_TO_2: now also IC5.11 (PA1)
- net AUX_2_TO_1: now also IC5.10 (PA0)
- net BTN_0_J: now also IC5.38 (PA15)
- net BTN_1_J: now also IC5.39 (PB3)
- net BTN_2_J: now also IC5.40 (PB4)
- net BTN_3_J: now also IC5.41 (PB5)
- net BTN_4_J: now also IC5.42 (PB6)
- net BTN_5_QB: now also IC4.87 (PD6); no longer IC4.61 (PD14)
- net BTN_6_QB: now also IC4.85 (PD4); no longer IC4.59 (PD12)
- net BTN_7_QB: now also IC4.83 (PD2); no longer IC4.57 (PD10)
- net BTN_8_QB: now also IC4.81 (PD0); no longer IC4.55 (PD8)
- net BTN_9_J: now also IC5.43 (PB7)
- net DISPLAY_GPIO_0: now also IC5.17 (PA7)
- net DISPLAY_GPIO_1: now also IC5.18 (PB0)
- net DISPLAY_GPIO_2: now also IC5.19 (PB1)
- net DISPLAY_GPIO_3: now also IC5.20 (PB2)
- net DISPLAY_GPIO_4: now also IC5.21 (PB10)
- net DISPLAY_SPI_MISO: now also IC5.27 (PB14)
- net DISPLAY_SPI_MOSI: now also IC5.28 (PB15)
- net DISPLAY_SPI_SCK: now also IC5.26 (PB13)
- net ENC_A: now also IC5.3 (PC14-OSC32_IN)
- net ENC_B: now also IC5.4 (PC15-OSC32_OUT)
- net ENC_SW: now also IC5.2 (PC13)
- net GND: now also IC5.23 (VSS_1), IC5.35 (VSS_2), IC5.47 (VSS_3), IC5.8 (VSSA)
- net LED_1_RD: now also IC5.25 (PB12)
- net LED_2_QB: now also IC4.88 (PD7); no longer IC4.62 (PD15)
- net LED_3_QB: now also IC4.86 (PD5); no longer IC4.60 (PD13)
- net LED_4_QB: now also IC4.84 (PD3); no longer IC4.58 (PD11)
- net LED_5_QB: now also IC4.82 (PD1); no longer IC4.56 (PD9)
- net MCU2_DEB_SWCLK: now also IC5.37 (PA14)
- net MCU2_DEB_SWDIO: now also IC5.34 (PA13)
- net MCU2_NRST: now also IC5.7 (NRST)
- net USART_1_TO_2: now also IC5.13 (PA3)
- net USART_2_TO_1: now also IC5.12 (PA2)
- net at C61.1: now also IC5.22 (VCAP_1)
- net at J12.5 (Pin_5): now also IC5.29 (PA8)
- net at J12.4 (Pin_4): now also IC5.30 (PA9)
- net at J12.3 (Pin_3): now also IC5.31 (PA10)
- net at J12.2 (Pin_2): now also IC5.32 (PA11)
- net at J12.1 (Pin_1): now also IC5.33 (PA12)
- net at R39.2: now also IC5.44 (BOOT0)
- net at C60.1: now also IC5.46 (VCAP_2)
- net CODEC_RESET: now reaches IC4.33 (PC5)
- net CODEC_SPI_SCK: now reaches IC4.52 (PB13)
- net CODEC_SPI_MISO: now reaches IC4.53 (PB14)
- net CODEC_SPI_MOSI: now reaches IC4.54 (PB15)
- net CODEC_I2C_ADDR0: no longer names the net of IC4.44 (PE14)
- net CODEC_I2C_ADDR1: no longer names the net of IC4.43 (PE13)
- net CODEC_I2C_SCL: no longer names the net of IC4.46 (PB10)
- net CODEC_I2C_SDA: no longer names the net of IC4.47 (PB11)
- net CODEC_JACKDET: no longer names the net of IC4.45 (PE15)
- net INA_SW: no longer names the net of IC4.1 (PE2)
- net INB_SW: no longer names the net of IC4.2 (PE3)
- new net CODEC_SPI_CS: IC4.55 (PD8)
- no-connect marks 43 -> 49
Other:
- moved on the sheet: C56, C57, C58, C59, C60, C61, C62, C63, D17, D18, J12, R36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

Commit message: schematic rev b finish?
Parts:
- renumbered C49 to C61, C59 to C62, C55 to C63, C63 to C64, C54 to C65, C46 to C66, C56 to C67, C57 to C68, C45 to C69, C58 to C70, C47 to C71, C48 to C72, C62 to C73, C61 to C74, C53 to C75, C52 to C76, C50 to C77, C51 to C78, IC3 to IC6, J10 to J12, J12 to J13, R39 to R36, R36 to R37, R34 to R38, R37 to R39, R38 to R40
Connections:
- net CODEC_SPI_CS is gone; now on net USART_1_TO_2: IC4.55 (PD8)
- net AUX_1_TO_2: now also IC4.57 (PD10); no longer IC4.65 (PC8)
- net AUX_2_TO_1: now also IC4.58 (PD11); no longer IC4.66 (PC9)
- net USART_1_TO_2: no longer IC4.63 (PC6)
- net USART_2_TO_1: now also IC4.56 (PD9); no longer IC4.64 (PC7)
- net CODEC_I2C_SCL: now reaches IC4.46 (PB10)
- net CODEC_I2C_SDA: now reaches IC4.47 (PB11)
- net HPDAC_I2S_WS: now reaches IC4.51 (PB12)
- net HPDAC_I2C_SCL: now reaches IC4.59 (PD12)
- net HPDAC_I2C_SDA: now reaches IC4.60 (PD13)
- net FLASH_SPI_NCS: now reaches IC4.77 (PA15)
- net FLASH_SPI_NCS: now also IC6.1 (~{CS})
- net FLASH_SPI_MCK: now reaches IC4.78 (PC10)
- net FLASH_SPI_MCK: now also IC6.6 (CLK)
- net FLASH_SPI_MOSI: now reaches IC4.80 (PC12)
- net FLASH_SPI_MOSI: now also IC6.5 (DI_(IO0))
- net CODEC_I2S_CK renamed CODEC_I2S_BCK
- net CODEC_SPI_MISO renamed HPDAC_I2S_SDI
- net CODEC_SPI_MOSI renamed HPDAC_I2S_SDO
- net CODEC_SPI_SCK renamed HPDAC_I2S_BCK
- net FLASH_QPI_IO0: no longer names the net of IC4.37 (PE7)
- net FLASH_QPI_IO0: no longer IC6.5 (DI_(IO0))
- net FLASH_QPI_IO1: no longer names the net of IC4.38 (PE8)
- net FLASH_QPI_IO1: no longer IC6.2 (DO_(IO1))
- net FLASH_QPI_IO2: no longer names the net of IC6.3 (~{WP_(IO2)})
- net FLASH_QPI_IO2: no longer IC4.39 (PE9)
- net FLASH_QPI_IO3: no longer names the net of IC6.7 (~{HOLD_OR_}/RESET_(IO3))
- net FLASH_QPI_IO3: no longer IC4.40 (PE10)
- net FLASH_QPI_MCK: no longer names the net of IC4.36 (PB2)
- net FLASH_QPI_MCK: no longer IC6.6 (CLK)
- net FLASH_QPI_NCS renamed FLASH_SPI_MISO
- net FLASH_SPI_MISO: now also IC6.2 (DO_(IO1)); no longer IC6.1 (~{CS})
- new net HPDAC_I2S_MCK: IC4.63 (PC6)
- new net HPDAC_RESET: IC4.64 (PC7)
- no-connect marks 49 -> 47
Other:
- moved on the sheet: C65

Commit message: sd card is the way probably :(
Parts:
- added J19: Micro_SD_Card_Det2, Connector_Card:microSD_HC_Molex_104031-0811, symbol Connector:Micro_SD_Card_Det2
Changed lines of the file:
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@@
+	)
+	(symbol
+		(lib_id "Connector:Micro_SD_Card_Det2")
+		(at 203.2 251.46 0)
+		(unit 1)
+		(body_style 1)
+		(exclude_from_sim no)
+		(in_bom yes)
+		(on_board yes)
+		(in_pos_files yes)
+		(dnp no)
+		(fields_autoplaced yes)
+		(property "Reference" "J19"
+			(at 203.835 229.87 0)
+			(show_name no)
+			(do_not_autoplace no)
+			(effects
+				(font
+					(size 1.27 1.27)
+				)
+			)
+		)
+		(property "Value" "Micro_SD_Card_Det2"
+			(at 203.835 232.41 0)
+			(show_name no)
+			(do_not_autoplace no)
+			(effects
+				(font
+					(size 1.27 1.27)
+				)
+			)
+		)
+		(property "Footprint" "Connector_Card:microSD_HC_Molex_104031-0811"
+			(at 255.27 233.68 0)
+			(hide yes)
+			(show_name no)
+			(do_not_autoplace no)
+			(effects
+				(font
+					(size 1.27 1.27)
+				)
+			)
+		)
+		(property "Datasheet" "https://www.hirose.com/en/product/document?clcode=&productname=&series=DM3&documenttype=Catalog&lang=en&documentid=D49662_en"
+			(at 205.74 248.92 0)
+			(hide yes)
+			(show_name no)
+			(do_not_autoplace no)
+			(effects
+				(font
+					(size 1.27 1.27)
+				)
+			)
+		)
+		(property "Description" "Micro SD Card Socket with two card detection pins"
+			(at 203.2 251.46 0)
+			(hide yes)
+			(show_name no)
+			(do_not_autoplace no)
+			(effects
+				(font
+					(size 1.27 1.27)
+				)
+			)
+		)
+		(pin "5"
+		)
+		(pin "4"
+		)
+		(pin "2"
+		)
+		(pin "10"
+		)
+		(pin "8"
+		)
+		(pin "SH"
+		)
+		(pin "3"
+		)
+		(pin "1"
+		)
+		(pin "7"
+		)
+		(pin "6"
+		)
+		(pin "9"
+		)
+		(instances
+			(project "bt_pcb"
+				(path "/eb787481-08cd-41a4-a128-173fa6227c32/7b2258ec-f5b6-4970-96d8-f1fb6e4ed567"
+					(reference "J19")
+					(unit 1)
+				)
+			)
+		)
 	)
 	(symbol

Commit message: sd kind of in
Parts:
- removed IC6: W25Q512JVEIM, library:SON127P800X600X80-9N-D, symbol library:W25Q512JVEIM
- added C78: 2.2u, Capacitor_SMD:C_0603_1608Metric_Pad1.08x0.95mm_HandSolder, symbol Device:C
- added R38: 10k, Resistor_SMD:R_0603_1608Metric_Pad0.98x0.95mm_HandSolder, symbol Device:R
- renumbered C78 to C79, J19 to J14, R35 to R32, R36 to R33, R37 to R34, R38 to R35, R39 to R36, R40 to R37
Connections:
- net FLASH_SPI_MCK is gone; now on net SDMMC_D2: IC4.78 (PC10)
- net FLASH_SPI_MISO is gone; now on net SDMMC_D3: IC4.79 (PC11)
- net FLASH_SPI_MOSI is gone; now on net SDMMC_CK: IC4.80 (PC12)
- net +3V3: now also J14.4 (VDD), C78.1, R38.1
- net BTN_5_QB: now also IC4.91 (PB5); no longer IC4.87 (PD6)
- net BTN_6_QB: now also IC4.89 (PB3); no longer IC4.85 (PD4)
- net BTN_7_QB: now also IC4.87 (PD6); no longer IC4.83 (PD2)
- net BTN_8_QB: now also IC4.85 (PD4); no longer IC4.81 (PD0)
- net GND: now also J14.6 (VSS), J14.9 (DET_B), J14.SH (SHIELD), C78.2
- net LED_0_RD: now also IC4.93 (PB7); no longer IC4.67 (PA8)
- net LED_2_QB: now also IC4.92 (PB6); no longer IC4.88 (PD7)
- net LED_3_QB: now also IC4.90 (PB4); no longer IC4.86 (PD5)
- net LED_4_QB: now also IC4.88 (PD7); no longer IC4.84 (PD3)
- net LED_5_QB: now also IC4.86 (PD5); no longer IC4.82 (PD1)
- net SDMMC_D2: now reaches J14.1 (DAT2)
- net SDMMC_DET: now reaches J14.10 (DET_A)
- net SDMMC_DET: now also IC4.84 (PD3), R38.2
- net SDMMC_D3: now reaches J14.2 (DAT3/CD)
- net SDMMC_CMD: now reaches J14.3 (CMD)
- net SDMMC_CMD: now also IC4.83 (PD2)
- net SDMMC_CK: now reaches J14.5 (CLK)
- net SDMMC_D0: now reaches J14.7 (DAT0)
- net SDMMC_D0: now also IC4.65 (PC8)
- net SDMMC_D1: now reaches J14.8 (DAT1)
- net SDMMC_D1: now also IC4.66 (PC9)
- net FLASH_SPI_NCS: no longer names the net of IC4.77 (PA15)
- no-connect marks 47 -> 42
Other:
- moved on the sheet: C79, J14

Commit message: bom bom bom
Parts:
- IC4: now in the parts list
Changed lines of the file:
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@@
 		(body_style 1)
 		(exclude_from_sim no)
-		(in_bom no)
+		(in_bom yes)
 		(on_board yes)
 		(in_pos_files yes)

Commit message: reb b finished
Parts:
- renumbered C60 to C53, C61 to C54, C62 to C55, C63 to C56, C64 to C57, C65 to C58, C66 to C59, C67 to C60, C68 to C61, C69 to C62, C70 to C63, C71 to C64, C72 to C65, C73 to C66, C74 to C67, C75 to C68, C76 to C69, C77 to C70, C78 to C71, C79 to C72, R32 to R34, R33 to R35, R34 to R36, R35 to R37, R36 to R38, R37 to R39, R38 to R40
Connections:
- net CODEC_I2S_SDI renamed CODEC_I2S_MISO
- net CODEC_I2S_SDO renamed CODEC_I2S_MOSI
- net HPDAC_I2C_SCL: no longer names the net of IC4.59 (PD12)
- net HPDAC_I2C_SDA: no longer names the net of IC4.60 (PD13)
- net HPDAC_I2S_MCK: no longer names the net of IC4.63 (PC6)
- net HPDAC_I2S_SDI renamed HPDAC_IRQ
- net HPDAC_RESET: no longer names the net of IC4.64 (PC7)
- no-connect marks 42 -> 46
