File: pcb/bt_pcb/bt_pcb.kicad_pcb (KiCad board)
At the start: 4 copper layers, 135 x 80.5 mm, 232 parts, among them IC1 LTC3621EMS8E-25#PBF, IC2 ADAU1961WBCPZ-R7, IC3 STM32H750VBT6, IC4 STM32H523CEU6, IC5 W25Q512JVEIM, J1 Conn_01x02, J10 Conn_01x04, J11 Conn_01x04, J12 Conn_01x05, J13 Conn_01x05, J14 Conn_01x05, J15 Conn_01x04, J16 Conn_01x04, J17 ReanNYS216G, J18 ReanNYS216G, J19 ReanNYS216G, J2 694106301002, J20 ReanNYS216G, J3 Conn_01x01, J4 Conn_01x01, J5 Conn_01x03, J6 USB_C_Receptacle_USB2.0_16P, J7 Conn_01x04, J8 Conn_01x10, J9 Conn_01x04, SW1 SW_Push, SW10 SW_Push, SW2 SW_Push, SW3 SW_Push, SW4 SW_Push, SW5 SW_Push, SW6 SW_Push, SW7 SW_Push, SW8 SW_Push, SW9 SW_Push, U1 TLV76133DCY, U2 TLV76133DCY, U3 MCP6004, U4 MCP6004

Commit message: first reiteration
Parts:
- J13, J14: footprint Connector_PinHeader_2.54mm:PinHeader_1x05_P2.54mm_Vertical -> Connector_JST:JST_PH_B5B-PH-K_1x05_P2.00mm_Vertical
- J5: footprint Connector_PinHeader_2.54mm:PinHeader_1x03_P2.54mm_Vertical -> Connector_JST:JST_PH_B3B-PH-K_1x03_P2.00mm_Vertical
- moved J5 1.45 mm to (107.5, 90.5), turned to 0 degrees
- moved J13 1.12 mm to (115.0, 113.2), turned to 90 degrees
- moved J14 0.25 mm to (185.0, 113.0), turned to -90 degrees
Routing:
- net CODEC_HPR: track 16.1 -> 18.4 mm
- net CODEC_HPGND: track 13.0 -> 15.2 mm
- net MCU1_DEB_SWCLK: track 21.6 -> 19.4 mm
- net MCU1_DEB_SWDIO: track 21.5 -> 19.5 mm
- net CODEC_HPL: track 20.0 -> 21.9 mm
- net MCU2_DEB_SWDIO: track 14.5 -> 13.9 mm
- net MCU2_NRST: track 23.3 -> 23.9 mm

Commit message: doing pcb from scratch again
Parts:
- removed J19, J20: ReanNYS216G, library:NYS-216G
- removed the R18 at (159.8, 98.0)
- removed the R18 at (202.6, 131.5)
- removed R69, R71, R75, R77, R79, R82: 10k, Resistor_SMD:R_0603_1608Metric_Pad0.98x0.95mm_HandSolder
- removed R70, R73, R76: 634, Resistor_SMD:R_0603_1608Metric_Pad0.98x0.95mm_HandSolder
- removed R72, R74, R78: 91, Resistor_SMD:R_0603_1608Metric_Pad0.98x0.95mm_HandSolder
- removed R80, R81, R83, R84: 0, Resistor_SMD:R_0603_1608Metric_Pad0.98x0.95mm_HandSolder
- added C80: 2.7n, Capacitor_SMD:C_0603_1608Metric_Pad1.08x0.95mm_HandSolder, F.Cu at (142.0, 73.4)
- added C81: 470p, Capacitor_SMD:C_0603_1608Metric_Pad1.08x0.95mm_HandSolder, F.Cu at (147.0, 71.4)
- added C82: 10n, Capacitor_SMD:C_0603_1608Metric_Pad1.08x0.95mm_HandSolder, F.Cu at (150.1, 62.5)
- added C83: 10u, Capacitor_SMD:C_0805_2012Metric_Pad1.18x1.45mm_HandSolder, F.Cu at (141.0, 60.0)
- added R18: 680, Resistor_SMD:R_0603_1608Metric_Pad0.98x0.95mm_HandSolder, F.Cu at (-118.7, 99.0)
- added SW11: SW_Push, Button_Switch_THT:SW_TH_Tactile_Omron_B3F-102x, F.Cu at (70.2, 107.2)
- C1, C10, C11, C12, C13, C14, C2, C3, C34, C35, C36, C4, C5, C6, C7, C8, C9, D1, D2, IC1, J1, J13, J14, J17, J18, J2, J3, J4, J5, L1, R1, RV1, RV2, RV3, U1, U2: moved to B.Cu
- C55, C56, C57, C58, C59, C60, C61, C62, C68, C69, C79, IC5, R3, R4, R45, R49, R5, R53, R57, R6, R68, U3, U4: moved to F.Cu
- C63: footprint Capacitor_SMD:C_0805_2012Metric_Pad1.18x1.45mm_HandSolder -> Capacitor_SMD:C_0603_1608Metric_Pad1.08x0.95mm_HandSolder; moved to F.Cu
- C64: value 2.7n -> 100n; moved to F.Cu
- C65: value 10n -> 10u; footprint Capacitor_SMD:C_0603_1608Metric_Pad1.08x0.95mm_HandSolder -> Capacitor_SMD:C_0805_2012Metric_Pad1.18x1.45mm_HandSolder; moved to F.Cu
- C66, C74: value 470p -> 2.7n; moved to F.Cu
- C67: value 10u -> 10n; footprint Capacitor_SMD:C_0805_2012Metric_Pad1.18x1.45mm_HandSolder -> Capacitor_SMD:C_0603_1608Metric_Pad1.08x0.95mm_HandSolder; moved to F.Cu
- C70: value 2.7n -> 470p; moved to F.Cu
- C71, C77: value 470p -> 10u; footprint Capacitor_SMD:C_0603_1608Metric_Pad1.08x0.95mm_HandSolder -> Capacitor_SMD:C_0805_2012Metric_Pad1.18x1.45mm_HandSolder; moved to F.Cu
- C72: value 10n -> 10u; moved to F.Cu
- C73: value 10u -> 100n; footprint Capacitor_SMD:C_0805_2012Metric_Pad1.18x1.45mm_HandSolder -> Capacitor_SMD:C_0603_1608Metric_Pad1.08x0.95mm_HandSolder; moved to F.Cu
- C75: value 10u -> 470p; footprint Capacitor_SMD:C_0805_2012Metric_Pad1.18x1.45mm_HandSolder -> Capacitor_SMD:C_0603_1608Metric_Pad1.08x0.95mm_HandSolder; moved to F.Cu
- C76: value 2.7n -> 10n; moved to F.Cu
- C78: value 10n -> 470p; moved to F.Cu
- J10, J11: value Conn_01x04 -> Conn_01x03; footprint Connector_PinHeader_2.54mm:PinHeader_1x04_P2.54mm_Vertical -> Connector_JST:JST_PH_B3B-PH-K_1x03_P2.00mm_Vertical; moved to B.Cu
- J12: footprint Connector_PinHeader_2.54mm:PinHeader_1x05_P2.54mm_Vertical -> Connector_JST:JST_PH_B5B-PH-K_1x05_P2.00mm_Vertical; moved to B.Cu
- J15, J16: value Conn_01x04 -> ReanNYS216G; footprint Connector_PinHeader_2.54mm:PinHeader_1x04_P2.54mm_Vertical -> library:NYS-216G; moved to B.Cu
- J6: value USB_C_Receptacle_USB2.0_16P -> Conn_01x03; footprint Connector_USB:USB_C_Receptacle_GCT_USB4105-xx-A_16P_TopMnt_Horizontal -> Connector_JST:JST_PH_B3B-PH-K_1x03_P2.00mm_Vertical; moved to B.Cu
- J7: value Conn_01x04 -> ER-OLEDM0383-1-SPI_Conn_01x10; footprint Connector_PinHeader_2.54mm:PinHeader_1x04_P2.54mm_Vertical -> library:ER-OLEDM0383-1-SPI
- J8: value Conn_01x10 -> Conn_01x03; footprint Connector_PinHeader_2.54mm:PinHeader_1x10_P2.54mm_Vertical -> Connector_JST:JST_PH_B3B-PH-K_1x03_P2.00mm_Vertical; moved to B.Cu
- J9: value Conn_01x04 -> USB_C_Receptacle_USB2.0_16P; footprint Connector_PinHeader_2.54mm:PinHeader_1x04_P2.54mm_Vertical -> Connector_USB:USB_C_Receptacle_GCT_USB4105-xx-A_16P_TopMnt_Horizontal; moved to B.Cu
- R10, R9: value 5k1 -> 10k; moved to B.Cu
- R11, R12: value 10k -> 5k1
- R19, R20, R21, R39, R40: value 10k -> 680
- R25, R26, R27, R28, R44: value 680 -> 10k
- R41: value 10k -> 634
- R42: value 10k -> 91
- R43: value 680 -> 470
- R46, R54, R59: value 91 -> 10k; moved to F.Cu
- R47, R55: value 470 -> 91; moved to F.Cu
- R48, R56: value 10k -> 470; moved to F.Cu
- R50, R58: value 10k -> 91; moved to F.Cu
- R51: value 91 -> 470; moved to F.Cu
- R52: value 470 -> 10k; moved to F.Cu
- R60: value 470 -> 634; moved to F.Cu
- R61: value 47k -> 10k; moved to F.Cu
- R62: value 0 -> 91; moved to F.Cu
- R63, R66: value 0 -> 634; moved to F.Cu
- R64: value 47k -> 91; moved to F.Cu
- R65: value 0 -> 10k; moved to F.Cu
- R67: value 634 -> 10k; moved to F.Cu
- R7: value 4k7 -> 10k; moved to B.Cu
- R8: value 10k -> 4k7; moved to B.Cu
- RV4: footprint Connector_PinHeader_2.54mm:PinHeader_1x03_P2.54mm_Vertical -> Potentiometer_THT:Potentiometer_Alpha_RD901F-40-00D_Single_Vertical_CircularHoles
- SW1: value SW_Push -> RotaryEncoder_Switch; footprint Button_Switch_THT:SW_TH_Tactile_Omron_B3F-102x -> Rotary_Encoder:RotaryEncoder_Alps_EC11E-Switch_Vertical_H20mm_CircularMountingHoles
- moved D4 320.5 mm to (-106.2, 82.9), turned to 0 degrees
- moved D6 314.7 mm to (-106.2, 88.4), turned to 0 degrees
- moved D3 306.8 mm to (-93.8, 97.9), turned to 0 degrees
- moved D5 301.2 mm to (-93.8, 100.5), turned to 0 degrees
- moved D8 239.6 mm to (-106.2, 93.9), turned to 0 degrees
- moved R19 230.5 mm to (-118.7, 101.5)
- moved R20 226.4 mm to (-114.4, 81.5), turned to 0 degrees
- moved D7 225.3 mm to (-93.8, 103.1), turned to 0 degrees
- moved SW10 145.7 mm to (232.2, 116.8), turned to 90 degrees
- moved R27 143.5 mm to (63.7, 92.0), turned to 0 degrees
- moved R30 143.1 mm to (229.0, 80.5), turned to 180 degrees
- moved R25 141.5 mm to (63.7, 85.5), turned to 180 degrees
- moved R21 135.9 mm to (229.0, 87.5), turned to 0 degrees
- moved R28 135.4 mm to (73.7, 94.8), turned to 0 degrees
- moved R26 133.2 mm to (73.7, 84.8), turned to 0 degrees
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Connections:
- C63 pad 1: Net-(C63-Pad1) -> +3.3VA
- C63 pad 2: Net-(C63-Pad2) -> GND
- C64 pad 1: Net-(C63-Pad1) -> +3.3VA
- C64 pad 2: Net-(C64-Pad2) -> GND
- C65 pad 1: VCOM -> Net-(C65-Pad1)
- C65 pad 2: GND -> Net-(C65-Pad2)
- C66 pad 1: Net-(C66-Pad1) -> Net-(C65-Pad1)
- C66 pad 2: Net-(U3D--) -> Net-(C66-Pad2)
- C67 pad 1: Net-(C64-Pad2) -> VCOM
- C67 pad 2: Net-(C67-Pad2) -> GND
- C68 pad 2: Net-(U4A--) -> Net-(U3D--)
- C69 pad 1: Net-(U4A-+) -> Net-(C66-Pad2)
- C69 pad 2: /Codec and audio IO/Audio input/TA -> Net-(C69-Pad2)
- C70 pad 1: CODEC_INA+ -> Net-(C70-Pad1)
- C70 pad 2: CODEC_INA- -> Net-(U4A--)
- C71 pad 1: Net-(C71-Pad1) -> Net-(U4A-+)
- C71 pad 2: Net-(U4B--) -> /Codec and audio IO/Audio input/TA
- C72 pad 1: VCOM -> +3.3VA
- C73 pad 1: Net-(U4B-+) -> +3.3VA
- C73 pad 2: /Codec and audio IO/Audio input/RA -> GND
- C74 pad 1: Net-(C74-Pad1) -> CODEC_INA+
- C74 pad 2: Net-(U4C--) -> CODEC_INA-
- C75 pad 1: Net-(U4C-+) -> Net-(C75-Pad1)
- C75 pad 2: /Codec and audio IO/Audio input/TB -> Net-(U4B--)
- C76 pad 1: CODEC_INB+ -> VCOM
- C76 pad 2: CODEC_INB- -> GND
- C77 pad 1: Net-(C77-Pad1) -> Net-(U4B-+)
- C77 pad 2: Net-(U4D--) -> /Codec and audio IO/Audio input/RA
- C78 pad 1: VCOM -> Net-(C78-Pad1)
- C78 pad 2: GND -> Net-(U4C--)
- C79 pad 1: Net-(U4D-+) -> Net-(U4C-+)
- C79 pad 2: /Codec and audio IO/Audio input/RB -> /Codec and audio IO/Audio input/TB
- IC3 pad 3: OUTA_SW -> GND
- IC3 pad 4: OUTB_SW -> GND
- IC3 pad 51: EXP_SW_3 -> GND
- IC3 pad 52: EXP_SW_2 -> GND
- IC3 pad 53: EXP_SW_1 -> GND
- IC3 pad 54: EXP_SW_0 -> GND
- IC4 pad 14: Net-(IC4-PA4) -> GND
- IC4 pad 15: Net-(IC4-PA5) -> GND
- IC4 pad 16: Net-(IC4-PA6) -> GND
- IC4 pad 17: Net-(IC4-PA7) -> DISPLAY_GPIO_4
- IC4 pad 18: Net-(IC4-PB0) -> DISPLAY_GPIO_3
- IC4 pad 19: Net-(IC4-PB1) -> DISPLAY_GPIO_2
- IC4 pad 20: Net-(IC4-PB2) -> DISPLAY_GPIO_1
- IC4 pad 21: Net-(IC4-PB10) -> DISPLAY_GPIO_0
- IC4 pad 29: DISPLAY_GPIO_0 -> Net-(IC4-PA8)
- IC4 pad 30: DISPLAY_GPIO_1 -> Net-(IC4-PA9)
- IC4 pad 31: DISPLAY_GPIO_2 -> Net-(IC4-PA10)
- IC4 pad 32: DISPLAY_GPIO_3 -> Net-(IC4-PA11)
- IC4 pad 33: DISPLAY_GPIO_4 -> Net-(IC4-PA12)
- J10 pad 2: EXP_SW_2 -> EXP_2
- J10 pad 3: EXP_2 -> +3V3
- J11 pad 2: EXP_SW_3 -> EXP_3
- J11 pad 3: EXP_3 -> +3V3
- J12 pad 1: +3V3 -> MCU2_NRST
- J12 pad 2: ENC_SW -> MCU2_DEB_SWDIO
- J12 pad 3: ENC_B -> GND
- J12 pad 4: GND -> MCU2_DEB_SWCLK
- J12 pad 5: ENC_A -> +3V3
- J13 pad 1: MCU2_NRST -> MCU1_NRST
- J13 pad 2: MCU2_DEB_SWDIO -> MCU1_DEB_SWDIO
- J13 pad 4: MCU2_DEB_SWCLK -> MCU1_DEB_SWCLK
- J14 pad 1: MCU1_NRST -> Net-(IC4-PA12)
- J14 pad 2: MCU1_DEB_SWDIO -> Net-(IC4-PA11)
- J14 pad 3: GND -> Net-(IC4-PA10)
- J14 pad 4: MCU1_DEB_SWCLK -> Net-(IC4-PA9)
- J14 pad 5: +3V3 -> Net-(IC4-PA8)
- J17 pad R: /Codec and audio IO/Audio ouput/RA -> /Codec and audio IO/Audio input/RA
- J17 pad SN: Net-(J17-PadSN) -> GND
- J17 pad T: /Codec and audio IO/Audio ouput/TA -> /Codec and audio IO/Audio input/TA
- J18 pad R: /Codec and audio IO/Audio ouput/RB -> /Codec and audio IO/Audio input/RB
- J18 pad SN: Net-(J18-PadSN) -> GND
- J18 pad T: /Codec and audio IO/Audio ouput/TB -> /Codec and audio IO/Audio input/TB
- J7 pad 2: EXP_SW_0 -> +3V3
- J7 pad 3: EXP_0 -> DISPLAY_SPI_SCK
- J7 pad 4: +3V3 -> DISPLAY_SPI_MOSI
- J8 pad 2: +3V3 -> EXP_1
- J8 pad 3: DISPLAY_SPI_SCK -> +3V3
- R10 pad 1: Net-(J6-CC1) -> GND
- R10 pad 2: GND -> EXP_1
- R11 pad 1: GND -> Net-(J9-CC2)
- R11 pad 2: EXP_0 -> GND
- R12 pad 1: +3V3 -> Net-(J9-CC1)
- R12 pad 2: EXP_SW_0 -> GND
- R13 pad 2: EXP_1 -> EXP_2
- R14 pad 1: +3V3 -> GND
- R14 pad 2: EXP_SW_1 -> EXP_3
- R15 pad 1: GND -> +3V3
- R15 pad 2: EXP_2 -> ENC_B
- R16 pad 2: EXP_SW_2 -> ENC_A
- R17 pad 1: GND -> ENC_SW
- R17 pad 2: EXP_3 -> GND
- R19 pad 1: +3V3 -> LED_0_RD
- R19 pad 2: ENC_B -> Net-(D5-A)
- R20 pad 1: +3V3 -> LED_1_RD
- R20 pad 2: ENC_A -> Net-(D7-A)
- R21 pad 1: ENC_SW -> LED_2_QB
- R21 pad 2: GND -> Net-(D10-A)
- R22 pad 1: +3V3 -> LED_3_QB
- R22 pad 2: Net-(D3-A) -> Net-(D11-A)
- R23 pad 1: LED_0_RD -> LED_4_QB
- R23 pad 2: Net-(D5-A) -> Net-(D13-A)
- R24 pad 1: LED_1_RD -> LED_5_QB
- R24 pad 2: Net-(D7-A) -> Net-(D15-A)
- R25 pad 1: LED_2_QB -> BTN_0_J
- R25 pad 2: Net-(D10-A) -> GND
- R26 pad 1: LED_3_QB -> BTN_1_J
- R26 pad 2: Net-(D11-A) -> GND
- R27 pad 1: LED_4_QB -> BTN_2_J
- R27 pad 2: Net-(D13-A) -> GND
- R28 pad 1: LED_5_QB -> BTN_3_J
- R28 pad 2: Net-(D15-A) -> GND
- R29 pad 1: BTN_0_J -> BTN_4_J
- R30 pad 1: BTN_1_J -> BTN_5_QB
- R31 pad 1: BTN_2_J -> BTN_6_QB
- R32 pad 1: BTN_3_J -> BTN_7_QB
- R33 pad 1: BTN_4_J -> BTN_8_QB
- R34 pad 1: BTN_5_QB -> BTN_9_J
- R35 pad 1: BTN_6_QB -> GND
- R35 pad 2: GND -> Net-(IC3-BOOT0)
- R36 pad 1: BTN_7_QB -> GND
- R36 pad 2: GND -> Net-(IC4-BOOT0)
- R37 pad 1: BTN_8_QB -> +3V3
- R37 pad 2: GND -> MCU2_NRST
- R38 pad 1: BTN_9_J -> +3V3
- R38 pad 2: GND -> MCU1_NRST
- R39 pad 1: GND -> USART_2_TO_1
- R39 pad 2: Net-(IC3-BOOT0) -> Net-(D17-A)
- R40 pad 1: GND -> USART_1_TO_2
- R40 pad 2: Net-(IC4-BOOT0) -> Net-(D18-A)
- R41 pad 1: +3V3 -> Net-(U3A--)
- R41 pad 2: MCU2_NRST -> Net-(C57-Pad2)
- R42 pad 1: +3V3 -> Net-(C56-Pad1)
- R42 pad 2: MCU1_NRST -> Net-(C57-Pad2)
- R43 pad 1: USART_2_TO_1 -> Net-(C57-Pad1)
- R43 pad 2: Net-(D17-A) -> /Codec and audio IO/Audio ouput/TA
- R44 pad 1: USART_1_TO_2 -> Net-(C57-Pad1)
- R44 pad 2: Net-(D18-A) -> GND
- R45 pad 1: Net-(U3A--) -> Net-(U3B--)
- R45 pad 2: Net-(C57-Pad2) -> Net-(C61-Pad2)
- R46 pad 1: Net-(C56-Pad1) -> GND
- R46 pad 2: Net-(C57-Pad2) -> Net-(C58-Pad2)
- R47 pad 1: Net-(C57-Pad1) -> Net-(C60-Pad1)
- R47 pad 2: /Codec and audio IO/Audio ouput/TA -> Net-(C61-Pad2)
- R48 pad 1: Net-(C57-Pad1) -> Net-(C58-Pad2)
- R48 pad 2: GND -> /Codec and audio IO/Audio ouput/RA
- R49 pad 1: Net-(U3B--) -> Net-(U3C--)
- R49 pad 2: Net-(C61-Pad2) -> Net-(C65-Pad2)
- R50 pad 1: GND -> Net-(C62-Pad1)
- R50 pad 2: Net-(C58-Pad2) -> Net-(C65-Pad2)
- R51 pad 1: Net-(C60-Pad1) -> Net-(C65-Pad1)
- R51 pad 2: Net-(C61-Pad2) -> /Codec and audio IO/Audio ouput/TB
- R52 pad 1: Net-(C58-Pad2) -> Net-(C65-Pad1)
- R52 pad 2: /Codec and audio IO/Audio ouput/RA -> GND
- R53 pad 1: Net-(U3C--) -> Net-(U3D--)
- R53 pad 2: Net-(C63-Pad2) -> Net-(C69-Pad2)
- R54 pad 1: Net-(C62-Pad1) -> GND
- R54 pad 2: Net-(C63-Pad2) -> Net-(C66-Pad2)
- R55 pad 1: Net-(C63-Pad1) -> Net-(C68-Pad1)
- R55 pad 2: /Codec and audio IO/Audio ouput/TB -> Net-(C69-Pad2)
- R56 pad 1: Net-(C63-Pad1) -> Net-(C66-Pad2)
- R56 pad 2: GND -> /Codec and audio IO/Audio ouput/RB
- R57 pad 1: Net-(U3D--) -> Net-(U4A--)
- R57 pad 2: Net-(C67-Pad2) -> CODEC_INA+
- R58 pad 1: GND -> Net-(C70-Pad1)
- R58 pad 2: Net-(C64-Pad2) -> CODEC_INA+
- R59 pad 1: Net-(C66-Pad1) -> Net-(U4A-+)
- R59 pad 2: Net-(C67-Pad2) -> VCOM
- R60 pad 1: Net-(C64-Pad2) -> Net-(U4B--)
- R60 pad 2: /Codec and audio IO/Audio ouput/RB -> CODEC_INA-
- R61 pad 1: Net-(J17-PadSN) -> VCOM
- R61 pad 2: +3V3 -> Net-(U4B-+)
- R62 pad 1: Net-(J17-PadSN) -> Net-(C75-Pad1)
- R62 pad 2: OUTA_SW -> CODEC_INA-
- R63 pad 1: Net-(J17-PadSN) -> Net-(U4C--)
- R63 pad 2: GND -> CODEC_INB+
- R64 pad 1: Net-(J18-PadSN) -> Net-(C78-Pad1)
- R64 pad 2: +3V3 -> CODEC_INB+
- R65 pad 1: Net-(J18-PadSN) -> Net-(U4C-+)
- R65 pad 2: OUTB_SW -> VCOM
- R66 pad 1: Net-(J18-PadSN) -> Net-(U4D--)
- R66 pad 2: GND -> CODEC_INB-
- R67 pad 1: Net-(U4A--) -> VCOM
- R67 pad 2: CODEC_INA+ -> Net-(U4D-+)
- R68 pad 1: Net-(C68-Pad1) -> Net-(C81-Pad1)
- R68 pad 2: CODEC_INA+ -> CODEC_INB-
- R7 pad 1: VBUS -> GND
- R7 pad 2: VBUS_SENSE -> EXP_0
- R8 pad 1: VBUS_SENSE -> VBUS
- R8 pad 2: GND -> VBUS_SENSE
- R9 pad 1: Net-(J6-CC2) -> VBUS_SENSE
- SW10 pad 1: BTN_9_J -> BTN_8_QB
- SW2 pad 1: BTN_1_J -> BTN_0_J
- SW3 pad 1: BTN_2_J -> BTN_1_J
- SW4 pad 1: BTN_3_J -> BTN_2_J
- SW5 pad 1: BTN_4_J -> BTN_3_J
- SW6 pad 1: BTN_5_QB -> BTN_4_J
- SW7 pad 1: BTN_6_QB -> BTN_5_QB
- SW8 pad 1: BTN_7_QB -> BTN_6_QB
- SW9 pad 1: BTN_8_QB -> BTN_7_QB
- U3 pad 14: Net-(C66-Pad1) -> Net-(C68-Pad1)
- U4 pad 1: Net-(C68-Pad1) -> Net-(C70-Pad1)
- U4 pad 14: Net-(C77-Pad1) -> Net-(C81-Pad1)
- U4 pad 7: Net-(C71-Pad1) -> Net-(C75-Pad1)
- U4 pad 8: Net-(C74-Pad1) -> Net-(C78-Pad1)
Routing:
- net VCOM: track 115.4 -> 0.00 mm, vias 1 -> 0
- net OUTB_SW: track 111.7 -> 0.00 mm, vias 1 -> 0
- net +3V3: track 144.7 -> 36.0 mm, vias 20 -> 0
- net OUTA_SW: track 91.0 -> 0.00 mm, vias 1 -> 0
- net BTN_5_QB: track 77.2 -> 0.00 mm
- net USB_D+: track 75.3 -> 0.00 mm, vias 2 -> 0
- net USB_D-: track 75.2 -> 0.00 mm, vias 2 -> 0
- net EXP_SW_3: track 72.6 -> 0.00 mm, vias 1 -> 0
- net VBUS_SENSE: track 71.9 -> 0.00 mm, vias 2 -> 0
- net INB_SW: track 70.3 -> 0.00 mm, vias 1 -> 0
- net BTN_6_QB: track 69.8 -> 0.00 mm
- net LED_0_RD: track 68.7 -> 0.00 mm
- net BTN_9_J: track 68.3 -> 0.00 mm
- net LED_2_QB: track 64.3 -> 0.00 mm
- net BTN_7_QB: track 63.8 -> 0.00 mm
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- added copper zone on In1.Cu, net (none)
- added copper zone on In2.Cu, net (none)
- added copper zone on B.Cu, net +3.3VA
- added copper zone on B.Cu, net +3V3
- added copper zone on B.Cu, net VBUS
- removed copper zone on In1.Cu, net +3.3VA
- removed copper zone on In1.Cu, net +3V3
- removed copper zone on B.Cu, net GND
- removed copper zone on F.Cu, net GND
- removed copper zone on In1.Cu, net GND
- removed copper zone on In2.Cu, net GND
- removed copper zone on F.Cu, net VBUS
Other:
- board size 135 x 80.5 mm -> 180 x 70 mm
- board text removed: "busy-toad rev. A"

Commit message: layed components down
Parts:
- C1, C10, C11, C12, C13, C14, C2, C27, C3, C30, C31, C33, C34, C35, C36, C4, C5, C6, C7, C8, C9, D1, D2, IC1, J9, L1, R1, R10, R11, R12, R13, R14, R15, R16, R17, R7, R8, R9, RV1, RV2, RV3, U1, U2: moved to F.Cu
- moved R18 354.1 mm to (234.2, 70.5)
- moved D4 340.5 mm to (234.2, 75.3), turned to 90 degrees
- moved D3 330.3 mm to (235.5, 73.5), turned to 90 degrees
- moved R19 311.9 mm to (193.0, 113.1), turned to 90 degrees
- moved D6 305.0 mm to (197.8, 113.8), turned to 180 degrees
- moved D5 290.1 mm to (196.0, 112.5), turned to 180 degrees
- moved R20 215.1 mm to (100.7, 87.2), turned to 180 degrees
- moved D8 207.5 mm to (101.0, 82.4), turned to -90 degrees
- moved D7 194.5 mm to (99.8, 84.2), turned to -90 degrees
- moved C66 103.1 mm to (106.0, 65.1), turned to 90 degrees
- moved R54 99.3 mm to (125.9, 69.0), turned to 180 degrees
- moved C67 97.7 mm to (125.9, 70.5), turned to 180 degrees
- moved R56 96.8 mm to (104.5, 65.1), turned to 90 degrees
- moved C69 93.6 mm to (120.5, 71.0), turned to 90 degrees
- moved R52 92.8 mm to (125.9, 72.0)
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Routing:
- added copper zone on F.Cu, net +3.3VA
- added copper zone on F.Cu, net +3V3
- added copper zone on F.Cu, net VBUS
- removed copper zone on B.Cu, net +3.3VA
- removed copper zone on B.Cu, net +3V3
- removed copper zone on B.Cu, net VBUS

Commit message: routing stuff
Parts:
- moved J4 11.6 mm to (158.2, 88.8)
- moved R3 4.48 mm to (151.0, 86.8)
- moved R4 4.48 mm to (152.5, 86.8)
- moved C81 4.14 mm to (147.0, 75.5), turned to 90 degrees
- moved R66 4.14 mm to (144.0, 75.5), turned to 90 degrees
- moved R68 4.14 mm to (145.5, 75.5), turned to 90 degrees
- moved C78 3.86 mm to (147.0, 71.5), turned to -90 degrees
- moved R63 3.86 mm to (144.0, 71.5), turned to -90 degrees
- moved R64 3.86 mm to (145.5, 71.5), turned to -90 degrees
- moved C11 3.09 mm to (215.5, 75.0), turned to 0 degrees
- moved C14 3.04 mm to (202.0, 75.0), turned to 0 degrees
- moved C13 1.79 mm to (202.0, 73.0), turned to 180 degrees
- moved C10 1.60 mm to (215.5, 73.0), turned to 180 degrees
- moved C1 1.56 mm to (226.5, 71.8)
- moved C2 1.56 mm to (224.5, 71.8)
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Connections:
- IC4 pad 17: DISPLAY_GPIO_4 -> DISPLAY_GPIO_0
- IC4 pad 18: DISPLAY_GPIO_3 -> DISPLAY_GPIO_1
- IC4 pad 20: DISPLAY_GPIO_1 -> DISPLAY_GPIO_3
- IC4 pad 21: DISPLAY_GPIO_0 -> DISPLAY_GPIO_4
Routing:
- net VCOM: track 0.00 -> 123.7 mm, vias 0 -> 6
- net GND: track 61.8 -> 148.8 mm, vias 21 -> 69
- net +5V: track 0.00 -> 48.0 mm
- net CODEC_INA+: track 0.00 -> 41.8 mm
- net Net-(C65-Pad1): track 0.00 -> 40.0 mm
- net MCU2_DEB_SWDIO: track 0.00 -> 35.1 mm
- net CODEC_INA-: track 0.00 -> 32.3 mm, vias 0 -> 1
- net Net-(C66-Pad2): track 0.00 -> 31.8 mm
- net DISPLAY_GPIO_4: track 0.00 -> 31.5 mm, vias 0 -> 1
- net DISPLAY_GPIO_3: track 0.00 -> 31.1 mm, vias 0 -> 1
- net DISPLAY_GPIO_0: track 0.00 -> 30.9 mm, vias 0 -> 1
- net DISPLAY_GPIO_2: track 0.00 -> 30.6 mm, vias 0 -> 1
- net DISPLAY_GPIO_1: track 0.00 -> 30.3 mm, vias 0 -> 1
- net MCU2_NRST: track 0.00 -> 28.3 mm
- net Net-(C58-Pad2): track 0.00 -> 28.0 mm
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- added copper zone on F.Cu, net +5V
- added copper zone on F.Cu, net GND
- added copper zone on In1.Cu, net GND
- added copper zone on In2.Cu, net GND
- added copper zone on F.Cu, net Net-(D1-A)
- added copper zone on F.Cu, net Net-(IC1-INTVCC)
- added copper zone on F.Cu, net Net-(IC1-RUN)
- added copper zone on F.Cu, net Net-(IC1-SW)
- removed copper zone on In1.Cu, net (none)
- removed copper zone on In2.Cu, net (none)

Commit message: almost there
Parts:
- moved R39 33.9 mm to (124.1, 123.2)
- moved R40 33.9 mm to (124.1, 125.8)
- moved R2 32.8 mm to (144.2, 96.2), turned to 135 degrees
- moved D17 32.7 mm to (119.7, 123.3)
- moved D18 32.7 mm to (119.7, 125.9)
- moved J4 12.3 mm to (146.8, 93.2)
- moved R24 7.27 mm to (225.8, 111.0), turned to -90 degrees
- moved J13 4.32 mm to (203.8, 92.8)
- moved H4 3.25 mm to (128.2, 115.0)
- moved R3 1.77 mm to (150.8, 85.0)
- moved R4 1.77 mm to (152.2, 85.0)
- moved C46 1.37 mm to (114.5, 96.2)
- moved C47 1.37 mm to (116.0, 96.2)
- moved D5 1.25 mm to (196.0, 113.8)
- moved D6 1.25 mm to (197.8, 115.0)
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Routing:
- net +3V3: track 58.9 -> 551.9 mm, vias 9 -> 28
- net ENC_SW: track 0.00 -> 165.6 mm, vias 0 -> 3
- net ENC_B: track 0.00 -> 131.6 mm, vias 0 -> 4
- net ENC_A: track 0.00 -> 123.0 mm, vias 0 -> 4
- net +3.3VA: track 25.1 -> 125.0 mm
- net AUX_2_TO_1: track 0.00 -> 98.7 mm
- net AUX_1_TO_2: track 0.00 -> 97.7 mm
- net USART_2_TO_1: track 0.00 -> 96.7 mm
- net USART_1_TO_2: track 0.00 -> 96.6 mm
- net BTN_8_QB: track 0.00 -> 79.2 mm, vias 0 -> 2
- net BTN_5_QB: track 0.00 -> 76.6 mm, vias 0 -> 2
- net BTN_6_QB: track 0.00 -> 75.7 mm, vias 0 -> 2
- net VBUS_SENSE: track 1.62 -> 75.4 mm, vias 0 -> 2
- net BTN_7_QB: track 0.00 -> 71.7 mm, vias 0 -> 2
- net USB_D-: track 5.76 -> 76.4 mm, vias 0 -> 2
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- added copper zone on B.Cu, net +3.3VA
- added copper zone on B.Cu, net +3V3
Other:
- outline, holes or cut-outs redrawn

Commit message: maybe???
Parts:
- added G***: LOGO, LOGO, F.Cu at (171.0, 86.0)
- moved D18 28.4 mm to (132.5, 100.5), turned to -135 degrees
- moved D17 25.6 mm to (134.0, 102.0), turned to -135 degrees
- moved R40 23.2 mm to (129.8, 103.2), turned to 45 degrees
- moved R39 19.2 mm to (130.8, 105.2), turned to 45 degrees
- moved C70 4.00 mm to (157.0, 71.5), turned to -90 degrees
- moved C75 4.00 mm to (157.0, 75.5), turned to 90 degrees
- moved C78 4.00 mm to (147.0, 75.5), turned to 90 degrees
- moved C81 4.00 mm to (147.0, 71.5), turned to -90 degrees
- moved R57 4.00 mm to (160.0, 71.5), turned to -90 degrees
- moved R58 4.00 mm to (158.5, 71.5), turned to -90 degrees
- moved R60 4.00 mm to (160.0, 75.5), turned to 90 degrees
- moved R62 4.00 mm to (158.5, 75.5), turned to 90 degrees
- moved R63 4.00 mm to (144.0, 75.5), turned to 90 degrees
- moved R64 4.00 mm to (145.5, 75.5), turned to 90 degrees
- moved R66 4.00 mm to (144.0, 71.5), turned to -90 degrees
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Connections:
- C70 pad 2: Net-(U4A--) -> Net-(U4B--)
- C71 pad 1: Net-(U4A-+) -> Net-(U4B-+)
- C75 pad 2: Net-(U4B--) -> Net-(U4A--)
- C77 pad 1: Net-(U4B-+) -> Net-(U4A-+)
- C78 pad 2: Net-(U4C--) -> Net-(U4D--)
- C79 pad 1: Net-(U4C-+) -> Net-(U4D-+)
- C81 pad 2: Net-(U4D--) -> Net-(U4C--)
- C83 pad 1: Net-(U4D-+) -> Net-(U4C-+)
- R57 pad 1: Net-(U4A--) -> Net-(U4B--)
- R59 pad 1: Net-(U4A-+) -> Net-(U4B-+)
- R60 pad 1: Net-(U4B--) -> Net-(U4A--)
- R61 pad 2: Net-(U4B-+) -> Net-(U4A-+)
- R63 pad 1: Net-(U4C--) -> Net-(U4D--)
- R65 pad 1: Net-(U4C-+) -> Net-(U4D-+)
- R66 pad 1: Net-(U4D--) -> Net-(U4C--)
- R67 pad 2: Net-(U4D-+) -> Net-(U4C-+)
- U4 pad 1: Net-(C70-Pad1) -> Net-(C75-Pad1)
- U4 pad 14: Net-(C81-Pad1) -> Net-(C78-Pad1)
- U4 pad 7: Net-(C75-Pad1) -> Net-(C70-Pad1)
- U4 pad 8: Net-(C78-Pad1) -> Net-(C81-Pad1)
Routing:
- net +3V3: track 551.9 -> 656.7 mm, vias 28 -> 29
- net BTN_0_J: track 0.00 -> 66.1 mm, vias 0 -> 1
- net BTN_2_J: track 0.00 -> 65.4 mm, vias 0 -> 1
- net BTN_9_J: track 0.00 -> 52.0 mm, vias 0 -> 1
- net BTN_1_J: track 0.00 -> 50.3 mm, vias 0 -> 1
- net BTN_3_J: track 0.00 -> 48.3 mm, vias 0 -> 1
- net +3.3VA: track 125.0 -> 170.2 mm, vias 5 -> 7
- net BTN_4_J: track 0.00 -> 43.5 mm, vias 0 -> 1
- net CODEC_OUTA+: track 0.00 -> 37.7 mm, vias 0 -> 2
- net CODEC_OUTA-: track 0.00 -> 34.0 mm
- net GND: track 168.3 -> 202.0 mm, vias 125 -> 171
- net CODEC_OUTB-: track 0.00 -> 31.3 mm, vias 0 -> 2
- net CODEC_OUTB+: track 0.00 -> 30.2 mm
- net MCU2_DEB_SWCLK: track 0.00 -> 21.9 mm, vias 0 -> 2
- net CODEC_INB-: track 3.59 -> 24.7 mm
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Other:
- board text added: "+ -"
- board text added: "1→2 2→1"
- board text added: "3V3 CLK GND DIO NRST"
- board text added: "BUSY TOAD"
- board text added: "EXP0"
- board text added: "EXP1"
- board text added: "EXP2"
- board text added: "EXP3"
- board text added: "G. Ascari Rev. A"
- board text added: "HP"
- board text added: "IN.A"
- board text added: "IN.B"
- board text added: "L R GND"
- board text added: "LED1"
- board text added: "LED2"
- board text added: "MCU 1"
- board text added: "MCU 2"
- board text added: "NRST DIO GND CLK 3V3"
- board text added: "OUT.A"
- board text added: "OUT.B"
- board text added: "PWR"
- board text added: "UNUSED"
