File: pcb/bt_pcb/bt_pcb.kicad_sch (KiCad schematic)
At the start: 6 parts

Commit message: aaaaaaa
Parts:
- renumbered H4 to H2, H2 to H3, H5 to H4, H3 to H5

Commit message: schematic rev b finish?
Parts:
- renumbered H3 to H2, H5 to H3, H2 to H4, H4 to H5
Changed lines of the file:
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@@
 		(dnp no)
 		(fields_autoplaced yes)
-		(property "Reference" "#PWR02"
+		(property "Reference" "#PWR04"
 			(at 38.1 187.96 0)
 			(hide yes)
@@
 			(project "bt_pcb"
 				(path "/eb787481-08cd-41a4-a128-173fa6227c32"
-					(reference "#PWR02")
+					(reference "#PWR04")
 					(unit 1)
 				)
@@
 		(dnp no)
 		(fields_autoplaced yes)
-		(property "Reference" "H2"
+		(property "Reference" "H4"
 			(at 40.64 176.5299 0)
 			(show_name no)
@@
 			(project "bt_pcb"
 				(path "/eb787481-08cd-41a4-a128-173fa6227c32"
-					(reference "H2")
+					(reference "H4")
 					(unit 1)
 				)
@@
 		(dnp no)
 		(fields_autoplaced yes)
-		(property "Reference" "H4"
+		(property "Reference" "H5"
 			(at 66.04 176.5299 0)
 			(show_name no)
@@
 			(project "bt_pcb"
 				(path "/eb787481-08cd-41a4-a128-173fa6227c32"
-					(reference "H4")
+					(reference "H5")
 					(unit 1)
 				)
@@
 		(dnp no)
 		(fields_autoplaced yes)
-		(property "Reference" "#PWR05"
+		(property "Reference" "#PWR03"
 			(at 88.9 175.26 0)
 			(hide yes)
@@
 			(project "bt_pcb"
 				(path "/eb787481-08cd-41a4-a128-173fa6227c32"
-					(reference "#PWR05")
+					(reference "#PWR03")
 					(unit 1)
 				)
@@
 		(dnp no)
 		(fields_autoplaced yes)
-		(property "Reference" "H3"
+		(property "Reference" "H2"
 			(at 66.04 163.8299 0)
 			(show_name no)
@@
 			(project "bt_pcb"
 				(path "/eb787481-08cd-41a4-a128-173fa6227c32"
-					(reference "H3")
+					(reference "H2")
 					(unit 1)
 				)
@@
 		(dnp no)
 		(fields_autoplaced yes)
-		(property "Reference" "H5"
+		(property "Reference" "H3"
 			(at 91.44 163.8299 0)
 			(show_name no)
@@
 			(project "bt_pcb"
 				(path "/eb787481-08cd-41a4-a128-173fa6227c32"
-					(reference "H5")
+					(reference "H3")
 					(unit 1)
 				)
@@
 		(dnp no)
 		(fields_autoplaced yes)
-		(property "Reference" "#PWR04"
+		(property "Reference" "#PWR05"
 			(at 63.5 187.96 0)
 			(hide yes)
@@
 			(project "bt_pcb"
 				(path "/eb787481-08cd-41a4-a128-173fa6227c32"
-					(reference "#PWR04")
+					(reference "#PWR05")
 					(unit 1)
 				)
@@
 		(dnp no)
 		(fields_autoplaced yes)
-		(property "Reference" "#PWR03"
+		(property "Reference" "#PWR02"
 			(at 63.5 175.26 0)
 			(hide yes)
@@
 			(project "bt_pcb"
 				(path "/eb787481-08cd-41a4-a128-173fa6227c32"
-					(reference "#PWR03")
-					(unit 1)
-				)
+					(reference "#PWR02")
+					(unit 1)
+				)
