File: pcb/bt_pcb/audio_input.kicad_sch (KiCad schematic)
At the start: 29 parts, among them J16 ReanNYS216G, J17 ReanNYS216G, U4 MCP6004

Commit message: seeing the end of the tunnel
Parts:
- J17: renamed from J16; now not fitted
- J18: renamed from J17; now not fitted
Changed lines of the file:
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@@
 		(dnp no)
 		(fields_autoplaced yes)
-		(property "Reference" "#PWR0138"
+		(property "Reference" "#PWR0139"
 			(at 71.12 48.26 0)
 			(effects
@@
 			(project "bt_pcb"
 				(path "/eb787481-08cd-41a4-a128-173fa6227c32/4ada0139-8712-47ce-9d4c-ab8fef312f7b/aa7abd67-f1bd-4ae8-bc05-bae360f4c6c7"
-					(reference "#PWR0138")
+					(reference "#PWR0139")
 					(unit 1)
 				)
@@
 			)
 		)
-		(property "Description" ""
+		(property "Description" "AUDIO"
 			(at 132.08 48.26 0)
 			(effects
@@
 					(size 1.27 1.27)
 				)
+				(hide yes)
 			)
 		)
@@
 			)
 		)
-		(property "Description" ""
+		(property "Description" "AUDIO"
 			(at 161.29 20.32 0)
 			(effects
@@
 					(size 1.27 1.27)
 				)
+				(hide yes)
 			)
 		)
@@
 			)
 		)
-		(property "Description" ""
+		(property "Description" "AUDIO"
 			(at 160.02 83.82 0)
 			(effects
@@
 					(size 1.27 1.27)
 				)
+				(hide yes)
 			)
 		)
@@
 			)
 		)
-		(property "Description" ""
+		(property "Description" "AUDIO"
 			(at 113.03 33.02 0)
 			(effects
@@
 					(size 1.27 1.27)
 				)
+				(hide yes)
 			)
 		)
@@
 		(in_bom yes)
 		(on_board yes)
-		(dnp no)
-		(property "Reference" "J17"
+		(dnp yes)
+		(property "Reference" "J18"
 			(at 122.555 186.69 0)
 			(effects
@@
 			(project "bt_pcb"
 				(path "/eb787481-08cd-41a4-a128-173fa6227c32/4ada0139-8712-47ce-9d4c-ab8fef312f7b/aa7abd67-f1bd-4ae8-bc05-bae360f4c6c7"
-					(reference "J17")
+					(reference "J18")
 					(unit 1)
 				)
@@
 		(dnp no)
 		(fields_autoplaced yes)
-		(property "Reference" "#PWR0140"
+		(property "Reference" "#PWR0141"
 			(at 130.81 121.92 0)
 			(effects
@@
 			(project "bt_pcb"
 				(path "/eb787481-08cd-41a4-a128-173fa6227c32/4ada0139-8712-47ce-9d4c-ab8fef312f7b/aa7abd67-f1bd-4ae8-bc05-bae360f4c6c7"
-					(reference "#PWR0140")
+					(reference "#PWR0141")
 					(unit 1)
 				)
@@
 		(dnp no)
 		(fields_autoplaced yes)
-		(property "Reference" "#PWR0141"
+		(property "Reference" "#PWR0142"
 			(at 88.9 160.02 0)
 			(effects
@@
 			(project "bt_pcb"
 				(path "/eb787481-08cd-41a4-a128-173fa6227c32/4ada0139-8712-47ce-9d4c-ab8fef312f7b/aa7abd67-f1bd-4ae8-bc05-bae360f4c6c7"
-					(reference "#PWR0141")
+					(reference "#PWR0142")
 					(unit 1)
 				)
@@
 			)
 		)
-		(property "Description" ""
+		(property "Description" "AUDIO"
 			(at 113.03 123.19 0)
 			(effects
@@
 					(size 1.27 1.27)
 				)
+				(hide yes)
 			)
 		)
@@
 		(in_bom yes)
 		(on_board yes)
-		(dnp no)
-		(property "Reference" "J16"
+		(dnp yes)
+		(property "Reference" "J17"
 			(at 79.375 157.48 0)
 			(effects
@@
 			(project "bt_pcb"
 				(path "/eb787481-08cd-41a4-a128-173fa6227c32/4ada0139-8712-47ce-9d4c-ab8fef312f7b/aa7abd67-f1bd-4ae8-bc05-bae360f4c6c7"
-					(reference "J16")
+					(reference "J17")
 					(unit 1)
 				)
@@
 			)
 		)
-		(property "Description" ""
+		(property "Description" "AUDIO"
 			(at 179.07 106.68 0)
 			(effects
@@
 					(size 1.27 1.27)
 				)
+				(hide yes)
 			)
 		)
@@
 			)
 		)
-		(property "Description" ""
+		(property "Description" "AUDIO"
 			(at 160.02 46.99 0)
 			(effects
@@
 					(size 1.27 1.27)
 				)
+				(hide yes)
 			)
 		)
@@
 			)
 		)
-		(property "Description" ""
+		(property "Description" "AUDIO"
 			(at 113.03 59.69 0)
 			(effects
@@
 					(size 1.27 1.27)
 				)
+				(hide yes)
 			)
 		)
@@
 		(dnp no)
 		(fields_autoplaced yes)
-		(property "Reference" "#PWR0139"
+		(property "Reference" "#PWR0140"
 			(at 132.08 58.42 0)
 			(effects
@@
 			(project "bt_pcb"
 				(path "/eb787481-08cd-41a4-a128-173fa6227c32/4ada0139-8712-47ce-9d4c-ab8fef312f7b/aa7abd67-f1bd-4ae8-bc05-bae360f4c6c7"
-					(reference "#PWR0139")
+					(reference "#PWR0140")
 					(unit 1)
 				)
@@
 		(dnp no)
 		(fields_autoplaced yes)
-		(property "Reference" "#PWR0137"
+		(property "Reference" "#PWR0138"
 			(at 71.12 30.48 0)
 			(effects
@@
 			(project "bt_pcb"
 				(path "/eb787481-08cd-41a4-a128-173fa6227c32/4ada0139-8712-47ce-9d4c-ab8fef312f7b/aa7abd67-f1bd-4ae8-bc05-bae360f4c6c7"
-					(reference "#PWR0137")
+					(reference "#PWR0138")
 					(unit 1)
 				)
@@
 			)
 		)
-		(property "Description" ""
+		(property "Description" "AUDIO"
 			(at 113.03 96.52 0)
 			(effects
@@
 					(size 1.27 1.27)
 				)
+				(hide yes)
 			)
 		)
@@
 			)
 		)
-		(property "Description" ""
+		(property "Description" "APD"
 			(at 49.53 34.29 0)
 			(effects
@@
 					(size 1.27 1.27)
 				)
+				(hide yes)
 			)
 		)
@@
 			)
 		)
-		(property "Description" ""
+		(property "Description" "APD"
 			(at 60.96 34.29 0)
 			(effects
@@
 					(size 1.27 1.27)
 				)
+				(hide yes)
 			)
 		)
@@
 			)
 		)
-		(property "Description" ""
+		(property "Description" "AUDIO"
 			(at 160.02 110.49 0)
 			(effects
@@
 					(size 1.27 1.27)
 				)
+				(hide yes)
 			)
 		)
@@
 			)
 		)
-		(property "Description" ""
+		(property "Description" "AUDIO"
 			(at 130.81 111.76 0)
 			(effects
@@
 					(size 1.27 1.27)
 				)
+				(hide yes)
 			)
 		)
@@
 		(dnp no)
 		(fields_autoplaced yes)
-		(property "Reference" "#PWR0142"
+		(property "Reference" "#PWR0143"
 			(at 132.08 189.23 0)
 			(effects
@@
 			(project "bt_pcb"
 				(path "/eb787481-08cd-41a4-a128-173fa6227c32/4ada0139-8712-47ce-9d4c-ab8fef312f7b/aa7abd67-f1bd-4ae8-bc05-bae360f4c6c7"
-					(reference "#PWR0142")
+					(reference "#PWR0143")
 					(unit 1)
 				)
@@
 			)
 		)
-		(property "Description" ""
+		(property "Description" "AUDIO"
 			(at 179.07 43.18 0)
 			(effects
@@
 					(size 1.27 1.27)
 				)
-			)
-		)
+				(hide yes)
+			)
+		)

Commit message: aaaaaaa
Parts:
- J16: renamed from J17; now fitted
- J17: renamed from J18; now fitted
- renumbered C73 to C78, C74 to C79, C72 to C80, C78 to C81, C80 to C82, C84 to C83, C83 to C84, C77 to C85, C76 to C86, C79 to C87, C82 to C88, C71 to C89, C75 to C90, C81 to C91, R67 to R56, R69 to R57, R61 to R58, R63 to R59, R62 to R60, R64 to R61, R65 to R62, R66 to R63, R68 to R64, R70 to R65, R59 to R66, R60 to R67
Connections:
- net VCOM renamed IN_VMID

Commit message: schematic rev b finish?
Parts:
- renumbered C81 to C100, C87 to C101, C82 to C102, C91 to C103, C88 to C104, C84 to C105, C83 to C106, C89 to C93, C80 to C94, C78 to C95, C79 to C96, C90 to C97, C86 to C98, C85 to C99, R66 to R57, R67 to R58, R58 to R59, R59 to R61, R61 to R62, R62 to R63, R63 to R64, R56 to R65, R64 to R66, R57 to R67, R65 to R68, U4 to U5

Commit message: just need to fix usb
Connections:
- net CODEC_INA+: now also C97.2, R60.2, R62.2; no longer C97.1, R57.2, R58.2
- net CODEC_INA-: now also C97.1, R57.2, R58.2; no longer C97.2, R60.2, R62.2
- net CODEC_INB+: now also C103.2, R66.2, R68.2; no longer C103.1, R63.2, R64.2
- net CODEC_INB-: now also C103.1, R63.2, R64.2; no longer C103.2, R66.2, R68.2
- net RA: now also C94.2; no longer C100.2
- net RB: now also C102.2; no longer C106.2
- net TA: now also C100.2; no longer C94.2
- net TB: now also C106.2; no longer C102.2
Changed lines of the file:
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@@
+		)
+	)
+	(label "RA"
+		(at 107.95 33.02 180)
+		(effects
+			(font
+				(size 1.27 1.27)
+			)
+			(justify right bottom)
 		)
 	)
 	(label "TA"
-		(at 107.95 33.02 180)
-		(effects
-			(font
-				(size 1.27 1.27)
-			)
-			(justify right bottom)
-		)
-	)
-	(label "RA"
 		(at 107.95 59.69 180)
-		(effects
-			(font
-				(size 1.27 1.27)
-			)
-			(justify right bottom)
-		)
-	)
-	(label "RB"
-		(at 106.68 123.19 180)
-		(effects
-			(font
-				(size 1.27 1.27)
-			)
-			(justify right bottom)
-		)
-	)
-	(label "TB"
-		(at 106.68 96.52 180)
 		(effects
 			(font
@@
 		)
 	)
+	(label "TB"
+		(at 106.68 123.19 180)
+		(effects
+			(font
+				(size 1.27 1.27)
+			)
+			(justify right bottom)
+		)
+	)
 	(label "RA"
 		(at 93.98 146.05 0)
@@
 			)
 			(justify left bottom)
+		)
+	)
+	(label "RB"
+		(at 106.68 96.52 180)
+		(effects
+			(font
+				(size 1.27 1.27)
+			)
+			(justify right bottom)
+		)
+	)
+	(global_label "CODEC_INA+"
+		(shape output)
+		(at 184.15 57.15 0)
+		(fields_autoplaced yes)
+		(effects
+			(font
+				(size 1.27 1.27)
+			)
+			(justify left)
+		)
+		(property "Intersheetrefs" "${INTERSHEET_REFS}"
+			(at 198.9886 57.15 0)
+			(hide yes)
+			(show_name no)
+			(do_not_autoplace no)
+			(effects
+				(font
+					(size 1.27 1.27)
+				)
+				(justify left)
+			)
 		)
 	)
@@
 		)
 	)
-	(global_label "CODEC_INA+"
+	(global_label "CODEC_INA-"
 		(shape output)
 		(at 184.15 30.48 0)
@@
 		(property "Intersheetrefs" "${INTERSHEET_REFS}"
 			(at 198.9886 30.48 0)
+			(hide yes)
+			(show_name no)
+			(do_not_autoplace no)
+			(effects
+				(font
+					(size 1.27 1.27)
+				)
+				(justify left)
+			)
+		)
+	)
+	(global_label "CODEC_INB+"
+		(shape output)
+		(at 182.88 120.65 0)
+		(fields_autoplaced yes)
+		(effects
+			(font
+				(size 1.27 1.27)
+			)
+			(justify left)
+		)
+		(property "Intersheetrefs" "${INTERSHEET_REFS}"
+			(at 197.9 120.65 0)
 			(hide yes)
 			(show_name no)
@@
 	(global_label "CODEC_INB-"
 		(shape output)
-		(at 182.88 120.65 0)
-		(fields_autoplaced yes)
-		(effects
-			(font
-				(size 1.27 1.27)
-			)
-			(justify left)
-		)
-		(property "Intersheetrefs" "${INTERSHEET_REFS}"
-			(at 197.9 120.65 0)
-			(hide yes)
-			(show_name no)
-			(do_not_autoplace no)
-			(effects
-				(font
-					(size 1.27 1.27)
-				)
-				(justify left)
-			)
-		)
-	)
-	(global_label "CODEC_INB+"
-		(shape output)
 		(at 182.88 93.98 0)
 		(fields_autoplaced yes)
@@
 			(hide yes)
 			(show_name no)
-			(do_not_autoplace no)
-			(effects
-				(font
-					(size 1.27 1.27)
-				)
-				(justify left)
-			)
-		)
-	)
-	(global_label "CODEC_INA-"
-		(shape output)
-		(at 184.15 57.15 0)
-		(fields_autoplaced yes)
-		(effects
-			(font
-				(size 1.27 1.27)
-			)
-			(justify left)
-		)
-		(property "Intersheetrefs" "${INTERSHEET_REFS}"
-			(at 198.9886 57.15 0)
-			(hide yes)
-			(show_name no)
