File: pcb/bt_pcb/audio_input.kicad_sch (KiCad schematic)
At the start: 29 parts, among them J16 ReanNYS216G, J17 ReanNYS216G, U5 MCP6004

Commit message: sd kind of in
Parts:
- renumbered C99 to C100, C100 to C101, C101 to C102, C102 to C103, C103 to C104, C104 to C105, C105 to C106, C106 to C107, C93 to C94, C94 to C95, C95 to C96, C96 to C97, C97 to C98, C98 to C99, J16 to J17, J17 to J18, R57 to R55, R58 to R56, R59 to R57, R60 to R58, R61 to R59, R62 to R60, R63 to R61, R64 to R62, R65 to R63, R66 to R64, R67 to R65, R68 to R66

Commit message: reb b finished
Parts:
- renumbered C94 to C85, C95 to C86, C96 to C87, C97 to C88, C98 to C89, C99 to C90, C100 to C91, C101 to C92, C102 to C93, C103 to C94, C104 to C95, C105 to C96, C106 to C97, C107 to C98, R55 to R57, R56 to R58, R57 to R59, R58 to R60, R59 to R61, R60 to R62, R61 to R63, R62 to R64, R63 to R65, R64 to R66, R65 to R67, R66 to R68, U5 to U4
