File: pcb/bt_pcb/codec_and_audio.kicad_sch (KiCad schematic)
At the start: 35 parts, among them IC2 TLV320DAC3203IRGER, IC3 CS4282P, J3 Conn_01x03

Commit message: reb b finished
Parts:
- removed C19, C20, C33, C40, C49: 1u, Capacitor_SMD:C_0603_1608Metric_Pad1.08x0.95mm_HandSolder, symbol Device:C
- removed C22, C23, C48: 100n, Capacitor_SMD:C_0603_1608Metric_Pad1.08x0.95mm_HandSolder, symbol Device:C
- removed C43: 10u, Capacitor_SMD:C_0805_2012Metric_Pad1.18x1.45mm_HandSolder, symbol Device:C
- removed C44, C45: 47u, Capacitor_SMD:C_0805_2012Metric_Pad1.18x1.45mm_HandSolder, symbol Device:C
- removed IC2: TLV320DAC3203IRGER, library:QFN50P400X400X100-25N-D, symbol library:TLV320DAC3203IRGER
- added C27, C29, C30: 10u, Capacitor_SMD:C_0805_2012Metric_Pad1.18x1.45mm_HandSolder, symbol Device:C
- added C28, C42: 1u, Capacitor_SMD:C_0603_1608Metric_Pad1.08x0.95mm_HandSolder, symbol Device:C
- added C36: 100n, Capacitor_SMD:C_0603_1608Metric_Pad1.08x0.95mm_HandSolder, symbol Device:C
- added IC3: TAD5242IRGER, library:TAD5242IRGER, symbol library:TAD5242IRGER
- added R4, R5: 22, Resistor_SMD:R_0603_1608Metric_Pad0.98x0.95mm_HandSolder, symbol Device:R
- C34: value 1u -> 100n
- renumbered C18 to C16, C21 to C17, C24 to C18, C25 to C19, C26 to C20, C27 to C21, C28 to C22, C29 to C23, C30 to C24, C31 to C25, C32 to C26, C36 to C31, C37 to C32, C38 to C33, C41 to C37, C42 to C38, C46 to C40, C47 to C41, IC3 to IC2
Connections:
- net +3V3: now also C34.2, C35.1, C39.2, C27.1, C28.1, C29.1, IC3.10 (MD4), IC3.12 (MD5), IC3.23 (AVDD), IC3.6 (IOVDD)
- net GND: now also C34.1, C39.1, C27.2, C28.2, C29.2, C30.2, C36.1, C42.2, IC3.13 (MD0), IC3.14 (VSSA_1), IC3.15 (VSSA_2), IC3.16 (VSSA_3), IC3.17 (VSSA_4), IC3.18 (VSSA_5), IC3.25 (EP), IC3.4 (MD6), IC3.7 (MD1), IC3.8 (MD2), IC3.9 (MD3), IC3.A1 (VSS_1), IC3.A2 (VSS_2), IC3.A3 (VSS_3), IC3.A4 (VSS_4); no longer C34.2, C39.2, J3.3 (Pin_3)
- net HPDAC_I2S_BCK: now also IC3.2 (BCLK)
- net HPDAC_I2S_SDO: now also IC3.5 (DIN)
- net HPDAC_I2S_WS: now also IC3.3 (FSYNC)
- net at J3.2 (Pin_2): now also IC3.21 (OUT2P)
- net at J3.1 (Pin_1): now also R4.2
- net CODEC_I2S_SDI renamed CODEC_I2S_MOSI
- net CODEC_I2S_SDO renamed CODEC_I2S_MISO
- net OUT_VMID: no longer names the net of IC2.32 (DAC_VMID)
- new net: IC3.19 (OUT1M), R4.1
- new net: C30.1, C36.2, IC3.1 (DREG)
- new net: J3.3 (Pin_3), R5.2
- new net: IC3.20 (OUT1P), IC3.22 (OUT2M), R5.1
- new net: C42.1, IC3.24 (VREF)
- new net HPDAC_IRQ: IC3.11 (GPO)
- no-connect marks 12 -> 10
