File: pcb/bt_pcb/audio_output.kicad_sch (KiCad schematic)
At the start: 33 parts, among them J15 ReanNYS216G, J16 ReanNYS216G, U4 MCP6004

Commit message: reb b finished
Parts:
- removed C83, C91: 10n, Capacitor_SMD:C_0603_1608Metric_Pad1.08x0.95mm_HandSolder, symbol Device:C_Polarized
- renumbered C80 to C73, C81 to C74, C82 to C75, C84 to C76, C85 to C77, C86 to C78, C87 to C79, C88 to C80, C89 to C81, C90 to C82, C92 to C83, C93 to C84, R39 to R41, R40 to R42, R41 to R43, R42 to R44, R43 to R45, R44 to R46, R45 to R47, R46 to R48, R47 to R49, R48 to R50, R49 to R51, R50 to R52, R51 to R53, R52 to R54, R53 to R55, R54 to R56, U4 to U3
