File: pcb/bt_pcb/power_supply.kicad_sch (KiCad schematic)
At the start: 28 parts, among them IC1 LV3842XDBVR, J1 Conn_01x02, J2 Barrel_Jack_Switch, U1 TLV76133DCY, U2 TLV76133DCY

Commit message: seeing the end of the tunnel
Other:
- note removed: "SWPA5020S sunlord inductor"
Changed lines of the file:
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@@
 		)
 	)
-	(text "SWPA5020S\n\nsunlord inductor"
-		(exclude_from_sim no)
-		(at 132.588 28.956 0)
-		(effects
-			(font
-				(size 1.27 1.27)
-			)
-		)
-	)
 	(text "Rfbt     88.7k     100k\nRfbb     22.1k   47k||47k\n          5V      5.25V"
 		(exclude_from_sim no)
@@
 			)
 		)
-		(property "Description" ""
+		(property "Description" "DPD"
 			(at 260.35 105.41 0)
 			(effects
@@
 					(size 1.27 1.27)
 				)
+				(hide yes)
 			)
 		)
@@
 			)
 		)
-		(property "Description" ""
+		(property "Description" "POWERSUPPLY"
 			(at 215.9 105.41 0)
 			(effects
@@
 					(size 1.27 1.27)
 				)
+				(hide yes)
 			)
 		)
@@
 			)
 		)
-		(property "Description" ""
+		(property "Description" "POWERSUPPLY"
 			(at 189.23 40.64 0)
 			(effects
@@
 					(size 1.27 1.27)
 				)
+				(hide yes)
 			)
 		)
@@
 			)
 		)
-		(property "Description" ""
+		(property "Description" "POWERSUPPLY"
 			(at 105.41 111.76 0)
 			(effects
@@
 					(size 1.27 1.27)
 				)
+				(hide yes)
 			)
 		)
@@
 			)
 		)
-		(property "Description" ""
+		(property "Description" "POWERSUPPLY"
 			(at 214.63 40.64 0)
 			(effects
@@
 					(size 1.27 1.27)
 				)
+				(hide yes)
 			)
 		)
@@
 			)
 		)
-		(property "Description" ""
+		(property "Description" "POWERSUPPLY"
 			(at 227.33 40.64 0)
 			(effects
@@
 					(size 1.27 1.27)
 				)
+				(hide yes)
 			)
 		)
@@
 			)
 		)
-		(property "Description" ""
+		(property "Description" "POWERSUPPLY"
 			(at 215.9 143.51 0)
 			(effects
@@
 					(size 1.27 1.27)
 				)
+				(hide yes)
 			)
 		)
@@
 			)
 		)
-		(property "Description" ""
+		(property "Description" "POWERSUPPLY"
 			(at 201.93 40.64 0)
 			(effects
@@
 					(size 1.27 1.27)
 				)
+				(hide yes)
 			)
 		)
@@
 			)
 		)
-		(property "Description" ""
+		(property "Description" "DPD"
 			(at 246.38 105.41 0)
 			(effects
@@
 					(size 1.27 1.27)
 				)
+				(hide yes)
 			)
 		)
@@
 			)
 		)
-		(property "Description" ""
+		(property "Description" "POWERSUPPLY"
 			(at 100.33 25.4 0)
 			(effects
@@
 					(size 1.27 1.27)
 				)
+				(hide yes)
 			)
 		)
@@
 			)
 		)
-		(property "Description" ""
+		(property "Description" "APD"
 			(at 246.38 143.51 0)
 			(effects
@@
 					(size 1.27 1.27)
 				)
+				(hide yes)
 			)
 		)
@@
 			)
 		)
-		(property "Description" ""
+		(property "Description" "POWERSUPPLY"
 			(at 147.32 40.64 0)
 			(effects
@@
 					(size 1.27 1.27)
 				)
+				(hide yes)
 			)
 		)
@@
 			)
 		)
-		(property "Description" ""
+		(property "Description" "POWERSUPPLY"
 			(at 158.75 40.64 0)
 			(effects
@@
 					(size 1.27 1.27)
 				)
+				(hide yes)
 			)
 		)
@@
 			)
 		)
-		(property "Description" ""
+		(property "Description" "APD"
 			(at 260.35 143.51 0)
 			(effects
@@
 					(size 1.27 1.27)
 				)
+				(hide yes)
 			)
 		)
@@
 			)
 		)
-		(property "Description" ""
+		(property "Description" "POWERSUPPLY"
 			(at 115.57 111.76 0)
 			(effects
@@
 					(size 1.27 1.27)
 				)
+				(hide yes)
 			)
 		)

Commit message: aaaaaaa
Parts:
- renumbered C13 to C10, C7 to C11, C9 to C12, C14 to C13, C10 to C14, C11 to C2, C12 to C3, C2 to C4, C3 to C5, C4 to C6, C5 to C7, C6 to C8, C8 to C9, J2 to J1, J1 to J2, JP2 to JP1, JP1 to JP2, R2 to R1, R1 to R2

Commit message: schematic rev b finish?
Parts:
- added C13, C14: 1u, Capacitor_SMD:C_0603_1608Metric_Pad1.08x0.95mm_HandSolder, symbol Device:C
- added U2: TPS7A2018PDBV, Package_TO_SOT_SMD:SOT-23-5, symbol Regulator_Linear:TPS7A20xxxDBV
- renumbered C14 to C10, C2 to C11, C3 to C12, C10 to C15, C13 to C16, C15 to C17, C4 to C2, C5 to C3, C6 to C4, C7 to C5, C8 to C6, C11 to C7, C9 to C8, C12 to C9, J2 to J1, J1 to J2, JP2 to JP1, JP1 to JP2, R2 to R1, R1 to R2, U2 to U3
Connections:
- net +3V3: now also C13.2, U2.1 (IN), U2.3 (EN)
- net GND: now also C13.1, C14.1, U2.2 (GND)
- new net +1V8: C14.2, U2.5 (OUT)

Commit message: sd card is the way probably :(
Other:
- note removed: "DFE252012PD-3R3M=P2 1008 (2520 metric) 3.3uH NOT ANYMORE FIND SOMETHING ELSE"
- note removed: "This was done thx to SOME SUGGESTIONS schottky B5819W ??? analog 3v3 AMS1117-3.3 --> replaced with TLV76133DCY 5v buck MP2451DT-LF-Z from https://www.youtube.com/watch?v=n7kUYVMZIos&list=PLXSyc11qLa1ZGY3nD7to5eQGKGMREhNGl&index=8"
Changed lines of the file:
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@@
-		)
-	)
-	(text "This was done thx to SOME SUGGESTIONS\nschottky B5819W ???\nanalog 3v3 AMS1117-3.3  --> replaced with TLV76133DCY\n5v buck MP2451DT-LF-Z\nfrom https://www.youtube.com/watch?v=n7kUYVMZIos&list=PLXSyc11qLa1ZGY3nD7to5eQGKGMREhNGl&index=8"
-		(exclude_from_sim no)
-		(at 83.82 151.638 0)
-		(effects
-			(font
-				(size 1.27 1.27)
-			)
 		)
 	)
@@
 		)
 	)
-	(text "DFE252012PD-3R3M=P2\n1008 (2520 metric)\n3.3uH\nNOT ANYMORE\nFIND SOMETHING ELSE"
-		(exclude_from_sim no)
-		(at 65.278 33.02 0)
-		(effects
-			(font
-				(size 1.27 1.27)
-			)
-		)
-	)

Commit message: reb b finished
Parts:
- removed C13, C14: 1u, Capacitor_SMD:C_0603_1608Metric_Pad1.08x0.95mm_HandSolder, symbol Device:C
- removed U2: TPS7A2018PDBV, Package_TO_SOT_SMD:SOT-23-5, symbol Regulator_Linear:TPS7A20xxxDBV
- renumbered C15 to C13, C16 to C14, C17 to C15, U3 to U2
